Commit message: Fix diff drive plugin because of deprecation of legacyMode

File: ca_description/urdf/create_base_gazebo.urdf.xacro (robot description, xacro)
@@ -21,5 +21,5 @@
         <publishOdomTF>true</publishOdomTF>
         <publishWheelJointState>true</publishWheelJointState>
-        <legacyMode>true</legacyMode>
+        <legacyMode>false</legacyMode>
         <odometrySource>world</odometrySource>
         <publishTf>1</publishTf>

File: ca_description/urdf/create_wheel.xacro (robot description, xacro)
@@ -28,5 +28,5 @@
     <parent link="base_link" />
     <child link="${prefix}_wheel_link" />
-    <axis xyz="0 1 0" />
+    <axis xyz="0 -1 0" />
   </joint>
 </xacro:macro>
