Commit message: Addressed some changes for better visualizing April tags.

File: ca_description/urdf/april_tag.xacro (robot description, xacro)
@@ -9,15 +9,4 @@
           <box size="0.5 0.5 0.05" />
         </geometry>
-        <gazebo reference="april_tag_link">
-          <material>
-            <uri>file://media/materials/scripts/gazebo.material</uri>
-            <name>Gazebo/Wood</name>
-            <!--script>
-              <uri>model://create_april_tags/materials/scripts </uri>
-              <uri>model://create_april_tags/materials/textures </uri>
-              <name>AprilTag1</name>
-            </script-->
-          </material>
-        </gazebo>
       </visual>
     </link>
@@ -26,4 +15,15 @@
     <child link="april_tag_link"/>
   </joint>
+  <gazebo reference="april_tag_link">
+    <visual>
+      <material>
+        <script>
+          <uri>model://create_april_tags/materials/scripts </uri>
+          <uri>model://create_april_tags/materials/textures </uri>
+          <name>AprilTag5</name>
+        </script>
+      </material>
+    </visual>
+  </gazebo>
   </xacro:macro>
 </robot>

Commit message: Addressed some requested changes.

File: ca_description/urdf/april_tag.xacro (robot description, xacro)
@@ -1,9 +1,7 @@
 <?xml version="1.0" ?>
 <robot xmlns:xacro="http://ros.org/wiki/xacro">
-  <xacro:macro name="april_tag">
-    <xacro:property name="april_tag_z_offset" value="0.3"/>
-    <link name="april_tag_link">
+  <xacro:macro name="april_tag" params="name_prefix *origin">
+    <link name="${name_prefix}_april_tag_link">
       <visual>
-        <origin xyz=" 0 0 ${april_tag_z_offset}" rpy="0 0 0" />
         <geometry>
           <box size="0.5 0.5 0.05" />
@@ -11,9 +9,10 @@
       </visual>
     </link>
-  <joint name="april_tag_joint" type="fixed">
+  <joint name="${name_prefix}_april_tag_joint" type="fixed">
     <parent link="base_link" />
-    <child link="april_tag_link"/>
+    <child link="${name_prefix}_april_tag_link"/>
+    <xacro:insert_block name="origin"/>
   </joint>
-  <gazebo reference="april_tag_link">
+  <gazebo reference="${name_prefix}_april_tag_link">
     <visual>
       <material>

File: ca_description/urdf/create_base.xacro (robot description, xacro)
@@ -45,5 +45,7 @@
     <xacro:create_wheel prefix="right" y_offset="${wheel_separation / -2}" wheel_radius="${wheel_radius}" wheel_width="${wheel_width}"/>
     <xacro:caster_wheel/>
-    <xacro:april_tag/>
+    <xacro:april_tag name_prefix="create1">
+      <origin xyz=" 0 0 0.3" rpy="0 0 0" />
+    </xacro:april_tag>
     <!-- Simulation sensors -->
     <xacro:sim_create_base/>

Commit message: Addressed requested changes.
To do: decrease the size of the environment for using smaller image files from camera.

File: ca_description/urdf/april_tag.xacro (robot description, xacro)
@@ -1,5 +1,5 @@
 <?xml version="1.0" ?>
 <robot xmlns:xacro="http://ros.org/wiki/xacro">
-  <xacro:macro name="april_tag" params="name_prefix *origin">
+  <xacro:macro name="april_tag" params="name_prefix base_link *origin">
     <link name="${name_prefix}_april_tag_link">
       <visual>
@@ -10,5 +10,5 @@
     </link>
   <joint name="${name_prefix}_april_tag_joint" type="fixed">
-    <parent link="base_link" />
+    <parent link="${base_link}" />
     <child link="${name_prefix}_april_tag_link"/>
     <xacro:insert_block name="origin"/>

File: ca_description/urdf/create_base.xacro (robot description, xacro)
@@ -45,5 +45,5 @@
     <xacro:create_wheel prefix="right" y_offset="${wheel_separation / -2}" wheel_radius="${wheel_radius}" wheel_width="${wheel_width}"/>
     <xacro:caster_wheel/>
-    <xacro:april_tag name_prefix="create1">
+    <xacro:april_tag name_prefix="create1" base_link="base_link">
       <origin xyz=" 0 0 0.3" rpy="0 0 0" />
     </xacro:april_tag>
