Commit message: Added requested changes for the light sensor xacro file

File: ca_description/urdf/create_light_sensor.xacro (robot description, xacro)
@@ -1,39 +1,30 @@
 <?xml version="1.0"?>
 <robot xmlns:xacro="http://ros.org/wiki/xacro">
-<xacro:macro name="light_sensor" params="prefix pitch reflect">
+<xacro:macro name="light_sensor" params="prefix *origin *optical_origin">
     <xacro:include filename="$(find ca_description)/urdf/common_properties.xacro"/>
     <xacro:property name="name" value="${prefix}_light_sensor"/>
     <xacro:property name="parent_link" value="base_link"/>
-    <xacro:property name="x" value="0.095"/>
-    <xacro:property name="y" value="0.14"/>
-    <xacro:property name="z" value="0.065"/>
-    <xacro:property name="R" value="0"/>
-    <xacro:property name="P" value="${pitch}"/>
-    <xacro:property name="Y" value="${pi/2}"/>
         <joint name="${name}_joint" type="fixed">
-            <origin xyz="${x} ${y*reflect} ${z}" rpy="0 ${P} 0" doc="x es para adelante, y para izquierda, z para arriba"/>
+            <xacro:insert_block name="origin"/>
             <parent link="${parent_link}" />
             <child link="${name}_link" />
-            <axis xyz="0 1 0" />
         </joint>
-        <link name="${name}_link"/>
+        <link name="${name}_link">
         <visual>
-            <origin xyz="0 0 0" rpy="0 ${pi/2} 0" />
             <geometry>
-                <mesh filename="package://ca_description/meshes/last_lens.stl" scale=".0005 .0005 .0005  "/>
-                <box size=".02 .01 .01" doc="'x' es para arriba, 'y' para adelante y 'z' para la derecha"/>
+                <mesh filename="package://ca_description/meshes/last_lens.stl" />
             </geometry>
             <material name="blue">
-                <color rgba="0 0 1 1"/>
+                <color rgba="0 0 1.0 1.0"/>
             </material>
         </visual>
         </link>
         <joint name="${name}_optical_joint" type="fixed">
-            <origin xyz="0.042 0 0" rpy="${-pi/2} 0 ${-pi/2}" />
+            <xacro:insert_block name="optical_origin"/>
             <parent link="${name}_link" />
             <child link="${name}_optical_frame"/>
         </joint>
         <link name="${name}_optical_frame"/>
-        <gazebo reference="${name}">
+        <gazebo reference="${name}_link">
             <material>Gazebo/Blue</material>
         </gazebo>

Commit message: Added files for the robot to follow the lines. The python script is not fully functional. Still have to fix some issues.

File: ca_description/urdf/create_light_sensor.xacro (robot description, xacro)
@@ -3,5 +3,5 @@
 <xacro:macro name="color_sensor" params="name_prefix sensor_color *origin">
     <xacro:include filename="$(find ca_description)/urdf/common_properties.xacro"/>
-    <xacro:property name="name" value="${name_prefix}_light_sensor"/>
+    <xacro:property name="name" value="${name_prefix}_color_sensor"/>
     <xacro:property name="parent_link" value="base_link"/>
         <joint name="${name}_joint" type="fixed">
@@ -50,5 +50,5 @@
                 <cameraName>${name}_camera</cameraName>
                 <alwaysOn>true</alwaysOn>
-                <updateRate>30</updateRate>
+                <updateRate>50</updateRate>
                 <imageTopicName>rgb/image_raw</imageTopicName>
                 <depthImageTopicName>depth/image_raw</depthImageTopicName>
