Commit message: Move roomblock up

File: ca_description/urdf/roomblock.xacro (robot description, xacro)
@@ -9,5 +9,5 @@
   <xacro:include filename="$(find ca_description)/urdf/sensors/camera_sensor.xacro"/>
   <xacro:macro name="roomblock" params="parent visualize:=false">
-    <xacro:property name="z" value="0.061"/>
+    <xacro:property name="z" value="0.07"/>
     <xacro:property name="roomblock_link" value="block_link"/>
     <xacro:property name="parent_link" value="${parent}"/>

Commit message: Edit roomblock

File: ca_description/urdf/roomblock.xacro (robot description, xacro)
@@ -1,11 +1,11 @@
 <?xml version="1.0"?>
 <!--
-Block on top of the Create 2 that contains a Raspicam and an RPLidar
+Block on top of the iRobot Create 2
 -->
 <robot xmlns:xacro="http://ros.org/wiki/xacro">
   <xacro:include filename="$(find ca_description)/urdf/common_properties.xacro"/>
   <xacro:include filename="$(find ca_description)/urdf/roomblock_gazebo.xacro"/>
-  <xacro:include filename="$(find ca_description)/urdf/sensors/laser_sensor.xacro"/>
   <xacro:include filename="$(find ca_description)/urdf/sensors/camera_sensor.xacro"/>
+  <xacro:include filename="$(find ca_description)/urdf/sensors/lasers/rplidar.xacro"/>
   <xacro:macro name="roomblock" params="parent visualize:=false">
     <xacro:property name="z" value="0.07"/>
@@ -17,5 +17,5 @@
     <xacro:property name="roomblock_size_z" value="0.07"/>
     <joint name="block_joint" type="fixed">
-      <origin xyz="0 0 ${z}" rpy="0 0 0" />
+      <origin xyz="0 0 ${z}"/>
       <parent link="${parent_link}"/>
       <child link="${roomblock_link}" />
@@ -32,8 +32,12 @@
                                        y_length="${roomblock_size_y}"
                                        z_length="${roomblock_size_z}">
-        <origin xyz="0 0 ${roomblock_size_z/2}" rpy="0 0 0"/>
+        <origin xyz="0 0 ${roomblock_size_z/2}"/>
       </xacro:inertial_cuboid_with_pose>
     </link>
-    <xacro:laser_sensor parent="${roomblock_link}" visualize="$(arg visualize)"/>
+    <xacro:rplidar parent="${roomblock_link}" visualize="$(arg visualize)">
+      <origin xyz="0 0 0.1"/>
+    </xacro:rplidar>
+    <!-- TODO: REMOVE VISUALIZE USING ARG OR XACRO:ARG -->
+    <!-- TODO (eborghi): ADD CAMERA CAD? REMOVE CAMERA/USE ANOTHER ONE? -->
     <xacro:camera_sensor parent="${roomblock_link}"/>
     <xacro:roomblock_gazebo link_name="${roomblock_link}"/>

Commit message: WIP

File: ca_description/urdf/roomblock.xacro (robot description, xacro)
@@ -35,10 +35,10 @@
       </xacro:inertial_cuboid_with_pose>
     </link>
-    <xacro:rplidar parent="${roomblock_link}" visualize="$(arg visualize)">
+    <xacro:rplidar parent="${roomblock_link}" visualize="${visualize}">
       <origin xyz="0 0 0.1"/>
     </xacro:rplidar>
     <!-- TODO: REMOVE VISUALIZE USING ARG OR XACRO:ARG -->
     <!-- TODO (eborghi): ADD CAMERA CAD? REMOVE CAMERA/USE ANOTHER ONE? -->
-    <xacro:camera_sensor parent="${roomblock_link}"/>
+    <!-- <xacro:camera_sensor parent="${roomblock_link}"/> -->
     <xacro:roomblock_gazebo link_name="${roomblock_link}"/>
   </xacro:macro>

File: ca_description/urdf/sensors/lasers/rplidar.xacro (robot description, xacro)
@@ -1,11 +1,11 @@
 <?xml version="1.0"?>
 <robot xmlns:xacro="http://ros.org/wiki/xacro">
+<xacro:include filename="$(find ca_description)/urdf/sensors/lasers/rplidar_gazebo.xacro"/>
 <xacro:macro name="rplidar" params="parent visualize:=false *origin">
-  <xacro:include filename="$(find ca_description)/urdf/sensors/lasers/rplidar_gazebo.xacro"/>
-  <xacro:property name="parent_link" value="${parent}"/>
-  <xacro:property name="link_name" value="rplidar_link"/>
+  <xacro:property name="link_name"  value="rplidar_link"/>
+  <xacro:property name="laser_name" value="laser_link"/>
   <joint name="rplidar_joint" type="fixed">
     <xacro:insert_block name="origin"/>
-    <parent link="${parent_link}"/>
+    <parent link="${parent}"/>
     <child link="${link_name}"/>
   </joint>
@@ -17,6 +17,51 @@
     </visual>
   </link>
+  <joint name="laser_joint" type="fixed">
+    <origin xyz="0 0 0.0308"/>
+    <parent link="${link_name}"/>
+    <child link="${laser_name}"/>
+  </joint>
+  <link name="${laser_name}"/>
+  <!-- <xacro:property name="rplidar_a2_rate_hz" value="10"/>
+  <xacro:property name="rplidar_a2_min_range_m" value="0.15"/>
+  <xacro:property name="rplidar_a2_max_range_m" value="12.0"/>
+  <xacro:property name="rplidar_a2_samples" value="720"/>
+  <xacro:property name="rplidar_a2_resolution_mm" value="0.5"/>
+  <xacro:property name="rplidar_a2_min_angle_rad" value="${-pi}"/>
+  <xacro:property name="rplidar_a2_max_angle_rad" value="${pi}"/>
+  <xacro:property name="topic_name" value="laser/scan"/>
+  <gazebo reference="${laser_name}">
+    <material>Gazebo/FlatBlack</material>
+    <sensor type="ray" name="rplidar_sensor">
+      <visualize>true</visualize>
+      <update_rate>${rplidar_a2_rate_hz}</update_rate>
+      <ray>
+        <scan>
+          <horizontal>
+            <samples>${rplidar_a2_samples}</samples>
+            <resolution>1</resolution>
+            <min_angle>${rplidar_a2_min_angle_rad}</min_angle>
+            <max_angle>${rplidar_a2_max_angle_rad}</max_angle>
+          </horizontal>
+        </scan>
+        <range>
+          <min>${rplidar_a2_min_range_m}</min>
+          <max>${rplidar_a2_max_range_m}</max>
+          <resolution>${rplidar_a2_resolution_mm / 1000.0}</resolution>
+        </range>
+        <noise>
+          <type>gaussian</type>
+          <mean>0.0</mean>
+          <stddev>0.01</stddev>
+        </noise>
+      </ray>
+      <plugin name="gazebo_ros_rplidar_sensor" filename="libgazebo_ros_laser.so">
+        <topicName>${topic_name}</topicName>
+        <frameName>${laser_name}</frameName>
+      </plugin>
+    </sensor>
+  </gazebo> -->
   <!-- Gazebo plugin -->
-  <xacro:rplidar_gazebo link_name="{link_name}" visualize="$(arg visualize)"/>
+  <xacro:rplidar_gazebo link_name="${laser_name}" visualize="${visualize}"/>
 </xacro:macro>
 </robot>

File: ca_description/urdf/sensors/lasers/rplidar_gazebo.xacro (robot description, xacro)
@@ -11,8 +11,8 @@
   <xacro:property name="topic_name" value="laser/scan"/>
   <gazebo reference="${link_name}">
-    <material>Gazebo/Black</material>
+    <material>Gazebo/FlatBlack</material>
     <sensor type="ray" name="rplidar_sensor">
       <pose>0 0 0 0 0 0</pose>
-      <visualize>$(arg visualize)</visualize>
+      <visualize>${visualize}</visualize>
       <update_rate>${rplidar_a2_rate_hz}</update_rate>
       <ray>
