Commit message: Fix wheel rotation

File: ca_description/urdf/create_wheel.xacro (robot description, xacro)
@@ -8,7 +8,7 @@
   <joint name="${name}_joint" type="continuous">
     <xacro:insert_block name="origin"/>
-    <parent link="${parent_link}" />
-    <child link="${link_name}" />
-    <axis xyz="0 1 0" />
+    <parent link="${parent_link}"/>
+    <child link="${link_name}"/>
+    <axis xyz="0 0 1"/>
   </joint>
   <link name="${link_name}">
