Commit message: Fix URDF to include contact in bumpers

File: ca_description/urdf/create_base.xacro (robot description, xacro)
@@ -26,5 +26,5 @@
         </geometry>
       </visual>
-      <collision>
+      <collision name="base_link">
         <origin xyz="0 0 ${base_link_offset_z}" rpy="0 0 0" />
         <geometry>

File: ca_description/urdf/create_base_gazebo.xacro (robot description, xacro)
@@ -41,5 +41,5 @@
     </gazebo>
     <!-- Bumpers -->
-    <gazebo reference="base_link">
+    <gazebo reference="base_footprint">
       <gravity>true</gravity>
       <self_collide>false</self_collide>
@@ -48,10 +48,9 @@
         <update_rate>50</update_rate>
         <contact>
-          <collision>base_link_collision</collision>
-          <topic>bumpers</topic>
+          <collision>base_footprint_collision</collision>
         </contact>
         <!-- Plugin -->
         <plugin name="create_bumper_controller" filename="libcreate_bumper_plugin.so">
-          <frameName>base_link</frameName>
+          <frameName>base_footprint</frameName>
           <bumperTopicName>bumper</bumperTopicName>
         </plugin>

Commit message: Clean up and improve XACRO model

File: ca_description/urdf/create_base.xacro (robot description, xacro)
@@ -1,6 +1,6 @@
 <?xml version="1.0" ?>
 <robot xmlns:xacro="http://ros.org/wiki/xacro">
-  <xacro:macro name="create_base" params="diffdrive_update_rate:=40 wheel_separation wheel_radius:=0.036 wheel_width:=0.024 wheel_torque:=0.5 wheel_accel:=0.5 mass_kg:=3.5 base_diameter *mesh visualize:=false">
-    <xacro:include filename="$(find ca_description)/urdf/create_base_gazebo.urdf.xacro"/>
+  <xacro:macro name="create_base" params="wheel_separation wheel_radius wheel_width base_diameter *mesh visualize:=false">
+    <xacro:include filename="$(find ca_description)/urdf/create_base_gazebo.xacro"/>
     <xacro:include filename="$(find ca_description)/urdf/create_caster_wheel.xacro"/>
     <xacro:include filename="$(find ca_description)/urdf/create_wheel.xacro"/>
@@ -8,27 +8,18 @@
     <xacro:include filename="$(find ca_description)/urdf/sensors/wall_sensor.xacro"/>
     <xacro:include filename="$(find ca_description)/urdf/sensors/cliff_sensors.xacro"/>
-    <link name="base_footprint">
-    <visual>
-      <origin xyz="0 0 0" rpy="0 0 0" />
-      <geometry>
-        <box size="0.001 0.001 0.001" />
-      </geometry>
-      <material name="Green" />
-    </visual>
-    <collision>
-      <origin xyz="0 0 0.017" rpy="0 0 0" />
-      <geometry>
-        <box size="0.001 0.001 0.001" />
-      </geometry>
-    </collision>
-    </link>
+    <xacro:property name="base_link_offset_z" value="0.0308"/>
+    <xacro:property name="base_offset_z" value="0.017"/>
+    <xacro:property name="base_height" value="0.0611632"/>
+    <xacro:property name="base_mass" value="2"/>
+    <link name="base_footprint"/>
+    <joint name="base_footprint_joint" type="fixed">
+      <origin xyz="0 0 ${base_offset_z}" rpy="0 0 0" />
+      <parent link="base_footprint" />
+      <child link="base_link" />
+    </joint>
     <link name="base_link">
-      <inertial>
-        <mass value="2" />
-        <origin xyz="0 0 0.0" />
-        <inertia ixx="0.01" ixy="0.0" ixz="0.0" iyy="0.01" iyz="0.0" izz="0.5" />
-      </inertial>
+      <xacro:inertial_cylinder mass="${base_mass}" radius="${base_diameter/2}" length="${base_height}"/>
       <visual>
-        <origin xyz=" 0 0 0.0308" rpy="0 0 0" />
+        <origin xyz=" 0 0 ${base_link_offset_z}" rpy="0 0 0" />
         <geometry>
           <xacro:insert_block name="mesh" />
@@ -36,15 +27,10 @@
       </visual>
       <collision>
-        <origin xyz="0.0 0.0 0.0308" rpy="0 0 0" />
+        <origin xyz="0 0 ${base_link_offset_z}" rpy="0 0 0" />
         <geometry>
-          <cylinder length="0.0611632" radius="0.16495" />
+          <cylinder length="${base_height}" radius="${base_diameter/2}" />
         </geometry>
       </collision>
     </link>
-    <joint name="base_footprint_joint" type="fixed">
-      <origin xyz="0 0 0.017" rpy="0 0 0" />
-      <parent link="base_footprint" />
-      <child link="base_link" />
-    </joint>
     <xacro:wall_sensor visualize="${visualize}"/>
     <xacro:cliff_sensors visualize="${visualize}"/>

File: ca_description/urdf/create_base_gazebo.xacro (robot description, xacro)
@@ -2,4 +2,7 @@
 <robot xmlns:xacro="http://ros.org/wiki/xacro">
   <xacro:macro name="sim_create_base">
+    <xacro:property name="diffdrive_update_rate" value="40"/>
+    <xacro:property name="wheel_torque" value="0.5"/>
+    <xacro:property name="wheel_accel" value="0.5"/>
     <gazebo>
       <!-- Diff-drive controller -->
@@ -28,5 +31,5 @@
       <plugin name="p3d_base_controller" filename="libgazebo_ros_p3d.so">
         <alwaysOn>true</alwaysOn>
-        <updateRate>100.0</updateRate>
+        <updateRate>60.0</updateRate>
         <bodyName>base_link</bodyName>
         <topicName>gts</topicName>

File: ca_description/urdf/roomblock.xacro (robot description, xacro)
@@ -12,4 +12,8 @@
     <xacro:property name="roomblock_link" value="block_link"/>
     <xacro:property name="parent_link" value="${parent}"/>
+    <xacro:property name="roomblock_mass" value="0.1"/>
+    <xacro:property name="roomblock_size_x" value="0.1"/>
+    <xacro:property name="roomblock_size_y" value="0.1"/>
+    <xacro:property name="roomblock_size_z" value="0.07"/>
     <joint name="block_joint" type="fixed">
       <origin xyz="0 0 ${z}" rpy="0 0 0" />
@@ -24,4 +28,10 @@
         <material name="Grey" />
       </visual>
+      <xacro:inertial_cuboid_with_pose mass="${roomblock_mass}"
+                                       x_length="${roomblock_size_x}"
+                                       y_length="${roomblock_size_y}"
+                                       z_length="${roomblock_size_z}">
+        <origin xyz="0 0 ${roomblock_size_z/2}" rpy="0 0 0"/>
+      </xacro:inertial_cuboid_with_pose>
     </link>
     <xacro:laser_sensor parent="${roomblock_link}" visualize="$(arg visualize)"/>

Commit message: Improve IMU

File: ca_description/urdf/create_base.xacro (robot description, xacro)
@@ -35,5 +35,7 @@
     <xacro:wall_sensor visualize="${visualize}"/>
     <xacro:cliff_sensors visualize="${visualize}"/>
-    <xacro:imu_sensor/>
+    <xacro:imu_sensor name="imu">
+      <origin xyz="0 -0.04 0.13" rpy="0 0 0"/>
+    </xacro:imu_sensor>
     <xacro:create_wheel prefix="left" y_offset="${wheel_separation / 2}" wheel_radius="${wheel_radius}" wheel_width="${wheel_width}"/>
     <xacro:create_wheel prefix="right" y_offset="${wheel_separation / -2}" wheel_radius="${wheel_radius}" wheel_width="${wheel_width}"/>

File: ca_description/urdf/sensors/imu_sensor.xacro (robot description, xacro)
@@ -1,17 +1,11 @@
 <?xml version="1.0" ?>
 <robot xmlns:xacro="http://ros.org/wiki/xacro">
-<xacro:macro name="imu_sensor">
+<xacro:macro name="imu_sensor" params="name *origin">
   <xacro:include filename="$(find ca_description)/urdf/common_properties.xacro"/>
   <xacro:include filename="$(find ca_description)/urdf/sensors/imu_sensor_gazebo.xacro"/>
   <xacro:property name="parent_link" value="base_link"/>
-  <xacro:property name="link_name" value="imu_link"/>
-  <xacro:property name="x" value="0"/>
-  <xacro:property name="y" value="-0.04"/>
-  <xacro:property name="z" value="0.13"/>
-  <xacro:property name="R" value="0"/>
-  <xacro:property name="P" value="0"/>
-  <xacro:property name="Y" value="0"/>
-  <joint name="gyro_joint" type="fixed">
-    <origin xyz="${x} ${y} ${z}" rpy="${R} ${P} ${Y}"/>
+  <xacro:property name="link_name" value="${name}_link"/>
+  <joint name="${name}_joint" type="fixed">
+    <xacro:insert_block name="origin" />
     <parent link="${parent_link}" />
     <child link="${link_name}" />
@@ -20,5 +14,5 @@
     <xacro:dummy_inertia/>
   </link>
-  <xacro:imu_sensor_gazebo/>
+  <xacro:imu_sensor_gazebo name="${name}" link_name="${link_name}"/>
 </xacro:macro>
 </robot>

File: ca_description/urdf/sensors/imu_sensor_gazebo.xacro (robot description, xacro)
@@ -1,5 +1,5 @@
 <?xml version="1.0" ?>
 <robot xmlns:xacro="http://ros.org/wiki/xacro">
-<xacro:macro name="imu_sensor_gazebo">
+<xacro:macro name="imu_sensor_gazebo" params="name link_name">
   <gazebo>
     <plugin name="imu_controller" filename="libgazebo_ros_imu.so">
@@ -7,6 +7,6 @@
       <updateRate>30</updateRate>
       <bodyName>${link_name}</bodyName>
-      <topicName>imu/data</topicName>
-      <serviceName>imu/is_calibrated</serviceName>
+      <topicName>${name}/data</topicName>
+      <serviceName>${name}/is_calibrated</serviceName>
       <gaussianNoise>${0.0017*0.0017}</gaussianNoise>
       <xyzOffsets>0 0 0</xyzOffsets>

Commit message: Add base_footprint to Gazebo

File: ca_description/urdf/create_base.xacro (robot description, xacro)
@@ -12,9 +12,12 @@
     <xacro:property name="base_height" value="0.0611632"/>
     <xacro:property name="base_mass" value="2"/>
-    <link name="base_footprint"/>
-    <joint name="base_footprint_joint" type="fixed">
+    <link name="base_footprint">
+      <xacro:dummy_inertia/>
+    </link>
+    <joint name="base_footprint_joint" type="continuous">
       <origin xyz="0 0 ${base_offset_z}" rpy="0 0 0" />
       <parent link="base_footprint" />
       <child link="base_link" />
+      <axis xyz="1 0 0"/>
     </joint>
     <link name="base_link">
@@ -26,5 +29,5 @@
         </geometry>
       </visual>
-      <collision name="base_link">
+      <collision>
         <origin xyz="0 0 ${base_link_offset_z}" rpy="0 0 0" />
         <geometry>

Commit message: Add wirtual wall
Signed-off-by: ivan <ivanpauno@gmail.com>

Corrections

Signed-off-by: ivanpauno <ivanpauno@ekumenlabs.com>

Address Emi's comments

Signed-off-by: ivanpauno <ivanpauno@ekumenlabs.com>

Publish at a certain rate

Signed-off-by: ivanpauno <ivanpauno@ekumenlabs.com>

Launch files combining house and vitual wall

Signed-off-by: ivanpauno <ivanpauno@ekumenlabs.com>

Address newer comments

Signed-off-by: ivanpauno <ivanpauno@ekumenlabs.com>

Added map for two_floor_house world

Changed default value on launch-file

Changed the CMakeLists file

Added plugin to filter the virtual walls messages

Fixed EOF

fixup! Fixed EOF

Addressed the last comments

Addressed the new comments

Modified the state machine to detect virtual walls

Addressed comments

File: ca_description/urdf/create_base.xacro (robot description, xacro)
@@ -8,4 +8,5 @@
     <xacro:include filename="$(find ca_description)/urdf/sensors/wall_sensor.xacro"/>
     <xacro:include filename="$(find ca_description)/urdf/sensors/cliff_sensors.xacro"/>
+    <xacro:include filename="$(find ca_description)/urdf/sensors/omni_sensor.xacro"/>
     <xacro:property name="base_link_offset_z" value="0.0308"/>
     <xacro:property name="base_offset_z" value="0.017"/>
@@ -49,4 +50,7 @@
       <origin xyz="0 -0.04 0.13" rpy="0 0 0"/>
     </xacro:imu_sensor>
+    <xacro:omni_sensor name="omni_sensor" diameter="0.1">
+      <origin xyz="0.145 0 ${base_link_offset_z}" rpy="0 0 0"/>
+    </xacro:omni_sensor>
     <xacro:create_wheel prefix="left" y_offset="${wheel_separation / 2}" wheel_radius="${wheel_radius}" wheel_width="${wheel_width}"/>
     <xacro:create_wheel prefix="right" y_offset="${wheel_separation / -2}" wheel_radius="${wheel_radius}" wheel_width="${wheel_width}"/>

File: ca_description/urdf/create_base_gazebo.xacro (robot description, xacro)
@@ -40,4 +40,10 @@
       </plugin>
     </gazebo>
+    <!-- Virtual Wall detector -->
+    <gazebo>
+      <plugin name="virtual_wall_detector" filename="libvirtual_wall_detector.so">
+        <updateRate>10</updateRate>
+      </plugin>
+    </gazebo>
     <!-- Bumpers -->
     <gazebo reference="base_link">

Commit message: Added to create_base the invocation of the block parameter of light sensor

File: ca_description/urdf/create_base.xacro (robot description, xacro)
@@ -45,6 +45,12 @@
     <xacro:create_wheel prefix="right" y_offset="${wheel_separation / -2}" wheel_radius="${wheel_radius}" wheel_width="${wheel_width}"/>
     <xacro:caster_wheel/>
-    <xacro:light_sensor prefix="left" reflect="1"/>
-    <xacro:light_sensor prefix="right" reflect="-1"/>
+    <xacro:light_sensor prefix="left">
+      <origin xyz="0.095 0.14 0.065" rpy="0 ${pi/4} 0"/>
+      <optical_origin xyz="0.042 0 0" rpy="${-pi/2} 0 ${-pi/2}"/>
+    </xacro:light_sensor>
+    <xacro:light_sensor prefix="right">
+      <origin xyz="0.095 -0.14 0.065" rpy="0 ${pi/4} 0"/>
+      <optical_origin xyz="0.042 0 0" rpy="${-pi/2} 0 ${-pi/2}"/>
+    </xacro:light_sensor>
     <!-- Simulation sensors -->
     <xacro:sim_create_base/>

Commit message: Modified declaration of optical_frame

File: ca_description/urdf/create_base.xacro (robot description, xacro)
@@ -47,9 +47,7 @@
     <xacro:light_sensor prefix="left">
       <origin xyz="0.095 0.14 0.065" rpy="0 ${pi/4} 0"/>
-      <optical_origin xyz="0.042 0 0" rpy="${-pi/2} 0 ${-pi/2}"/>
     </xacro:light_sensor>
     <xacro:light_sensor prefix="right">
       <origin xyz="0.095 -0.14 0.065" rpy="0 ${pi/4} 0"/>
-      <optical_origin xyz="0.042 0 0" rpy="${-pi/2} 0 ${-pi/2}"/>
     </xacro:light_sensor>
     <!-- Simulation sensors -->

File: ca_description/urdf/create_light_sensor.xacro (robot description, xacro)
@@ -1,5 +1,5 @@
 <?xml version="1.0"?>
 <robot xmlns:xacro="http://ros.org/wiki/xacro">
-<xacro:macro name="light_sensor" params="prefix *origin *optical_origin">
+<xacro:macro name="light_sensor" params="prefix *origin">
     <xacro:include filename="$(find ca_description)/urdf/common_properties.xacro"/>
     <xacro:property name="name" value="${prefix}_light_sensor"/>
@@ -21,5 +21,5 @@
         </link>
         <joint name="${name}_optical_joint" type="fixed">
-            <xacro:insert_block name="optical_origin"/>
+            <origin xyz="0.052 0 0" rpy="${-pi/2} 0 ${-pi/2}"/>/>
             <parent link="${name}_link" />
             <child link="${name}_optical_frame"/>

Commit message: Modified sensor visual color and modified 'prefix' argument's name by 'name_prefix'

File: ca_description/urdf/create_base.xacro (robot description, xacro)
@@ -45,8 +45,8 @@
     <xacro:create_wheel prefix="right" y_offset="${wheel_separation / -2}" wheel_radius="${wheel_radius}" wheel_width="${wheel_width}"/>
     <xacro:caster_wheel/>
-    <xacro:light_sensor prefix="left">
+    <xacro:light_sensor name_prefix="left">
       <origin xyz="0.095 0.14 0.065" rpy="0 ${pi/4} 0"/>
     </xacro:light_sensor>
-    <xacro:light_sensor prefix="right">
+    <xacro:light_sensor name_prefix="right">
       <origin xyz="0.095 -0.14 0.065" rpy="0 ${pi/4} 0"/>
     </xacro:light_sensor>

File: ca_description/urdf/create_light_sensor.xacro (robot description, xacro)
@@ -1,7 +1,7 @@
 <?xml version="1.0"?>
 <robot xmlns:xacro="http://ros.org/wiki/xacro">
-<xacro:macro name="light_sensor" params="prefix *origin">
+<xacro:macro name="light_sensor" params="name_prefix *origin">
     <xacro:include filename="$(find ca_description)/urdf/common_properties.xacro"/>
-    <xacro:property name="name" value="${prefix}_light_sensor"/>
+    <xacro:property name="name" value="${name_prefix}_light_sensor"/>
     <xacro:property name="parent_link" value="base_link"/>
         <joint name="${name}_joint" type="fixed">
@@ -27,5 +27,5 @@
         <link name="${name}_optical_frame"/>
         <gazebo reference="${name}_link">
-            <material>Gazebo/Blue</material>
+            <material>Gazebo/DarkGrey</material>
         </gazebo>
 </xacro:macro>

Commit message: Modified xacro files for spawning the color sensor with its corresponding plugin.

File: ca_description/urdf/create_base.xacro (robot description, xacro)
@@ -45,8 +45,8 @@
     <xacro:create_wheel prefix="right" y_offset="${wheel_separation / -2}" wheel_radius="${wheel_radius}" wheel_width="${wheel_width}"/>
     <xacro:caster_wheel/>
-    <xacro:light_sensor name_prefix="left">
+    <xacro:light_sensor name_prefix="left" sensor_color="Yellow">
       <origin xyz="0.095 0.14 0.065" rpy="0 ${pi/4} 0"/>
     </xacro:light_sensor>
-    <xacro:light_sensor name_prefix="right">
+    <xacro:light_sensor name_prefix="right" sensor_color="White">
       <origin xyz="0.095 -0.14 0.065" rpy="0 ${pi/4} 0"/>
     </xacro:light_sensor>

File: ca_description/urdf/create_light_sensor.xacro (robot description, xacro)
@@ -1,5 +1,5 @@
 <?xml version="1.0"?>
 <robot xmlns:xacro="http://ros.org/wiki/xacro">
-<xacro:macro name="light_sensor" params="name_prefix *origin">
+<xacro:macro name="light_sensor" params="name_prefix sensor_color *origin">
     <xacro:include filename="$(find ca_description)/urdf/common_properties.xacro"/>
     <xacro:property name="name" value="${name_prefix}_light_sensor"/>
@@ -29,4 +29,40 @@
             <material>Gazebo/DarkGrey</material>
         </gazebo>
+        <gazebo reference="${name}_link">
+            <sensor name='camera' type='camera'>
+            <camera name='__default__'>
+                <horizontal_fov>0.5</horizontal_fov>
+                <image>
+                <width>40</width>
+                <height>40</height>
+                </image>
+                <clip>
+                <near>0.1</near>
+                <far>100</far>
+                </clip>
+            </camera>
+            <plugin name="gazebo_color_sensor_plugin" filename="libgazebo_color_sensor_plugin.so">
+                <publishTopicName>${name}_color_sensor</publishTopicName>
+                <sensorColor>${sensor_color}</sensorColor>
+                <cameraName>${name}_camera</cameraName>
+                <alwaysOn>true</alwaysOn>
+                <updateRate>10</updateRate>
+                <imageTopicName>rgb/image_raw</imageTopicName>
+                <depthImageTopicName>depth/image_raw</depthImageTopicName>
+                <pointCloudTopicName>depth/points</pointCloudTopicName>
+                <cameraInfoTopicName>rgb/camera_info</cameraInfoTopicName>
+                <depthImageCameraInfoTopicName>depth/camera_info</depthImageCameraInfoTopicName>
+                <frameName>${name}_camera_optical_frame</frameName>
+                <baseline>0.1</baseline>
+                <distortion_k1>0.0</distortion_k1>
+                <distortion_k2>0.0</distortion_k2>
+                <distortion_k3>0.0</distortion_k3>
+                <distortion_t1>0.0</distortion_t1>
+                <distortion_t2>0.0</distortion_t2>
+                <pointCloudCutoff>0.4</pointCloudCutoff>
+                <robotNamespace>/</robotNamespace>
+            </plugin>
+        </sensor>
+        </gazebo>
 </xacro:macro>
 </robot>

Commit message: Reduced environment size and adjusted camera rotation.
To do: upload apriltag_ros as as internal package in create_autonomy.

File: ca_description/urdf/create_base.xacro (robot description, xacro)
@@ -46,5 +46,5 @@
     <xacro:caster_wheel/>
     <xacro:april_tag name_prefix="create1" base_link="base_link">
-      <origin xyz=" 0 0 0.3" rpy="0 0 0" />
+      <origin xyz=" 0 0 0.3" rpy="0 0 1.58" />
     </xacro:april_tag>
     <!-- Simulation sensors -->

File: ca_description/urdf/create_base_gazebo.xacro (robot description, xacro)
@@ -35,5 +35,5 @@
         <topicName>gts</topicName>
         <gaussianNoise>0</gaussianNoise>
-        <frameName>map</frameName>
+        <frameName>/map</frameName>
         <xyzOffsets>0 0 0</xyzOffsets>
         <rpyOffsets>0 0 0</rpyOffsets>

Commit message: Added files for the robot to follow the lines. The python script is not fully functional. Still have to fix some issues.

File: ca_description/urdf/create_base.xacro (robot description, xacro)
@@ -45,10 +45,10 @@
     <xacro:create_wheel prefix="right" y_offset="${wheel_separation / -2}" wheel_radius="${wheel_radius}" wheel_width="${wheel_width}"/>
     <xacro:caster_wheel/>
-    <xacro:light_sensor name_prefix="left" sensor_color="Yellow">
+    <xacro:color_sensor name_prefix="left" sensor_color="Yellow">
       <origin xyz="0.095 0.14 0.065" rpy="0 ${pi/4} 0"/>
-    </xacro:light_sensor>
-    <xacro:light_sensor name_prefix="right" sensor_color="White">
+    </xacro:color_sensor>
+    <xacro:color_sensor name_prefix="right" sensor_color="White">
       <origin xyz="0.095 -0.14 0.065" rpy="0 ${pi/4} 0"/>
-    </xacro:light_sensor>
+    </xacro:color_sensor>
     <!-- Simulation sensors -->
     <xacro:sim_create_base/>

File: ca_description/urdf/create_light_sensor.xacro (robot description, xacro)
@@ -1,7 +1,7 @@
 <?xml version="1.0"?>
 <robot xmlns:xacro="http://ros.org/wiki/xacro">
-<xacro:macro name="light_sensor" params="name_prefix sensor_color *origin">
+<xacro:macro name="color_sensor" params="name_prefix sensor_color *origin">
     <xacro:include filename="$(find ca_description)/urdf/common_properties.xacro"/>
-    <xacro:property name="name" value="${name_prefix}_light_sensor"/>
+    <xacro:property name="name" value="${name_prefix}_color_sensor"/>
     <xacro:property name="parent_link" value="base_link"/>
         <joint name="${name}_joint" type="fixed">
@@ -45,10 +45,10 @@
                 <!--Threshold for defining the amount of pixels in an image that has to be the goal color for being considered a positive detection-->
                 <!--Cant be bigger than width*height-->
-                <pixelThreshold>10</pixelThreshold>
-                <publishTopicName>${name}_color_sensor</publishTopicName>
+                <pixelThreshold>100</pixelThreshold>
+                <publishTopicName>${name}</publishTopicName>
                 <sensorColor>${sensor_color}</sensorColor>
                 <cameraName>${name}_camera</cameraName>
                 <alwaysOn>true</alwaysOn>
-                <updateRate>10</updateRate>
+                <updateRate>50</updateRate>
                 <imageTopicName>rgb/image_raw</imageTopicName>
                 <depthImageTopicName>depth/image_raw</depthImageTopicName>
