Commit message: Fixed naming issues with color sensor plugin and changed sensor dimensions.

File: ca_description/urdf/create_base.xacro (robot description, xacro)
@@ -45,8 +45,29 @@
     <xacro:create_wheel prefix="right" y_offset="${wheel_separation / -2}" wheel_radius="${wheel_radius}" wheel_width="${wheel_width}"/>
     <xacro:caster_wheel/>
+<<<<<<< Updated upstream
     <xacro:light_sensor name_prefix="left" sensor_color="Yellow">
       <origin xyz="0.095 0.14 0.065" rpy="0 ${pi/4} 0"/>
     </xacro:light_sensor>
     <xacro:light_sensor name_prefix="right" sensor_color="White">
+=======
+<<<<<<< Updated upstream
+    <xacro:color_sensor name_prefix="left" sensor_color="Yellow">
+      <origin xyz="0.095 0.14 0.065" rpy="0 ${pi/4} 0"/>
+    </xacro:color_sensor>
+    <xacro:color_sensor name_prefix="right" sensor_color="White">
+=======
+<<<<<<< Updated upstream
+    <xacro:light_sensor name_prefix="left" sensor_color="Yellow">
+      <origin xyz="0.095 0.14 0.065" rpy="0 ${pi/4} 0"/>
+    </xacro:light_sensor>
+    <xacro:light_sensor name_prefix="right" sensor_color="White">
+=======
+    <xacro:color_sensor name_prefix="left" sensor_color="yellow">
+      <origin xyz="0.095 0.14 0.065" rpy="0 ${pi/4} 0"/>
+    </xacro:color_sensor>
+    <xacro:color_sensor name_prefix="right" sensor_color="white">
+>>>>>>> Stashed changes
+>>>>>>> Stashed changes
+>>>>>>> Stashed changes
       <origin xyz="0.095 -0.14 0.065" rpy="0 ${pi/4} 0"/>
     </xacro:light_sensor>

File: ca_description/urdf/create_light_sensor.xacro (robot description, xacro)
@@ -34,5 +34,5 @@
                 <horizontal_fov>0.5</horizontal_fov>
                 <image>
-                <width>40</width>
+                <width>20</width>
                 <height>40</height>
                 </image>
@@ -42,7 +42,8 @@
                 </clip>
             </camera>
-            <plugin name="gazebo_color_sensor_plugin" filename="libgazebo_color_sensor_plugin.so">
+            <plugin name="color_sensor_plugin" filename="libcolor_sensor_plugin.so">
                 <!--Threshold for defining the amount of pixels in an image that has to be the goal color for being considered a positive detection-->
                 <!--Cant be bigger than width*height-->
+<<<<<<< Updated upstream
                 <pixelThreshold>10</pixelThreshold>
                 <publishTopicName>${name}_color_sensor</publishTopicName>
@@ -51,4 +52,30 @@
                 <alwaysOn>true</alwaysOn>
                 <updateRate>10</updateRate>
+=======
+<<<<<<< Updated upstream
+                <pixelThreshold>100</pixelThreshold>
+                <publishTopicName>${name}</publishTopicName>
+                <sensorColor>${sensor_color}</sensorColor>
+                <cameraName>${name}_camera</cameraName>
+                <alwaysOn>true</alwaysOn>
+                <updateRate>50</updateRate>
+=======
+<<<<<<< Updated upstream
+                <pixelThreshold>10</pixelThreshold>
+                <publishTopicName>${name}_color_sensor</publishTopicName>
+                <sensorColor>${sensor_color}</sensorColor>
+                <cameraName>${name}_camera</cameraName>
+                <alwaysOn>true</alwaysOn>
+                <updateRate>10</updateRate>
+=======
+                <pixelThreshold>50</pixelThreshold>
+                <publishTopicName>${name}</publishTopicName>
+                <sensorColor>${sensor_color}</sensorColor>
+                <cameraName>${name}_camera</cameraName>
+                <alwaysOn>true</alwaysOn>
+                <updateRate>30</updateRate>
+>>>>>>> Stashed changes
+>>>>>>> Stashed changes
+>>>>>>> Stashed changes
                 <imageTopicName>rgb/image_raw</imageTopicName>
                 <depthImageTopicName>depth/image_raw</depthImageTopicName>

Commit message: Fixed some stash-related mistakes in the code.

File: ca_description/urdf/create_base.xacro (robot description, xacro)
@@ -45,31 +45,10 @@
     <xacro:create_wheel prefix="right" y_offset="${wheel_separation / -2}" wheel_radius="${wheel_radius}" wheel_width="${wheel_width}"/>
     <xacro:caster_wheel/>
-<<<<<<< Updated upstream
-    <xacro:light_sensor name_prefix="left" sensor_color="Yellow">
-      <origin xyz="0.095 0.14 0.065" rpy="0 ${pi/4} 0"/>
-    </xacro:light_sensor>
-    <xacro:light_sensor name_prefix="right" sensor_color="White">
-=======
-<<<<<<< Updated upstream
-    <xacro:color_sensor name_prefix="left" sensor_color="Yellow">
-      <origin xyz="0.095 0.14 0.065" rpy="0 ${pi/4} 0"/>
-    </xacro:color_sensor>
-    <xacro:color_sensor name_prefix="right" sensor_color="White">
-=======
-<<<<<<< Updated upstream
-    <xacro:light_sensor name_prefix="left" sensor_color="Yellow">
-      <origin xyz="0.095 0.14 0.065" rpy="0 ${pi/4} 0"/>
-    </xacro:light_sensor>
-    <xacro:light_sensor name_prefix="right" sensor_color="White">
-=======
     <xacro:color_sensor name_prefix="left" sensor_color="yellow">
       <origin xyz="0.095 0.14 0.065" rpy="0 ${pi/4} 0"/>
     </xacro:color_sensor>
     <xacro:color_sensor name_prefix="right" sensor_color="white">
->>>>>>> Stashed changes
->>>>>>> Stashed changes
->>>>>>> Stashed changes
       <origin xyz="0.095 -0.14 0.065" rpy="0 ${pi/4} 0"/>
-    </xacro:light_sensor>
+    </xacro:color_sensor>
     <!-- Simulation sensors -->
     <xacro:sim_create_base/>

File: ca_description/urdf/create_light_sensor.xacro (robot description, xacro)
@@ -1,5 +1,5 @@
 <?xml version="1.0"?>
 <robot xmlns:xacro="http://ros.org/wiki/xacro">
-<xacro:macro name="light_sensor" params="name_prefix sensor_color *origin">
+<xacro:macro name="color_sensor" params="name_prefix sensor_color *origin">
     <xacro:include filename="$(find ca_description)/urdf/common_properties.xacro"/>
     <xacro:property name="name" value="${name_prefix}_light_sensor"/>
@@ -45,28 +45,4 @@
                 <!--Threshold for defining the amount of pixels in an image that has to be the goal color for being considered a positive detection-->
                 <!--Cant be bigger than width*height-->
-<<<<<<< Updated upstream
-                <pixelThreshold>10</pixelThreshold>
-                <publishTopicName>${name}_color_sensor</publishTopicName>
-                <sensorColor>${sensor_color}</sensorColor>
-                <cameraName>${name}_camera</cameraName>
-                <alwaysOn>true</alwaysOn>
-                <updateRate>10</updateRate>
-=======
-<<<<<<< Updated upstream
-                <pixelThreshold>100</pixelThreshold>
-                <publishTopicName>${name}</publishTopicName>
-                <sensorColor>${sensor_color}</sensorColor>
-                <cameraName>${name}_camera</cameraName>
-                <alwaysOn>true</alwaysOn>
-                <updateRate>50</updateRate>
-=======
-<<<<<<< Updated upstream
-                <pixelThreshold>10</pixelThreshold>
-                <publishTopicName>${name}_color_sensor</publishTopicName>
-                <sensorColor>${sensor_color}</sensorColor>
-                <cameraName>${name}_camera</cameraName>
-                <alwaysOn>true</alwaysOn>
-                <updateRate>10</updateRate>
-=======
                 <pixelThreshold>50</pixelThreshold>
                 <publishTopicName>${name}</publishTopicName>
@@ -75,7 +51,4 @@
                 <alwaysOn>true</alwaysOn>
                 <updateRate>30</updateRate>
->>>>>>> Stashed changes
->>>>>>> Stashed changes
->>>>>>> Stashed changes
                 <imageTopicName>rgb/image_raw</imageTopicName>
                 <depthImageTopicName>depth/image_raw</depthImageTopicName>

Commit message: Corrected xacro file confusing naming of 'light' and 'color' words. Also, deleted some unnecessary tags.

File: ca_description/urdf/create_base.xacro (robot description, xacro)
@@ -5,5 +5,5 @@
     <xacro:include filename="$(find ca_description)/urdf/create_caster_wheel.xacro"/>
     <xacro:include filename="$(find ca_description)/urdf/create_wheel.xacro"/>
-    <xacro:include filename="$(find ca_description)/urdf/create_light_sensor.xacro"/>
+    <xacro:include filename="$(find ca_description)/urdf/create_color_sensor.xacro"/>
     <xacro:include filename="$(find ca_description)/urdf/sensors/imu_sensor.xacro"/>
     <xacro:include filename="$(find ca_description)/urdf/sensors/wall_sensor.xacro"/>
@@ -45,9 +45,9 @@
     <xacro:create_wheel prefix="right" y_offset="${wheel_separation / -2}" wheel_radius="${wheel_radius}" wheel_width="${wheel_width}"/>
     <xacro:caster_wheel/>
+    <xacro:color_sensor name_prefix="right" sensor_color="white">
+      <origin xyz="0.095 -0.14 0.065" rpy="0 ${pi/4} 0"/>
+    </xacro:color_sensor>
     <xacro:color_sensor name_prefix="left" sensor_color="yellow">
       <origin xyz="0.095 0.14 0.065" rpy="0 ${pi/4} 0"/>
-    </xacro:color_sensor>
-    <xacro:color_sensor name_prefix="right" sensor_color="white">
-      <origin xyz="0.095 -0.14 0.065" rpy="0 ${pi/4} 0"/>
     </xacro:color_sensor>
     <!-- Simulation sensors -->

File: ca_description/urdf/create_color_sensor.xacro (robot description, xacro)
@@ -3,5 +3,5 @@
 <xacro:macro name="color_sensor" params="name_prefix sensor_color *origin">
     <xacro:include filename="$(find ca_description)/urdf/common_properties.xacro"/>
-    <xacro:property name="name" value="${name_prefix}_light_sensor"/>
+    <xacro:property name="name" value="${name_prefix}_color_sensor"/>
     <xacro:property name="parent_link" value="base_link"/>
         <joint name="${name}_joint" type="fixed">
@@ -49,5 +49,4 @@
                 <sensorColor>${sensor_color}</sensorColor>
                 <cameraName>${name}_camera</cameraName>
-                <always_on>true</always_on>
                 <updateRate>30</updateRate>
                 <imageTopicName>rgb/image_raw</imageTopicName>

Commit message: Supress warning of invalid parent link

File: ca_description/urdf/create_base.xacro (robot description, xacro)
@@ -12,4 +12,12 @@
     <xacro:property name="base_height" value="0.0611632"/>
     <xacro:property name="base_mass" value="2"/>
+    <!-- The root link base_footprint has an inertia specified in the URDF,
+         but KDL does not support a root link with an inertia.
+         As a workaround, you can add an extra dummy link to your URDF. -->
+    <joint name="fixed_joint" type="fixed">
+      <parent link="dummy_link"/>
+      <child link="base_footprint"/>
+    </joint>
+    <link name="dummy_link"/>
     <link name="base_footprint">
       <xacro:dummy_inertia/>

Commit message: Do some modifications

File: ca_description/urdf/create_base.xacro (robot description, xacro)
@@ -46,5 +46,16 @@
     </link>
     <xacro:wall_sensor visualize="${visualize}"/>
-    <xacro:cliff_sensors visualize="${visualize}"/>
+    <xacro:cliff_sensor name="side_left">
+      <origin xyz="0.07 0.14 0.01" rpy="0 ${pi/2 - 0.09} 0" />
+    </xacro:cliff_sensor>
+    <xacro:cliff_sensor name="side_right">
+      <origin xyz="0.07 -0.14 0.01" rpy="0 ${pi/2 - 0.09} 0" />
+    </xacro:cliff_sensor>
+    <xacro:cliff_sensor name="front_left">
+      <origin xyz="0.15 0.04 0.01" rpy="0 ${pi/2 - 0.09} 0" />
+    </xacro:cliff_sensor>
+    <xacro:cliff_sensor name="front_right">
+      <origin xyz="0.15 -0.04 0.01" rpy="0 ${pi/2 - 0.09} 0" />
+    </xacro:cliff_sensor>
     <xacro:imu_sensor name="imu">
       <origin xyz="0 -0.04 0.13" rpy="0 0 0"/>

File: ca_description/urdf/sensors/cliff_sensors.xacro (robot description, xacro)
@@ -1,29 +1,15 @@
 <?xml version="1.0" ?>
 <robot xmlns:xacro="http://ros.org/wiki/xacro">
-<xacro:macro name="cliff_sensors" params="visualize:=false">
+<xacro:macro name="cliff_sensor" params="name *origin visualize:=false">
   <xacro:include filename="$(find ca_description)/urdf/common_properties.xacro"/>
   <xacro:include filename="$(find ca_description)/urdf/sensors/cliff_sensors_gazebo.xacro"/>
   <xacro:property name="parent_link" value="base_link"/>
-  <xacro:macro name="cliff" params="name *origin">
-    <joint name="${name}_cliff_sensor_joint" type="fixed">
-      <xacro:insert_block name="origin" />
-      <parent link="${parent_link}" />
-      <child link="${name}_cliff_sensor_link" />
-    </joint>
-    <link name="${name}_cliff_sensor_link" />
-    <xacro:cliff_plugin visualize="${visualize}" name="${name}"/>
-  </xacro:macro>
-  <xacro:cliff name="side_left">
-    <origin xyz="0.07 0.14 0.01" rpy="0 ${pi/2 - 0.09} 0" />
-  </xacro:cliff>
-  <xacro:cliff name="side_right">
-    <origin xyz="0.07 -0.14 0.01" rpy="0 ${pi/2 - 0.09} 0" />
-  </xacro:cliff>
-  <xacro:cliff name="front_left">
-    <origin xyz="0.15 0.04 0.01" rpy="0 ${pi/2 - 0.09} 0" />
-  </xacro:cliff>
-  <xacro:cliff name="front_right">
-    <origin xyz="0.15 -0.04 0.01" rpy="0 ${pi/2 - 0.09} 0" />
-  </xacro:cliff>
+  <joint name="${name}_cliff_sensor_joint" type="fixed">
+    <xacro:insert_block name="origin" />
+    <parent link="${parent_link}" />
+    <child link="${name}_cliff_sensor_link" />
+  </joint>
+  <link name="${name}_cliff_sensor_link" />
+  <xacro:cliff_plugin visualize="${visualize}" name="${name}"/>
 </xacro:macro>
 </robot>

Commit message: Set parent for cliff sensors

File: ca_description/urdf/create_base.xacro (robot description, xacro)
@@ -46,14 +46,14 @@
     </link>
     <xacro:wall_sensor visualize="${visualize}"/>
-    <xacro:cliff_sensor name="side_left">
+    <xacro:cliff_sensor name="side_left" parent="base_link">
       <origin xyz="0.07 0.14 0.01" rpy="0 ${pi/2 - 0.09} 0" />
     </xacro:cliff_sensor>
-    <xacro:cliff_sensor name="side_right">
+    <xacro:cliff_sensor name="side_right" parent="base_link">
       <origin xyz="0.07 -0.14 0.01" rpy="0 ${pi/2 - 0.09} 0" />
     </xacro:cliff_sensor>
-    <xacro:cliff_sensor name="front_left">
+    <xacro:cliff_sensor name="front_left" parent="base_link">
       <origin xyz="0.15 0.04 0.01" rpy="0 ${pi/2 - 0.09} 0" />
     </xacro:cliff_sensor>
-    <xacro:cliff_sensor name="front_right">
+    <xacro:cliff_sensor name="front_right" parent="base_link">
       <origin xyz="0.15 -0.04 0.01" rpy="0 ${pi/2 - 0.09} 0" />
     </xacro:cliff_sensor>

File: ca_description/urdf/sensors/cliff_sensors.xacro (robot description, xacro)
@@ -1,8 +1,8 @@
 <?xml version="1.0" ?>
 <robot xmlns:xacro="http://ros.org/wiki/xacro">
-<xacro:macro name="cliff_sensor" params="name *origin visualize:=false">
+<xacro:macro name="cliff_sensor" params="name parent *origin visualize:=false">
   <xacro:include filename="$(find ca_description)/urdf/common_properties.xacro"/>
   <xacro:include filename="$(find ca_description)/urdf/sensors/cliff_sensors_gazebo.xacro"/>
-  <xacro:property name="parent_link" value="base_link"/>
+  <xacro:property name="parent_link" value="${parent}"/>
   <joint name="${name}_cliff_sensor_joint" type="fixed">
     <xacro:insert_block name="origin" />

Commit message: Remove dummy link

File: ca_description/urdf/create_base.xacro (robot description, xacro)
@@ -17,14 +17,14 @@
          but KDL does not support a root link with an inertia.
          As a workaround, you can add an extra dummy link to your URDF. -->
-    <joint name="fixed_joint" type="fixed">
+    <!-- <joint name="fixed_joint" type="fixed">
       <parent link="dummy_link"/>
       <child link="base_footprint"/>
     </joint>
-    <link name="dummy_link"/>
+    <link name="dummy_link"/> -->
     <link name="base_footprint">
       <xacro:dummy_inertia/>
     </link>
     <joint name="base_footprint_joint" type="continuous">
-      <origin xyz="0 0 ${base_offset_z}" rpy="0 0 0" />
+      <origin xyz="0 0 ${base_offset_z}"/>
       <parent link="base_footprint" />
       <child link="base_link" />
@@ -34,5 +34,5 @@
       <xacro:inertial_cylinder mass="${base_mass}" radius="${base_diameter/2}" length="${base_height}"/>
       <visual>
-        <origin xyz=" 0 0 ${base_link_offset_z}" rpy="0 0 0" />
+        <origin xyz=" 0 0 ${base_link_offset_z}"/>
         <geometry>
           <xacro:insert_block name="mesh" />
@@ -40,5 +40,5 @@
       </visual>
       <collision>
-        <origin xyz="0 0 ${base_link_offset_z}" rpy="0 0 0" />
+        <origin xyz="0 0 ${base_link_offset_z}"/>
         <geometry>
           <cylinder length="${base_height}" radius="${base_diameter/2}" />
