Commit message: Improve robot_description and fix base_footprint

File: ca_description/urdf/create_base.xacro (robot description, xacro)
@@ -10,30 +10,22 @@
   <xacro:include filename="$(find ca_description)/urdf/sensors/omni_sensor.xacro"/>
   <xacro:macro name="create_base" params="wheel_separation wheel_radius wheel_width base_diameter *mesh">
-    <xacro:property name="base_link_offset_z" value="0.0308"/>
-    <xacro:property name="base_offset_z" value="0.017"/>
-    <xacro:property name="base_height" value="0.0611632"/>
-    <xacro:property name="base_mass" value="2"/>
+    <xacro:property name="caster_radius" value="0.018"/>
+    <xacro:property name="base_offset_z" value="${wheel_radius}"/>
+    <xacro:property name="base_height"   value="0.0611632"/>
+    <xacro:property name="base_mass"     value="2"/>
     <xacro:arg name="visualize" default="false"/>
-    <!-- The root link base_footprint has an inertia specified in the URDF,
-         but KDL does not support a root link with an inertia.
-         As a workaround, you can add an extra dummy link to your URDF. -->
-    <!-- <joint name="fixed_joint" type="fixed">
-      <parent link="dummy_link"/>
-      <child link="base_footprint"/>
+    <link name="base_footprint"/>
+    <joint name="base_footprint_joint" type="fixed">
+      <origin xyz="0 0 ${base_offset_z}"/>
+      <parent link="base_footprint"/>
+      <child link="base_link"/>
     </joint>
-    <link name="dummy_link"/> -->
-    <link name="base_footprint">
-      <xacro:dummy_inertia/>
-    </link>
-    <joint name="base_footprint_joint" type="continuous">
-      <origin xyz="0 0 ${base_offset_z}"/>
-      <parent link="base_footprint" />
-      <child link="base_link" />
-      <axis xyz="1 0 0"/>
-    </joint>
-    <link name="base_link">
-      <xacro:inertial_cylinder mass="${base_mass}" radius="${base_diameter/2}" length="${base_height}"/>
+    <xacro:property name="base_link_origin" value="0 0 ${base_offset_z - caster_radius}"/>
+  <link name="base_link">
+    <xacro:inertial_cylinder_with_pose mass="${base_mass}" radius="${base_diameter/2}" length="${base_height}">
+      <origin xyz="${base_link_origin}"/>
+      </xacro:inertial_cylinder_with_pose>
       <visual>
-        <origin xyz=" 0 0 ${base_link_offset_z}"/>
+        <origin xyz="${base_link_origin}"/>
         <geometry>
           <xacro:insert_block name="mesh" />
@@ -41,5 +33,5 @@
       </visual>
       <collision>
-        <origin xyz="0 0 ${base_link_offset_z}"/>
+        <origin xyz="${base_link_origin}"/>
         <geometry>
           <cylinder length="${base_height}" radius="${base_diameter/2}" />
@@ -65,15 +57,16 @@
       <origin xyz="0 -0.04 0.13"/>
     </xacro:imu_sensor>
-    <xacro:omni_sensor diameter="0.1">
-      <origin xyz="0.145 0 ${base_link_offset_z}"/>
+    <xacro:omni_sensor>
+      <origin xyz="0.145 0 0.0308"/>
     </xacro:omni_sensor>
     <xacro:wheel name="wheel_left" radius="${wheel_radius}" width="${wheel_width}">
-      <origin xyz="0 ${wheel_separation/2} 0.015" rpy="0 ${pi/2} ${pi/2}"/>
+      <origin xyz="0 ${wheel_separation/2} 0" rpy="0 ${pi/2} ${pi/2}"/>
     </xacro:wheel>
     <xacro:wheel name="wheel_right" radius="${wheel_radius}" width="${wheel_width}">
-      <origin xyz="0 ${-wheel_separation/2} 0.015" rpy="0 ${pi/2} ${pi/2}"/>
+      <origin xyz="0 ${-wheel_separation/2} 0" rpy="0 ${pi/2} ${pi/2}"/>
     </xacro:wheel>
-    <xacro:caster_wheel>
-      <origin xyz="0.13 0 0"/>
+    <xacro:property name="caster_z" value="${-caster_radius}"/>
+    <xacro:caster_wheel radius="${caster_radius}">
+      <origin xyz="0.13 0 ${caster_z}"/>
     </xacro:caster_wheel>
     <!-- Simulation sensors -->

File: ca_description/urdf/create_base_gazebo.xacro (robot description, xacro)
@@ -24,12 +24,11 @@
         <publishOdomTF>true</publishOdomTF>
         <publishWheelJointState>true</publishWheelJointState>
-        <legacyMode>false</legacyMode>
         <odometrySource>world</odometrySource>
-        <publishTf>1</publishTf>
+        <publishTf>true</publishTf>
       </plugin>
       <!-- Ground truth -->
       <plugin name="p3d_base_controller" filename="libgazebo_ros_p3d.so">
         <alwaysOn>true</alwaysOn>
-        <updateRate>60.0</updateRate>
+        <updateRate>60</updateRate>
         <robotNamespace>create1_tf</robotNamespace>
         <bodyName>base_link</bodyName>
@@ -37,6 +36,6 @@
         <gaussianNoise>0</gaussianNoise>
         <frameName>map</frameName>
-        <xyzOffsets>0 0 0</xyzOffsets>
-        <rpyOffsets>0 0 0</rpyOffsets>
+        <xyzOffset>0 0 0</xyzOffset>
+        <rpyOffset>0 0 0</rpyOffset>
       </plugin>
     </gazebo>
@@ -65,23 +64,4 @@
       </sensor>
     </gazebo>
-    <!-- Wheels -->
-    <gazebo reference="wheel_left_link">
-      <mu1>1.0</mu1>
-      <mu2>1.0</mu2>
-      <kp>1000000.0</kp>
-      <kd>100.0</kd>
-      <minDepth>0.001</minDepth>
-      <maxVel>1.0</maxVel>
-      <material>Gazebo/Grey</material>
-    </gazebo>
-    <gazebo reference="wheel_right_link">
-      <mu1>1.0</mu1>
-      <mu2>1.0</mu2>
-      <kp>1000000.0</kp>
-      <kd>100.0</kd>
-      <minDepth>0.001</minDepth>
-      <maxVel>1.0</maxVel>
-      <material>Gazebo/Grey</material>
-    </gazebo>
     <!-- Cliff Publisher detector -->
     <gazebo>

File: ca_description/urdf/create_caster_wheel.xacro (robot description, xacro)
@@ -1,10 +1,9 @@
 <?xml version="1.0" ?>
 <robot xmlns:xacro="http://ros.org/wiki/xacro">
-<xacro:macro name="caster_wheel" params="name:=caster_wheel parent:=base_link *origin">
+<xacro:macro name="caster_wheel" params="name:=caster_wheel parent:=base_link radius *origin">
   <xacro:include filename="$(find ca_description)/urdf/common_properties.xacro"/>
   <xacro:property name="parent_link" value="${parent}"/>
   <xacro:property name="link_name"   value="${name}_link"/>
-  <xacro:property name="radius"      value="0.018"/>
-  <xacro:property name="mass"        value="0.018"/>
+  <xacro:property name="mass"        value="1"/>
   <!-- fixed because there's no transmission -->
   <joint name="front_castor_joint" type="fixed">
@@ -27,4 +26,10 @@
   </link>
   <gazebo reference="${link_name}">
+    <mu1>0.2</mu1>
+    <mu2>0.2</mu2>
+    <kp>1000000.0</kp>
+    <kd>100.0</kd>
+    <minDepth>0.001</minDepth>
+    <maxVel>1.0</maxVel>
     <material>Gazebo/Grey</material>
   </gazebo>

File: ca_description/urdf/create_wheel.xacro (robot description, xacro)
@@ -5,5 +5,5 @@
   <xacro:property name="parent_link" value="${parent}"/>
   <xacro:property name="link_name"   value="${name}_link"/>
-  <xacro:property name="mass"        value="0.1"/>
+  <xacro:property name="mass"        value="0.5"/>
   <joint name="${name}_joint" type="continuous">
     <xacro:insert_block name="origin"/>
@@ -25,4 +25,13 @@
     </collision>
   </link>
+  <gazebo reference="${link_name}">
+    <mu1>1.0</mu1>
+    <mu2>1.0</mu2>
+    <kp>1000000.0</kp>
+    <kd>100.0</kd>
+    <minDepth>0.001</minDepth>
+    <maxVel>1.0</maxVel>
+    <material>Gazebo/Grey</material>
+  </gazebo>
 </xacro:macro>
 </robot>

File: ca_description/urdf/sensors/omni_sensor.xacro (robot description, xacro)
@@ -1,6 +1,5 @@
 <?xml version="1.0" ?>
 <robot xmlns:xacro="http://ros.org/wiki/xacro">
-<xacro:macro name="omni_sensor" params="name:=omni_sensor parent:=base_link diameter *origin">
-  <xacro:include filename="$(find ca_description)/urdf/common_properties.xacro"/>
+<xacro:macro name="omni_sensor" params="name:=omni_sensor parent:=base_link *origin">
   <xacro:property name="parent_link" value="${parent}"/>
   <xacro:property name="link_name" value="${name}_link"/>

Commit message: Fix wheel Tf: make wheels child of base_footprint

File: ca_description/urdf/create_base.xacro (robot description, xacro)
@@ -68,8 +68,8 @@
     </xacro:omni_sensor>
     <xacro:wheel name="wheel_left" radius="${wheel_radius}" width="${wheel_width}">
-      <origin xyz="0 ${wheel_separation/2} 0" rpy="0 ${pi/2} ${pi/2}"/>
+      <origin xyz="0 ${wheel_separation/2} ${base_offset_z}" rpy="0 ${pi/2} ${pi/2}"/>
     </xacro:wheel>
     <xacro:wheel name="wheel_right" radius="${wheel_radius}" width="${wheel_width}">
-      <origin xyz="0 ${-wheel_separation/2} 0" rpy="0 ${pi/2} ${pi/2}"/>
+      <origin xyz="0 ${-wheel_separation/2} ${base_offset_z}" rpy="0 ${pi/2} ${pi/2}"/>
     </xacro:wheel>
     <xacro:property name="caster_z" value="${-caster_radius}"/>

File: ca_description/urdf/create_wheel.xacro (robot description, xacro)
@@ -1,5 +1,5 @@
 <?xml version="1.0" ?>
 <robot xmlns:xacro="http://ros.org/wiki/xacro">
-<xacro:macro name="wheel" params="name:=wheel parent:=base_link radius width *origin">
+<xacro:macro name="wheel" params="name:=wheel parent:=base_footprint radius width *origin">
   <xacro:include filename="$(find ca_description)/urdf/common_properties.xacro"/>
   <xacro:property name="parent_link" value="${parent}"/>
