Commit message: Fix inertias

File: ca_description/urdf/common_properties.xacro (robot description, xacro)
@@ -8,3 +8,57 @@
   </inertial>
 </xacro:macro>
+<xacro:macro name="inertial_cuboid" params="mass x_length y_length z_length">
+    <inertial>
+      <mass value="${mass}" />
+      <origin xyz="0 0 0" />
+      <inertia ixx="${(1/12) * mass * (y_length*y_length + z_length*z_length)}" ixy="0.0" ixz="0.0"
+               iyy="${(1/12) * mass * (x_length*x_length + z_length*z_length)}" iyz="0.0"
+               izz="${(1/12) * mass * (x_length*x_length + y_length*y_length)}" />
+    </inertial>
+  </xacro:macro>
+  <xacro:macro name="inertial_cuboid_with_pose" params="mass x_length y_length z_length *origin">
+    <inertial>
+      <xacro:insert_block name="origin"/>
+      <mass value="${mass}" />
+      <inertia ixx="${(1/12) * mass * (y_length*y_length + z_length*z_length)}" ixy="0.0" ixz="0.0"
+               iyy="${(1/12) * mass * (x_length*x_length + z_length*z_length)}" iyz="0.0"
+               izz="${(1/12) * mass * (x_length*x_length + y_length*y_length)}" />
+    </inertial>
+  </xacro:macro>
+  <xacro:macro name="inertial_cylinder" params="mass radius length">
+    <inertial>
+      <mass value="${mass}"/>
+      <origin xyz="0 0 0" />
+      <inertia ixx="${(1/12) * mass * (3*radius*radius + length*length)}" ixy="0.0" ixz="0.0"
+               iyy="${(1/12) * mass * (3*radius*radius + length*length)}" iyz="0.0"
+               izz="${(1/2) * mass * (radius*radius)}" />
+    </inertial>
+  </xacro:macro>
+  <xacro:macro name="inertial_cylinder_with_pose" params="mass radius length *origin">
+    <inertial>
+      <xacro:insert_block name="origin"/>
+      <mass value="${mass}" />
+      <inertia ixx="${(1/12) * mass * (3*radius*radius + length*length)}" ixy="0.0" ixz="0.0"
+	             iyy="${(1/12) * mass * (3*radius*radius + length*length)}" iyz="0.0"
+	             izz="${(1/2) * mass * (radius*radius)}" />
+    </inertial>
+  </xacro:macro>
+  <xacro:macro name="inertial_sphere" params="mass diameter">
+    <inertial>
+      <mass value="${mass}" />
+      <origin xyz="0 0 0" />
+      <inertia ixx="${(2/5) * mass * ( (diameter*0.5) * (diameter*0.5) )}" ixy="0.0" ixz="0.0"
+	             iyy="${(2/5) * mass * ( (diameter*0.5) * (diameter*0.5) )}" iyz="0.0"
+	             izz="${(2/5) * mass * ( (diameter*0.5) * (diameter*0.5) )}" />
+    </inertial>
+  </xacro:macro>
+  <xacro:macro name="inertial_sphere_with_pose" params="mass diameter *origin">
+    <inertial>
+      <xacro:insert_block name="origin"/>
+      <mass value="${mass}" />
+      <inertia ixx="${(2/5) * mass * ( (diameter*0.5) * (diameter*0.5) )}" ixy="0.0" ixz="0.0"
+	             iyy="${(2/5) * mass * ( (diameter*0.5) * (diameter*0.5) )}" iyz="0.0"
+	             izz="${(2/5) * mass * ( (diameter*0.5) * (diameter*0.5) )}" />
+    </inertial>
+  </xacro:macro>
 </robot>

File: ca_description/urdf/create_caster_wheel.xacro (robot description, xacro)
@@ -13,5 +13,5 @@
   <xacro:property name="radius" value="0.018"/>
   <link name="${link_name}">
-    <xacro:dummy_inertia/>
+    <xacro:inertial_sphere mass="0.05" diameter="${2*radius}"/>
     <visual>
       <origin xyz="0 0 0" rpy="${R} ${P} ${Y}" />

File: ca_description/urdf/create_wheel.xacro (robot description, xacro)
@@ -10,5 +10,7 @@
   <xacro:property name="Y" value="${pi/2}"/>
   <link name="${prefix}_wheel_link">
-    <xacro:dummy_inertia/>
+    <xacro:inertial_cylinder_with_pose mass="0.1" radius="${wheel_radius}" length="${wheel_width}">
+      <origin xyz="0 0 0" rpy="${R} ${P} ${Y}" />
+    </xacro:inertial_cylinder_with_pose>
     <visual>
       <origin xyz="0 0 0" rpy="${R} ${P} ${Y}" />
@@ -28,5 +30,5 @@
     <parent link="base_link" />
     <child link="${prefix}_wheel_link" />
-    <axis xyz="0 -1 0" />
+    <axis xyz="0 1 0" />
   </joint>
 </xacro:macro>

Commit message: Create a cliff plugin
Changed the plugin from the simulation to now publish a boolean

Addressed all the comments

Fixed the xacro name issues

Added passing the number of the robot via launch-file

Added functional cliff msg publisher

Fixed minor issues

Addressed most of the comments

Addressed the create_cliff comments

Changed the xacro fails to avoid repetition

Modified the SMACH to work with the cliff message

Modified the rosnode to use as a smartpointer

Addressed the xacro comments

Changed the cliff variables to work with a dictionary

fixup! Changed the cliff variables to work with a dictionary

File: ca_description/urdf/common_properties.xacro (robot description, xacro)
@@ -62,3 +62,4 @@
     </inertial>
   </xacro:macro>
+  <xacro:property name="cm_to_meters" value="${1/100}"/>
 </robot>

File: ca_description/urdf/create_2.xacro (robot description, xacro)
@@ -3,4 +3,5 @@
   <xacro:include filename="$(find ca_description)/urdf/create_base.xacro"/>
   <xacro:include filename="$(find ca_description)/urdf/roomblock.xacro"/>
+  <xacro:property name="robot_name" value="$(arg robot_name)"/>
   <xacro:property name="wheel_separation" value="0.235"/>
   <xacro:property name="base_diameter" value="0.3485"/>

File: ca_description/urdf/create_base_gazebo.xacro (robot description, xacro)
@@ -83,4 +83,11 @@
       <material>Gazebo/Grey</material>
     </gazebo>
+    <!-- Cliff Publisher detector -->
+    <gazebo>
+      <plugin name="cliff_msg_publisher" filename="libcliff_msg_publisher.so">
+        <updateRate>10</updateRate>
+        <robotNumber>${robot_name}</robotNumber>
+      </plugin>
+    </gazebo>
   </xacro:macro>
 </robot>

File: ca_description/urdf/sensors/cliff_sensors.xacro (robot description, xacro)
@@ -5,41 +5,25 @@
   <xacro:include filename="$(find ca_description)/urdf/sensors/cliff_sensors_gazebo.xacro"/>
   <xacro:property name="parent_link" value="base_link"/>
-  <xacro:property name="name_side_left" value="side_left"/>
-  <xacro:property name="name_side_right" value="side_right"/>
-  <xacro:property name="name_front_left" value="front_left"/>
-  <xacro:property name="name_front_right" value="front_right"/>
-  <joint name="${name_side_left}_cliff_sensor_joint" type="fixed">
-    <origin xyz="0.07 0.14 0.01" rpy="0 ${pi/2} 0" />
-    <parent link="${parent_link}" />
-    <child link="${name_side_left}_cliff_sensor_link" />
-  </joint>
-  <joint name="${name_side_right}_cliff_sensor_joint" type="fixed">
-    <origin xyz="0.07 -0.14 0.01" rpy="0 ${pi/2} 0" />
-    <parent link="${parent_link}" />
-    <child link="${name_side_right}_cliff_sensor_link" />
-  </joint>
-  <joint name="${name_front_left}_front_cliff_sensor_joint" type="fixed">
-    <origin xyz="0.15 0.04 0.01" rpy="0 ${pi/2} 0" />
-    <parent link="${parent_link}" />
-    <child link="${name_front_left}_cliff_sensor_link" />
-  </joint>
-  <joint name="${name_front_right}_cliff_sensor_joint" type="fixed">
-    <origin xyz="0.15 -0.04 0.01" rpy="0 ${pi/2} 0" />
-    <parent link="${parent_link}" />
-    <child link="${name_front_right}_cliff_sensor_link" />
-  </joint>
-  <link name="${name_side_left}_cliff_sensor_link">
-    <xacro:dummy_inertia/>
-  </link>
-  <link name="${name_side_right}_cliff_sensor_link">
-    <xacro:dummy_inertia/>
-  </link>
-  <link name="${name_front_left}_cliff_sensor_link">
-    <xacro:dummy_inertia/>
-  </link>
-  <link name="${name_front_right}_cliff_sensor_link">
-    <xacro:dummy_inertia/>
-  </link>
-  <xacro:sim_create_cliff_sensors visualize="${visualize}"/>
+  <xacro:macro name="cliff" params="name *origin">
+    <joint name="${name}_cliff_sensor_joint" type="fixed">
+      <xacro:insert_block name="origin" />
+      <parent link="${parent_link}" />
+      <child link="${name}_cliff_sensor_link" />
+    </joint>
+    <link name="${name}_cliff_sensor_link" />
+    <xacro:cliff_plugin visualize="${visualize}" name="${name}"/>
+  </xacro:macro>
+  <xacro:cliff name="side_left">
+    <origin xyz="0.07 0.14 0.01" rpy="0 ${pi/2 - 0.09} 0" />
+  </xacro:cliff>
+  <xacro:cliff name="side_right">
+    <origin xyz="0.07 -0.14 0.01" rpy="0 ${pi/2 - 0.09} 0" />
+  </xacro:cliff>
+  <xacro:cliff name="front_left">
+    <origin xyz="0.15 0.04 0.01" rpy="0 ${pi/2 - 0.09} 0" />
+  </xacro:cliff>
+  <xacro:cliff name="front_right">
+    <origin xyz="0.15 -0.04 0.01" rpy="0 ${pi/2 - 0.09} 0" />
+  </xacro:cliff>
 </xacro:macro>
 </robot>

File: ca_description/urdf/sensors/cliff_sensors_gazebo.xacro (robot description, xacro)
@@ -1,116 +1,37 @@
 <?xml version="1.0" ?>
 <robot xmlns:xacro="http://ros.org/wiki/xacro">
-<xacro:macro name="sim_create_cliff_sensors" params="visualize:=false">
+<xacro:macro name="cliff_plugin" params="visualize:=false name">
   <xacro:property name="min_range_m" value="0.01"/>
   <xacro:property name="max_range_m" value="0.04"/>
   <xacro:property name="rate_hz" value="20.0"/>
-  <gazebo reference="${name_side_left}_cliff_sensor_link">
-    <sensor type="ray" name="${name_side_left}_cliff_sensor">
-      <always_on>true</always_on>
-      <update_rate>${rate_hz}</update_rate>
-      <pose>0 0 0 0 0 0</pose>
-      <visualize>${visualize}</visualize>
-      <ray>
-        <scan>
-          <horizontal>
-            <samples>1</samples>
-            <resolution>1</resolution>
-            <min_angle>0</min_angle>
-            <max_angle>0</max_angle>
-          </horizontal>
-        </scan>
-        <range>
-          <min>${min_range_m}</min>
-          <max>${max_range_m}</max>
-          <resolution>0.1</resolution>
-        </range>
-      </ray>
-      <plugin name="gazebo_ros_${name_side_left}_cliff_sensor" filename="libgazebo_ros_laser.so">
-        <topicName>${name_side_left}_cliff_sensor/scan</topicName>
-        <frameName>${name_side_left}_cliff_sensor_link</frameName>
-      </plugin>
-    </sensor>
-  </gazebo>
-  <gazebo reference="${name_side_right}_cliff_sensor_link">
-    <sensor type="ray" name="${name_side_right}_cliff_sensor">
-      <always_on>true</always_on>
-      <update_rate>${rate_hz}</update_rate>
-      <pose>0 0 0 0 0 0</pose>
-      <visualize>${visualize}</visualize>
-      <ray>
-        <scan>
-          <horizontal>
-            <samples>1</samples>
-            <resolution>1</resolution>
-            <min_angle>0</min_angle>
-            <max_angle>0</max_angle>
-          </horizontal>
-        </scan>
-        <range>
-          <min>${min_range_m}</min>
-          <max>${max_range_m}</max>
-          <resolution>0.1</resolution>
-        </range>
-      </ray>
-      <plugin name="gazebo_ros_${name_side_right}_cliff_sensor" filename="libgazebo_ros_laser.so">
-        <topicName>${name_side_right}_cliff_sensor/scan</topicName>
-        <frameName>${name_side_right}_cliff_sensor_link</frameName>
-      </plugin>
-    </sensor>
-  </gazebo>
-  <gazebo reference="${name_front_left}_cliff_sensor_link">
-    <sensor type="ray" name="${name_front_left}_cliff_sensor">
-      <always_on>true</always_on>
-      <update_rate>${rate_hz}</update_rate>
-      <pose>0 0 0 0 0 0</pose>
-      <visualize>${visualize}</visualize>
-      <ray>
-        <scan>
-          <horizontal>
-            <samples>1</samples>
-            <resolution>1</resolution>
-            <min_angle>0</min_angle>
-            <max_angle>0</max_angle>
-          </horizontal>
-        </scan>
-        <range>
-          <min>${min_range_m}</min>
-          <max>${max_range_m}</max>
-          <resolution>0.1</resolution>
-        </range>
-      </ray>
-      <plugin name="gazebo_ros_${name_front_left}_cliff_sensor" filename="libgazebo_ros_laser.so">
-        <topicName>${name_front_left}_cliff_sensor/scan</topicName>
-        <frameName>${name_front_left}_cliff_sensor</frameName>
-      </plugin>
-    </sensor>
-  </gazebo>
-  <gazebo reference="${name_front_right}_cliff_sensor_link">
-    <sensor type="ray" name="${name_front_right}_cliff_sensor">
-      <always_on>true</always_on>
-      <update_rate>${rate_hz}</update_rate>
-      <pose>0 0 0 0 0 0</pose>
-      <visualize>${visualize}</visualize>
-      <ray>
-        <scan>
-          <horizontal>
-            <samples>1</samples>
-            <resolution>1</resolution>
-            <min_angle>0</min_angle>
-            <max_angle>0</max_angle>
-          </horizontal>
-        </scan>
-        <range>
-          <min>${min_range_m}</min>
-          <max>${max_range_m}</max>
-          <resolution>0.1</resolution>
-        </range>
-      </ray>
-      <plugin name="gazebo_ros_${name_front_right}_cliff_sensor" filename="libgazebo_ros_laser.so">
-        <topicName>${name_front_right}_cliff_sensor/scan</topicName>
-        <frameName>${name_front_right}_cliff_sensor</frameName>
-      </plugin>
-    </sensor>
-  </gazebo>
+  <xacro:property name="min_cliff_value_cm" value="3.85"/>
+    <gazebo reference="${name}_cliff_sensor_link">
+      <sensor type="ray" name="${name}_cliff_sensor">
+        <always_on>true</always_on>
+        <update_rate>${rate_hz}</update_rate>
+        <pose>0 0 0 0 0 0</pose>
+        <visualize>${visualize}</visualize>
+        <ray>
+          <scan>
+            <horizontal>
+              <samples>1</samples>
+              <resolution>1</resolution>
+              <min_angle>0</min_angle>
+              <max_angle>0</max_angle>
+            </horizontal>
+          </scan>
+          <range>
+            <min>${min_range_m}</min>
+            <max>${max_range_m}</max>
+            <resolution>0.1</resolution>
+          </range>
+        </ray>
+        <plugin name="${name}_cliff_sensor" filename="libcreate_cliff_plugin.so">
+          <topicName>${name}_cliff_sensor/raw</topicName>
+          <frameName>${name}_cliff_sensor_link</frameName>
+          <cliffValue>${min_cliff_value_cm*cm_to_meters}</cliffValue>
+        </plugin>
+      </sensor>
+    </gazebo>
 </xacro:macro>
 </robot>

Commit message: Improve dummy inertia

File: ca_description/urdf/common_properties.xacro (robot description, xacro)
@@ -1,12 +1,5 @@
 <?xml version="1.0"?>
 <robot xmlns:xacro="http://ros.org/wiki/xacro">
-<xacro:macro name="dummy_inertia">
-  <inertial>
-    <mass value="0.01" />
-    <origin xyz="0 0 0" />
-    <inertia ixx="0.001" ixy="0.0" ixz="0.0" iyy="0.001" iyz="0.0" izz="0.001" />
-  </inertial>
-</xacro:macro>
-<xacro:macro name="inertial_cuboid" params="mass x_length y_length z_length">
+  <xacro:macro name="inertial_cuboid" params="mass x_length y_length z_length">
     <inertial>
       <mass value="${mass}" />
@@ -16,4 +9,7 @@
                izz="${(1/12) * mass * (x_length*x_length + y_length*y_length)}" />
     </inertial>
+  </xacro:macro>
+  <xacro:macro name="dummy_inertia">
+    <xacro:inertial_cuboid mass="0.001" x_length="0.001" y_length="0.001" z_length="0.001"/>
   </xacro:macro>
   <xacro:macro name="inertial_cuboid_with_pose" params="mass x_length y_length z_length *origin">

Commit message: Fix cliff plugins

File: ca_description/urdf/common_properties.xacro (robot description, xacro)
@@ -58,4 +58,4 @@
     </inertial>
   </xacro:macro>
-  <xacro:property name="cm_to_meters" value="${1/100}"/>
+  <xacro:property name="cm_to_meters" value="${1./100.}"/>
 </robot>

File: ca_description/urdf/create_base.xacro (robot description, xacro)
@@ -50,14 +50,14 @@
     </xacro:wall_sensor>
     <xacro:cliff_sensor name="side_left_cliff_sensor">
-      <origin xyz="0.07 0.14 0.01" rpy="0 ${pi/2 - 0.09} 0" />
+      <origin xyz="0.07 0.14 -0.01" rpy="0 ${pi/2 - 0.09} 0"/>
     </xacro:cliff_sensor>
     <xacro:cliff_sensor name="side_right_cliff_sensor">
-      <origin xyz="0.07 -0.14 0.01" rpy="0 ${pi/2 - 0.09} 0" />
+      <origin xyz="0.07 -0.14 -0.01" rpy="0 ${pi/2 - 0.09} 0"/>
     </xacro:cliff_sensor>
     <xacro:cliff_sensor name="front_left_cliff_sensor">
-      <origin xyz="0.15 0.04 0.01" rpy="0 ${pi/2 - 0.09} 0" />
+      <origin xyz="0.15 0.04 -0.01" rpy="0 ${pi/2 - 0.09} 0"/>
     </xacro:cliff_sensor>
     <xacro:cliff_sensor name="front_right_cliff_sensor">
-      <origin xyz="0.15 -0.04 0.01" rpy="0 ${pi/2 - 0.09} 0" />
+      <origin xyz="0.15 -0.04 -0.01" rpy="0 ${pi/2 - 0.09} 0"/>
     </xacro:cliff_sensor>
     <xacro:imu_sensor name="imu">

File: ca_description/urdf/create_base_gazebo.xacro (robot description, xacro)
@@ -68,6 +68,7 @@
     <gazebo>
       <plugin name="cliff_msg_publisher" filename="libcliff_msg_publisher.so">
+        <frameName>base_footprint</frameName>
+        <robotNumber>${robot_name}</robotNumber>
         <updateRate>10</updateRate>
-        <robotNumber>${robot_name}</robotNumber>
       </plugin>
     </gazebo>

File: ca_description/urdf/sensors/cliff_sensors.xacro (robot description, xacro)
@@ -5,6 +5,7 @@
   <xacro:property name="parent_link"        value="${parent}"/>
   <xacro:property name="link_name"          value="${name}_link"/>
-  <xacro:property name="min_range_m"        value="0.01"/>
-  <xacro:property name="max_range_m"        value="0.04"/>
+  <xacro:property name="min_range_cm"       value="0.5"/>
+  <xacro:property name="max_range_cm"       value="5"/>
+  <xacro:property name="resolution_cm"      value="0.1"/>
   <xacro:property name="rate_hz"            value="20.0"/>
   <xacro:property name="min_cliff_value_cm" value="3.85"/>
@@ -16,5 +17,5 @@
   <link name="${link_name}" />
   <gazebo reference="${link_name}">
-    <sensor type="ray" name="${name}_sensor">
+    <sensor type="ray" name="${name}">
       <always_on>true</always_on>
       <update_rate>${rate_hz}</update_rate>
@@ -30,7 +31,7 @@
         </scan>
         <range>
-          <min>${min_range_m}</min>
-          <max>${max_range_m}</max>
-          <resolution>0.1</resolution>
+          <min>${min_range_cm*cm_to_meters}</min>
+          <max>${max_range_cm*cm_to_meters}</max>
+          <resolution>${resolution_cm*cm_to_meters}</resolution>
         </range>
       </ray>

Commit message: Add battery to improve drift

File: ca_description/urdf/common_properties.xacro (robot description, xacro)
@@ -58,4 +58,5 @@
     </inertial>
   </xacro:macro>
-  <xacro:property name="cm_to_meters" value="${1./100.}"/>
+  <xacro:property name="cm_to_m" value="${1./100.}"/>
+  <xacro:property name="in_to_m" value="0.0254"/>
 </robot>

File: ca_description/urdf/create_base.xacro (robot description, xacro)
@@ -3,10 +3,11 @@
   <xacro:include filename="$(find ca_description)/urdf/common_properties.xacro"/>
   <xacro:include filename="$(find ca_description)/urdf/create_base_gazebo.xacro"/>
+  <xacro:include filename="$(find ca_description)/urdf/create_battery.xacro"/>
   <xacro:include filename="$(find ca_description)/urdf/create_caster_wheel.xacro"/>
   <xacro:include filename="$(find ca_description)/urdf/create_wheel.xacro"/>
+  <xacro:include filename="$(find ca_description)/urdf/sensors/cliff_sensors.xacro"/>
   <xacro:include filename="$(find ca_description)/urdf/sensors/imu_sensor.xacro"/>
+  <xacro:include filename="$(find ca_description)/urdf/sensors/omni_sensor.xacro"/>
   <xacro:include filename="$(find ca_description)/urdf/sensors/wall_sensor.xacro"/>
-  <xacro:include filename="$(find ca_description)/urdf/sensors/cliff_sensors.xacro"/>
-  <xacro:include filename="$(find ca_description)/urdf/sensors/omni_sensor.xacro"/>
   <xacro:macro name="create_base" params="wheel_separation wheel_radius wheel_width base_diameter *mesh">
     <xacro:property name="caster_radius" value="0.018"/>
@@ -77,4 +78,7 @@
       <origin xyz="0.13 0 ${caster_z}"/>
     </xacro:caster_wheel>
+    <xacro:battery>
+      <origin xyz="0.085 0 ${base_height}"/>
+    </xacro:battery>
     <!-- Simulation sensors -->
     <xacro:sim_create_base/>

File: ca_description/urdf/create_caster_wheel.xacro (robot description, xacro)
@@ -5,5 +5,5 @@
   <xacro:property name="parent_link" value="${parent}"/>
   <xacro:property name="link_name"   value="${name}_link"/>
-  <xacro:property name="mass"        value="1"/>
+  <xacro:property name="mass"        value="0.2"/>
   <!-- fixed because there's no transmission -->
   <joint name="front_castor_joint" type="fixed">

File: ca_description/urdf/sensors/cliff_sensors.xacro (robot description, xacro)
@@ -31,7 +31,7 @@
         </scan>
         <range>
-          <min>${min_range_cm*cm_to_meters}</min>
-          <max>${max_range_cm*cm_to_meters}</max>
-          <resolution>${resolution_cm*cm_to_meters}</resolution>
+          <min>${min_range_cm*cm_to_m}</min>
+          <max>${max_range_cm*cm_to_m}</max>
+          <resolution>${resolution_cm*cm_to_m}</resolution>
         </range>
       </ray>
@@ -39,5 +39,5 @@
         <topicName>${name}/raw</topicName>
         <frameName>${link_name}</frameName>
-        <cliffValue>${min_cliff_value_cm*cm_to_meters}</cliffValue>
+        <cliffValue>${min_cliff_value_cm*cm_to_m}</cliffValue>
       </plugin>
     </sensor>
