Commit message: Use base_link for collision instead of base_footprint

File: ca_description/urdf/create_base_gazebo.xacro (robot description, xacro)
@@ -41,5 +41,5 @@
     </gazebo>
     <!-- Bumpers -->
-    <gazebo reference="base_footprint">
+    <gazebo reference="base_link">
       <gravity>true</gravity>
       <self_collide>false</self_collide>
@@ -49,9 +49,9 @@
         <update_rate>50</update_rate>
         <contact>
-          <collision>base_footprint_collision</collision>
+          <collision>base_link_collision</collision>
         </contact>
         <!-- Plugin -->
         <plugin name="create_bumper_controller" filename="libcreate_bumper_plugin.so">
-          <frameName>base_footprint</frameName>
+          <frameName>base_link</frameName>
           <bumperTopicName>bumper</bumperTopicName>
         </plugin>

Commit message: Add ca_camera package
Fix Tf for real robot

Add camera sensors for real robot

Fix permissions in Docker for USB

Automatically source workspace in Docker

Add support for depthimage_to_laserscan

Standardize launch files

Support real RPLidar A2

Add new keyboard teleop

Move map_server to navigate.launch

Make real robot work with Cartographer

File: ca_description/urdf/create_base_gazebo.xacro (robot description, xacro)
@@ -31,5 +31,5 @@
         <alwaysOn>true</alwaysOn>
         <updateRate>60</updateRate>
-        <robotNamespace>create1_tf</robotNamespace>
+        <robotNamespace>${robot_name}</robotNamespace>
         <bodyName>base_link</bodyName>
         <topicName>gts</topicName>

File: ca_description/urdf/sensors/lasers/rplidar.xacro (robot description, xacro)
@@ -13,5 +13,5 @@
 <xacro:property name="min_angle_rad" value="${-pi}"/>
 <xacro:property name="max_angle_rad" value="${pi}"/>
-<xacro:property name="topic_name"    value="laser/scan"/>
+<xacro:property name="topic_name"    value="${name}/scan"/>
 <joint name="${name}_joint" type="fixed">
   <origin xyz="${laser_origin}"/>

Commit message: Localization improvements with robot_localization

File: ca_description/urdf/create_base_gazebo.xacro (robot description, xacro)
@@ -21,10 +21,10 @@
           <robotBaseFrame>base_footprint</robotBaseFrame>
           <publishWheelTF>true</publishWheelTF>
-          <publishOdomTF>true</publishOdomTF>
+          <publishOdomTF>false</publishOdomTF>
           <publishWheelJointState>true</publishWheelJointState>
-          <odometrySource>world</odometrySource>
+          <odometrySource>encoder</odometrySource>
           <publishTf>true</publishTf>
         </plugin>
-    </xacro:unless>
+      </xacro:unless>
       <!-- ros_control plugin -->
       <xacro:if value="$(arg enable_ros_control)">

File: ca_description/urdf/stacks/turtlebot.xacro (robot description, xacro)
@@ -11,5 +11,5 @@
   <joint name="pole_${name}_joint" type="fixed">
     <xacro:insert_block name="origin"/>
-    <parent link="${parent}"/>
+    <parent link="${parent}" rpy="0 0 ${pi}"/>
     <child link="${link_name}"/>
   </joint>

Commit message: Set wheel odometry rate to 30 Hz

File: ca_description/urdf/create_base_gazebo.xacro (robot description, xacro)
@@ -2,7 +2,4 @@
 <robot xmlns:xacro="http://ros.org/wiki/xacro">
   <xacro:macro name="sim_create_base">
-    <xacro:property name="diffdrive_update_rate" value="40"/>
-    <xacro:property name="wheel_torque" value="0.5"/>
-    <xacro:property name="wheel_accel" value="0.5"/>
     <gazebo>
       <!-- Diff-drive controller -->
@@ -10,11 +7,11 @@
         <alwaysOn>true</alwaysOn>
         <rosDebugLevel>na</rosDebugLevel>
-        <updateRate>${diffdrive_update_rate}</updateRate>
+        <updateRate>30</updateRate>
         <leftJoint>wheel_left_joint</leftJoint>
         <rightJoint>wheel_right_joint</rightJoint>
         <wheelSeparation>${wheel_separation}</wheelSeparation>
         <wheelDiameter>${wheel_radius * 2}</wheelDiameter>
-        <wheelTorque>${wheel_torque}</wheelTorque>
-        <wheelAcceleration>${wheel_accel}</wheelAcceleration>
+        <wheelTorque>0.5</wheelTorque>
+        <wheelAcceleration>0.5</wheelAcceleration>
         <commandTopic>cmd_vel</commandTopic>
         <odometryTopic>odom</odometryTopic>
