Commit message: Clean up URDFs

File: ca_description/urdf/create_2.xacro (robot description, xacro)
@@ -16,4 +16,6 @@
   </xacro:create_base>
   <!-- Roomblock -->
-  <xacro:roomblock parent="base_link" visualize="$(arg visualize)"/>
+  <xacro:roomblock visualize="$(arg visualize)">
+    <origin xyz="0 0 0.07"/>
+  </xacro:roomblock>
 </robot>

File: ca_description/urdf/create_base.xacro (robot description, xacro)
@@ -45,26 +45,34 @@
       </collision>
     </link>
-    <xacro:wall_sensor visualize="${visualize}"/>
-    <xacro:cliff_sensor name="side_left" parent="base_link">
+    <xacro:wall_sensor visualize="${visualize}">
+      <origin xyz="0.09 -0.12 0.042" rpy="0 0 -1"/>
+    </xacro:wall_sensor>
+    <xacro:cliff_sensor name="side_left_cliff_sensor">
       <origin xyz="0.07 0.14 0.01" rpy="0 ${pi/2 - 0.09} 0" />
     </xacro:cliff_sensor>
-    <xacro:cliff_sensor name="side_right" parent="base_link">
+    <xacro:cliff_sensor name="side_right_cliff_sensor">
       <origin xyz="0.07 -0.14 0.01" rpy="0 ${pi/2 - 0.09} 0" />
     </xacro:cliff_sensor>
-    <xacro:cliff_sensor name="front_left" parent="base_link">
+    <xacro:cliff_sensor name="front_left_cliff_sensor">
       <origin xyz="0.15 0.04 0.01" rpy="0 ${pi/2 - 0.09} 0" />
     </xacro:cliff_sensor>
-    <xacro:cliff_sensor name="front_right" parent="base_link">
+    <xacro:cliff_sensor name="front_right_cliff_sensor">
       <origin xyz="0.15 -0.04 0.01" rpy="0 ${pi/2 - 0.09} 0" />
     </xacro:cliff_sensor>
     <xacro:imu_sensor name="imu">
-      <origin xyz="0 -0.04 0.13" rpy="0 0 0"/>
+      <origin xyz="0 -0.04 0.13"/>
     </xacro:imu_sensor>
-    <xacro:omni_sensor name="omni_sensor" diameter="0.1">
-      <origin xyz="0.145 0 ${base_link_offset_z}" rpy="0 0 0"/>
+    <xacro:omni_sensor diameter="0.1">
+      <origin xyz="0.145 0 ${base_link_offset_z}"/>
     </xacro:omni_sensor>
-    <xacro:create_wheel prefix="left" y_offset="${wheel_separation / 2}" wheel_radius="${wheel_radius}" wheel_width="${wheel_width}"/>
-    <xacro:create_wheel prefix="right" y_offset="${wheel_separation / -2}" wheel_radius="${wheel_radius}" wheel_width="${wheel_width}"/>
-    <xacro:caster_wheel/>
+    <xacro:wheel name="wheel_left" radius="${wheel_radius}" width="${wheel_width}">
+      <origin xyz="0 ${wheel_separation/2} 0.015" rpy="0 ${pi/2} ${pi/2}"/>
+    </xacro:wheel>
+    <xacro:wheel name="wheel_right" radius="${wheel_radius}" width="${wheel_width}">
+      <origin xyz="0 ${-wheel_separation/2} 0.015" rpy="0 ${pi/2} ${pi/2}"/>
+    </xacro:wheel>
+    <xacro:caster_wheel>
+      <origin xyz="0.13 0 0"/>
+    </xacro:caster_wheel>
     <!-- Simulation sensors -->
     <xacro:sim_create_base/>

File: ca_description/urdf/create_base_gazebo.xacro (robot description, xacro)
@@ -11,6 +11,6 @@
         <rosDebugLevel>na</rosDebugLevel>
         <updateRate>${diffdrive_update_rate}</updateRate>
-        <leftJoint>left_wheel_joint</leftJoint>
-        <rightJoint>right_wheel_joint</rightJoint>
+        <leftJoint>wheel_left_joint</leftJoint>
+        <rightJoint>wheel_right_joint</rightJoint>
         <wheelSeparation>${wheel_separation}</wheelSeparation>
         <wheelDiameter>${wheel_radius * 2}</wheelDiameter>
@@ -65,5 +65,5 @@
     </gazebo>
     <!-- Wheels -->
-    <gazebo reference="left_wheel_link">
+    <gazebo reference="wheel_left_link">
       <mu1>1.0</mu1>
       <mu2>1.0</mu2>
@@ -74,5 +74,5 @@
       <material>Gazebo/Grey</material>
     </gazebo>
-    <gazebo reference="right_wheel_link">
+    <gazebo reference="wheel_right_link">
       <mu1>1.0</mu1>
       <mu2>1.0</mu2>

File: ca_description/urdf/create_caster_wheel.xacro (robot description, xacro)
@@ -1,19 +1,19 @@
 <?xml version="1.0" ?>
 <robot xmlns:xacro="http://ros.org/wiki/xacro">
-<xacro:macro name="caster_wheel">
+<xacro:macro name="caster_wheel" params="name:=caster_wheel parent:=base_link *origin">
   <xacro:include filename="$(find ca_description)/urdf/common_properties.xacro"/>
-  <xacro:property name="link_name" value="caster_wheel_link"/>
-  <xacro:property name="parent_link" value="base_link"/>
-  <xacro:property name="x" value="0.13"/>
-  <xacro:property name="y" value="0"/>
-  <xacro:property name="z" value="0"/>
-  <xacro:property name="R" value="0"/>
-  <xacro:property name="P" value="${pi/2}"/>
-  <xacro:property name="Y" value="${pi/2}"/>
-  <xacro:property name="radius" value="0.018"/>
+  <xacro:property name="parent_link" value="${parent}"/>
+  <xacro:property name="link_name"   value="${name}_link"/>
+  <xacro:property name="radius"      value="0.018"/>
+  <xacro:property name="mass"        value="0.018"/>
+  <!-- fixed because there's no transmission -->
+  <joint name="front_castor_joint" type="fixed">
+    <xacro:insert_block name="origin"/>
+    <parent link="${parent_link}" />
+    <child link="${link_name}" />
+  </joint>
   <link name="${link_name}">
-    <xacro:inertial_sphere mass="0.05" diameter="${2*radius}"/>
+    <xacro:inertial_sphere mass="${mass}" diameter="${2*radius}"/>
     <visual>
-      <origin xyz="0 0 0" rpy="${R} ${P} ${Y}" />
       <geometry>
         <sphere radius="${radius}" />
@@ -21,5 +21,4 @@
     </visual>
     <collision>
-      <origin xyz="0 0 0" rpy="${R} ${P} ${Y}" />
       <geometry>
         <sphere radius="${radius}" />
@@ -27,11 +26,4 @@
     </collision>
   </link>
-  <!-- fixed because there's no transmission -->
-  <joint name="front_castor_joint" type="fixed">
-    <origin xyz="${x} ${y} ${z}" rpy="0 0 0" />
-    <parent link="${parent_link}" />
-    <child link="${link_name}" />
-    <axis xyz="0 1 0" />
-  </joint>
   <gazebo reference="${link_name}">
     <material>Gazebo/Grey</material>

File: ca_description/urdf/create_wheel.xacro (robot description, xacro)
@@ -1,35 +1,28 @@
 <?xml version="1.0" ?>
 <robot xmlns:xacro="http://ros.org/wiki/xacro">
-<xacro:macro name="create_wheel" params="prefix y_offset wheel_radius wheel_width">
+<xacro:macro name="wheel" params="name:=wheel parent:=base_link radius width *origin">
   <xacro:include filename="$(find ca_description)/urdf/common_properties.xacro"/>
-  <xacro:property name="x" value="0"/>
-  <xacro:property name="y" value="${y_offset}"/>
-  <xacro:property name="z" value="0.015"/>
-  <xacro:property name="R" value="0"/>
-  <xacro:property name="P" value="${pi/2}"/>
-  <xacro:property name="Y" value="${pi/2}"/>
-  <link name="${prefix}_wheel_link">
-    <xacro:inertial_cylinder_with_pose mass="0.1" radius="${wheel_radius}" length="${wheel_width}">
-      <origin xyz="0 0 0" rpy="${R} ${P} ${Y}" />
-    </xacro:inertial_cylinder_with_pose>
+  <xacro:property name="parent_link" value="${parent}"/>
+  <xacro:property name="link_name"   value="${name}_link"/>
+  <xacro:property name="mass"        value="0.1"/>
+  <joint name="${name}_joint" type="continuous">
+    <xacro:insert_block name="origin"/>
+    <parent link="${parent_link}" />
+    <child link="${link_name}" />
+    <axis xyz="0 1 0" />
+  </joint>
+  <link name="${link_name}">
+    <xacro:inertial_cylinder mass="${mass}" radius="${radius}" length="${width}"/>
     <visual>
-      <origin xyz="0 0 0" rpy="${R} ${P} ${Y}" />
       <geometry>
-        <cylinder radius="${wheel_radius}" length="${wheel_width}" />
+        <cylinder radius="${radius}" length="${width}" />
       </geometry>
     </visual>
     <collision>
-      <origin xyz="0 0 0" rpy="${R} ${P} ${Y}" />
       <geometry>
-        <cylinder radius="${wheel_radius}" length="${wheel_width}" />
+        <cylinder radius="${radius}" length="${width}" />
       </geometry>
     </collision>
   </link>
- <joint name="${prefix}_wheel_joint" type="continuous">
-    <origin xyz="${x} ${y} ${z}" rpy="0 0 0" />
-    <parent link="base_link" />
-    <child link="${prefix}_wheel_link" />
-    <axis xyz="0 1 0" />
-  </joint>
 </xacro:macro>
 </robot>

File: ca_description/urdf/roomblock.xacro (robot description, xacro)
@@ -5,21 +5,19 @@
 <robot xmlns:xacro="http://ros.org/wiki/xacro">
   <xacro:include filename="$(find ca_description)/urdf/common_properties.xacro"/>
-  <xacro:include filename="$(find ca_description)/urdf/roomblock_gazebo.xacro"/>
   <xacro:include filename="$(find ca_description)/urdf/sensors/camera_sensor.xacro"/>
   <xacro:include filename="$(find ca_description)/urdf/sensors/lasers/rplidar.xacro"/>
-  <xacro:macro name="roomblock" params="parent visualize:=false">
-    <xacro:property name="z" value="0.07"/>
-    <xacro:property name="roomblock_link" value="block_link"/>
-    <xacro:property name="parent_link" value="${parent}"/>
-    <xacro:property name="roomblock_mass" value="0.1"/>
-    <xacro:property name="roomblock_size_x" value="0.1"/>
-    <xacro:property name="roomblock_size_y" value="0.1"/>
-    <xacro:property name="roomblock_size_z" value="0.07"/>
+  <xacro:macro name="roomblock" params="name:=roomblock parent:=base_link visualize:=false *origin">
+    <xacro:property name="parent_link"    value="${parent}"/>
+    <xacro:property name="link_name"      value="${name}_link"/>
+    <xacro:property name="mass"           value="0.1"/>
+    <xacro:property name="size_x"         value="0.1"/>
+    <xacro:property name="size_y"         value="0.1"/>
+    <xacro:property name="size_z"         value="0.07"/>
     <joint name="block_joint" type="fixed">
-      <origin xyz="0 0 ${z}"/>
+      <xacro:insert_block name="origin"/>
       <parent link="${parent_link}"/>
-      <child link="${roomblock_link}" />
+      <child link="${link_name}" />
     </joint>
-    <link name="${roomblock_link}">
+    <link name="${link_name}">
       <visual>
         <geometry>
@@ -28,18 +26,19 @@
         <material name="Grey" />
       </visual>
-      <xacro:inertial_cuboid_with_pose mass="${roomblock_mass}"
-                                       x_length="${roomblock_size_x}"
-                                       y_length="${roomblock_size_y}"
-                                       z_length="${roomblock_size_z}">
-        <origin xyz="0 0 ${roomblock_size_z/2}"/>
+      <xacro:inertial_cuboid_with_pose mass="${mass}"
+                                       x_length="${size_x}"
+                                       y_length="${size_y}"
+                                       z_length="${size_z}">
+        <origin xyz="0 0 ${size_z/2}"/>
       </xacro:inertial_cuboid_with_pose>
     </link>
-    <xacro:rplidar parent="${roomblock_link}" visualize="${visualize}">
+    <gazebo reference="${link_name}">
+      <material>Gazebo/Grey</material>
+    </gazebo>
+    <xacro:rplidar parent="${link_name}" visualize="${visualize}">
       <origin xyz="0 0 0.1"/>
     </xacro:rplidar>
-    <!-- TODO: REMOVE VISUALIZE USING ARG OR XACRO:ARG -->
     <!-- TODO (eborghi): ADD CAMERA CAD? REMOVE CAMERA/USE ANOTHER ONE? -->
-    <!-- <xacro:camera_sensor parent="${roomblock_link}"/> -->
-    <xacro:roomblock_gazebo link_name="${roomblock_link}"/>
+    <xacro:camera_sensor name="raspicam" parent="${link_name}"/>
   </xacro:macro>
 </robot>

File: ca_description/urdf/sensors/camera_sensor.xacro (robot description, xacro)
@@ -2,10 +2,8 @@
 <robot xmlns:xacro="http://ros.org/wiki/xacro">
 <xacro:include filename="$(find ca_description)/urdf/sensors/camera_generic.xacro"/>
-<xacro:macro name="camera_sensor" params="parent">
-  <xacro:property name="x" value="0.04"/>
-  <xacro:property name="y" value="0.0"/>
-  <xacro:property name="z" value="0.06"/>
-  <xacro:generic_camera name="raspicam" parent="${parent}">
-    <origin xyz="${x} ${y} ${z}" rpy="0 0 0"/>
+<xacro:macro name="camera_sensor" params="name:=camera parent:=base_link">
+  <xacro:property name="parent_link" value="${parent}"/>
+  <xacro:generic_camera name="${name}" parent="${parent_link}">
+    <origin xyz="0.04 0 0.06"/>
   </xacro:generic_camera>
 </xacro:macro>

File: ca_description/urdf/sensors/cliff_sensors.xacro (robot description, xacro)
@@ -1,15 +1,45 @@
 <?xml version="1.0" ?>
 <robot xmlns:xacro="http://ros.org/wiki/xacro">
-<xacro:macro name="cliff_sensor" params="name parent *origin visualize:=false">
+<xacro:macro name="cliff_sensor" params="name:=cliff_sensor parent:=base_link *origin visualize:=false">
   <xacro:include filename="$(find ca_description)/urdf/common_properties.xacro"/>
-  <xacro:include filename="$(find ca_description)/urdf/sensors/cliff_sensors_gazebo.xacro"/>
-  <xacro:property name="parent_link" value="${parent}"/>
-  <joint name="${name}_cliff_sensor_joint" type="fixed">
+  <xacro:property name="parent_link"        value="${parent}"/>
+  <xacro:property name="link_name"          value="${name}_link"/>
+  <xacro:property name="min_range_m"        value="0.01"/>
+  <xacro:property name="max_range_m"        value="0.04"/>
+  <xacro:property name="rate_hz"            value="20.0"/>
+  <xacro:property name="min_cliff_value_cm" value="3.85"/>
+  <joint name="${name}_joint" type="fixed">
     <xacro:insert_block name="origin" />
     <parent link="${parent_link}" />
-    <child link="${name}_cliff_sensor_link" />
+    <child link="${link_name}" />
   </joint>
-  <link name="${name}_cliff_sensor_link" />
-  <xacro:cliff_plugin visualize="${visualize}" name="${name}"/>
+  <link name="${link_name}" />
+  <gazebo reference="${link_name}">
+    <sensor type="ray" name="${name}_sensor">
+      <always_on>true</always_on>
+      <update_rate>${rate_hz}</update_rate>
+      <visualize>${visualize}</visualize>
+      <ray>
+        <scan>
+          <horizontal>
+            <samples>1</samples>
+            <resolution>1</resolution>
+            <min_angle>0</min_angle>
+            <max_angle>0</max_angle>
+          </horizontal>
+        </scan>
+        <range>
+          <min>${min_range_m}</min>
+          <max>${max_range_m}</max>
+          <resolution>0.1</resolution>
+        </range>
+      </ray>
+      <plugin name="gazebo_ros_${name}" filename="libcreate_cliff_plugin.so">
+        <topicName>${name}/raw</topicName>
+        <frameName>${link_name}</frameName>
+        <cliffValue>${min_cliff_value_cm*cm_to_meters}</cliffValue>
+      </plugin>
+    </sensor>
+  </gazebo>
 </xacro:macro>
 </robot>

File: ca_description/urdf/sensors/imu_sensor.xacro (robot description, xacro)
@@ -1,8 +1,7 @@
 <?xml version="1.0" ?>
 <robot xmlns:xacro="http://ros.org/wiki/xacro">
-<xacro:macro name="imu_sensor" params="name *origin">
+<xacro:macro name="imu_sensor" params="name:=imu_sensor parent:=base_link *origin">
   <xacro:include filename="$(find ca_description)/urdf/common_properties.xacro"/>
-  <xacro:include filename="$(find ca_description)/urdf/sensors/imu_sensor_gazebo.xacro"/>
-  <xacro:property name="parent_link" value="base_link"/>
+  <xacro:property name="parent_link" value="${parent}"/>
   <xacro:property name="link_name" value="${name}_link"/>
   <joint name="${name}_joint" type="fixed">
@@ -11,8 +10,17 @@
     <child link="${link_name}" />
   </joint>
-  <link name="${link_name}">
-    <xacro:dummy_inertia/>
-  </link>
-  <xacro:imu_sensor_gazebo name="${name}" link_name="${link_name}"/>
+  <link name="${link_name}"/>
+  <gazebo reference="${link_name}">
+    <plugin name="${name}" filename="libgazebo_ros_imu.so">
+      <alwaysOn>true</alwaysOn>
+      <updateRate>30</updateRate>
+      <bodyName>${link_name}</bodyName>
+      <topicName>${name}/data</topicName>
+      <serviceName>${name}/is_calibrated</serviceName>
+      <gaussianNoise>${0.0017*0.0017}</gaussianNoise>
+      <xyzOffsets>0 0 0</xyzOffsets>
+      <rpyOffsets>0 0 0</rpyOffsets>
+    </plugin>
+  </gazebo>
 </xacro:macro>
 </robot>

File: ca_description/urdf/sensors/lasers/rplidar.xacro (robot description, xacro)
@@ -1,11 +1,19 @@
 <?xml version="1.0"?>
 <robot xmlns:xacro="http://ros.org/wiki/xacro">
-<xacro:include filename="$(find ca_description)/urdf/sensors/lasers/rplidar_gazebo.xacro"/>
-<xacro:macro name="rplidar" params="parent visualize:=false *origin">
-  <xacro:property name="link_name"  value="rplidar_link"/>
-  <xacro:property name="laser_name" value="laser_link"/>
-  <joint name="rplidar_joint" type="fixed">
+<xacro:macro name="rplidar" params="name:=rplidar parent:=base_link visualize:=false *origin">
+  <xacro:property name="parent_link"              value="${parent}"/>
+  <xacro:property name="link_name"                value="${name}_link"/>
+  <xacro:property name="laser_link"               value="laser_link"/>
+  <xacro:property name="rplidar_a2_rate_hz"       value="10"/>
+  <xacro:property name="rplidar_a2_min_range_m"   value="0.15"/>
+  <xacro:property name="rplidar_a2_max_range_m"   value="12.0"/>
+  <xacro:property name="rplidar_a2_samples"       value="720"/>
+  <xacro:property name="rplidar_a2_resolution_mm" value="0.5"/>
+  <xacro:property name="rplidar_a2_min_angle_rad" value="${-pi}"/>
+  <xacro:property name="rplidar_a2_max_angle_rad" value="${pi}"/>
+  <xacro:property name="topic_name"               value="laser/scan"/>
+  <joint name="${name}_joint" type="fixed">
     <xacro:insert_block name="origin"/>
-    <parent link="${parent}"/>
+    <parent link="${parent_link}"/>
     <child link="${link_name}"/>
   </joint>
@@ -20,19 +28,11 @@
     <origin xyz="0 0 0.0308"/>
     <parent link="${link_name}"/>
-    <child link="${laser_name}"/>
+    <child link="${laser_link}"/>
   </joint>
-  <link name="${laser_name}"/>
-  <!-- <xacro:property name="rplidar_a2_rate_hz" value="10"/>
-  <xacro:property name="rplidar_a2_min_range_m" value="0.15"/>
-  <xacro:property name="rplidar_a2_max_range_m" value="12.0"/>
-  <xacro:property name="rplidar_a2_samples" value="720"/>
-  <xacro:property name="rplidar_a2_resolution_mm" value="0.5"/>
-  <xacro:property name="rplidar_a2_min_angle_rad" value="${-pi}"/>
-  <xacro:property name="rplidar_a2_max_angle_rad" value="${pi}"/>
-  <xacro:property name="topic_name" value="laser/scan"/>
-  <gazebo reference="${laser_name}">
+  <link name="${laser_link}"/>
+  <gazebo reference="${laser_link}">
     <material>Gazebo/FlatBlack</material>
-    <sensor type="ray" name="rplidar_sensor">
-      <visualize>true</visualize>
+    <sensor type="ray" name="${name}_sensor">
+      <visualize>${visualize}</visualize>
       <update_rate>${rplidar_a2_rate_hz}</update_rate>
       <ray>
@@ -56,12 +56,10 @@
         </noise>
       </ray>
-      <plugin name="gazebo_ros_rplidar_sensor" filename="libgazebo_ros_laser.so">
+      <plugin name="gazebo_ros_${name}" filename="libgazebo_ros_laser.so">
         <topicName>${topic_name}</topicName>
-        <frameName>${laser_name}</frameName>
+        <frameName>${laser_link}</frameName>
       </plugin>
     </sensor>
-  </gazebo> -->
-  <!-- Gazebo plugin -->
-  <xacro:rplidar_gazebo link_name="${laser_name}" visualize="${visualize}"/>
+  </gazebo>
 </xacro:macro>
 </robot>

File: ca_description/urdf/sensors/omni_sensor.xacro (robot description, xacro)
@@ -1,8 +1,7 @@
 <?xml version="1.0" ?>
 <robot xmlns:xacro="http://ros.org/wiki/xacro">
-<xacro:macro name="omni_sensor" params="name diameter *origin">
+<xacro:macro name="omni_sensor" params="name:=omni_sensor parent:=base_link diameter *origin">
   <xacro:include filename="$(find ca_description)/urdf/common_properties.xacro"/>
-  <xacro:include filename="$(find ca_description)/urdf/sensors/omni_sensor_gazebo.xacro"/>
-  <xacro:property name="parent_link" value="base_link"/>
+  <xacro:property name="parent_link" value="${parent}"/>
   <xacro:property name="link_name" value="${name}_link"/>
   <joint name="${name}_joint" type="fixed">
@@ -11,8 +10,7 @@
     <child link="${link_name}" />
   </joint>
-  <link name="${link_name}">
-    <xacro:dummy_inertia/>
-  </link>
-  <xacro:omni_sensor_gazebo name="${name}" diameter="${diameter}"/>
+  <link name="${link_name}"/>
+  <gazebo>
+  </gazebo>
 </xacro:macro>
 </robot>

File: ca_description/urdf/sensors/wall_sensor.xacro (robot description, xacro)
@@ -1,23 +1,44 @@
 <?xml version="1.0" ?>
 <robot xmlns:xacro="http://ros.org/wiki/xacro">
-<xacro:macro name="wall_sensor" params="visualize:=false">
+<xacro:macro name="wall_sensor" params="name:=wall_sensor parent:=base_link visualize:=false *origin">
   <xacro:include filename="$(find ca_description)/urdf/common_properties.xacro"/>
-  <xacro:include filename="$(find ca_description)/urdf/sensors/wall_sensor_gazebo.xacro"/>
-  <xacro:property name="x" value="0.09"/>
-  <xacro:property name="y" value="-0.120"/>
-  <xacro:property name="z" value="0.042"/>
-  <xacro:property name="R" value="0"/>
-  <xacro:property name="P" value="0"/>
-  <xacro:property name="Y" value="-1.0"/>
-  <xacro:property name="parent_link" value="base_link"/>
+  <xacro:property name="parent_link" value="${parent}"/>
+  <xacro:property name="link_name"   value="${name}_link"/>
+  <xacro:property name="topic_name"  value="/wall_sensor/scan"/>
+  <xacro:property name="rate_hz"     value="20.0"/>
+  <xacro:property name="min_range_m" value="0.0160"/>
+  <xacro:property name="max_range_m" value="0.04"/>
   <joint name="base_wall_sensor_joint" type="fixed">
-    <origin xyz="${x} ${y} ${z}" rpy="${R} ${P} ${Y}" />
+    <xacro:insert_block name="origin"/>
     <parent link="${parent_link}" />
-    <child link="wall_sensor_link" />
+    <child link="${link_name}" />
   </joint>
-  <link name="wall_sensor_link">
-    <xacro:dummy_inertia/>
-  </link>
-  <xacro:sim_create_wall_sensor visualize="${visualize}"/>
+  <link name="${link_name}"/>
+  <gazebo reference="${link_name}">
+    <sensor type="ray" name="${name}_sensor">
+      <always_on>true</always_on>
+      <update_rate>${rate_hz}</update_rate>
+      <visualize>${visualize}</visualize>
+      <ray>
+        <scan>
+          <horizontal>
+            <samples>1</samples>
+            <resolution>1</resolution>
+            <min_angle>0</min_angle>
+            <max_angle>0</max_angle>
+          </horizontal>
+        </scan>
+        <range>
+          <min>${min_range_m}</min>
+          <max>${max_range_m}</max>
+          <resolution>0.1</resolution>
+        </range>
+      </ray>
+      <plugin name="gazebo_ros_${name}" filename="libgazebo_ros_laser.so">
+        <topicName>${topic_name}</topicName>
+        <frameName>${link_name}</frameName>
+      </plugin>
+    </sensor>
+  </gazebo>
 </xacro:macro>
 </robot>
