Commit message: More updates

File: ca_description/urdf/create_2.xacro (robot description, xacro)
@@ -15,7 +15,10 @@
     <mesh filename="package://ca_description/meshes/create_2.dae" />
   </xacro:create_base>
+  <xacro:property name="stack" value="$(arg stack)"/>
   <!-- Roomblock -->
-  <xacro:roomblock visualize="$(arg visualize)">
-    <origin xyz="0 0 0.07"/>
-  </xacro:roomblock>
+  <xacro:if value="${stack == 'roomblock'}">
+    <xacro:roomblock visualize="$(arg visualize)">
+      <origin xyz="0 0 0.07"/>
+    </xacro:roomblock>
+  </xacro:if>
 </robot>

File: ca_description/urdf/roomblock.xacro (robot description, xacro)
@@ -7,4 +7,5 @@
   <xacro:include filename="$(find ca_description)/urdf/sensors/camera_sensor.xacro"/>
   <xacro:include filename="$(find ca_description)/urdf/sensors/lasers/rplidar.xacro"/>
+  <xacro:include filename="$(find ca_description)/urdf/sensors/lasers/astra.xacro"/>
   <xacro:macro name="roomblock" params="name:=roomblock parent:=base_link visualize:=false *origin">
     <xacro:property name="parent_link"    value="${parent}"/>
@@ -36,7 +37,16 @@
       <material>Gazebo/Grey</material>
     </gazebo>
-    <xacro:rplidar parent="${link_name}" visualize="${visualize}">
-      <origin xyz="0 0 0.1"/>
-    </xacro:rplidar>
+    <xacro:property name="laser" default="$(arg laser)"/>
+    <xacro:if value="${laser == 'rplidar'}">
+      <xacro:rplidar_a2 parent="${link_name}" visualize="${visualize}">
+        <origin xyz="0 0 0.1"/>
+      </xacro:rplidar_a2>
+    </xacro:if>
+    <xacro:if value="${laser == 'astra'}">
+      <xacro:orbec_astra>
+      <!-- TODO: USE ORIGIN TAG -->
+        <origin xyz="0 0 0.1"/>
+      </xacro:orbec_astra>
+    </xacro:if>
     <!-- TODO (eborghi): ADD CAMERA CAD? REMOVE CAMERA/USE ANOTHER ONE? -->
     <xacro:camera_sensor name="raspicam" parent="${link_name}"/>

File: ca_description/urdf/sensors/imu_sensor.xacro (robot description, xacro)
@@ -11,5 +11,5 @@
   </joint>
   <link name="${link_name}"/>
-  <gazebo reference="${link_name}">
+  <gazebo>
     <plugin name="${name}" filename="libgazebo_ros_imu.so">
       <alwaysOn>true</alwaysOn>

File: ca_description/urdf/sensors/lasers/astra.xacro (robot description, xacro)
@@ -1,40 +1,37 @@
-<!-- Orbbec Astra RGBD Camera -->
-  <joint name="astra_joint" type="fixed">
-    <axis xyz="0 0 0" />
-    <origin xyz="-0.03 0 0.18" rpy="0 0 0"/>
-    <parent link="base_link"/>
-    <child link="camera_link"/>
+<?xml version="1.0"?>
+<robot xmlns:xacro="http://ros.org/wiki/xacro">
+<xacro:include filename="$(find ca_description)/urdf/sensors/lasers/sim_3d_sensor.xacro"/>
+<xacro:macro name="orbec_astra" params="name:=astra parent:=base_link visualize:=false *origin">
+  <xacro:property name="parent_link" value="${parent}"/>
+  <xacro:property name="link_name"   value="${name}_link"/>
+  <xacro:property name="link_rgb"    value="${name}_rgb_frame"/>
+  <xacro:property name="link_depth"  value="${name}_depth_frame"/>
+  <!-- Orbbec Astra RGBD Camera -->
+  <joint name="${name}_joint" type="fixed">
+    <origin xyz="-0.03 0 0.18"/>
+    <parent link="${parent_link}"/>
+    <child link="${link_name}"/>
   </joint>
-  <link name="camera_link">
-    <collision>
-      <origin xyz="0.02 0 0" rpy="0 0 0"/>
-      <geometry>0
-        <box size="0.001 0.001 0.001"/>
-      </geometry>
-    </collision>
+  <link name="${link_name}">
     <visual>
-      <origin xyz="-0.01 0 -0.03" rpy="1.5707 0 1.5707"/>
+      <origin xyz="-0.01 0 -0.03" rpy="${pi/2} 0 ${pi/2}"/>
       <geometry>
-        <mesh filename="package://rosbot_description/meshes/astra.dae" scale="0.001 0.001 0.001" />
+        <mesh filename="package://ca_description/meshes/astra.dae" scale="0.001 0.001 0.001" />
       </geometry>
     </visual>
-    <inertial>
-      <mass value="1e-5" />
-      <origin xyz="0 0 0" rpy="0 0 0"/>
-      <inertia ixx="0" ixy="0" ixz="0" iyy="0" iyz="0" izz="0" />
-    </inertial>
   </link>
-  <joint name="camera_optical_joint" type="fixed">
+  <joint name="${name}_optical_joint" type="fixed">
     <origin xyz="0 0 0" rpy="${-pi/2} 0 ${-pi/2}"/>
-    <parent link="camera_link"/>
-    <child link="camera_rgb_frame"/>
+    <parent link="${link_name}"/>
+    <child link="${link_rgb}"/>
   </joint>
-  <link name="camera_rgb_frame">
-  </link>
-  <joint name="camera_depth_joint" type="fixed">
+  <link name="${link_rgb}"/>
+  <joint name="${name}_depth_joint" type="fixed">
     <origin xyz="0 0 0" rpy="${-pi/2} 0 ${-pi/2}"/>
-    <parent link="camera_link"/>
-    <child link="camera_depth_frame"/>
+    <parent link="${link_name}"/>
+    <child link="${link_depth}"/>
   </joint>
-  <link name="camera_depth_frame">
-  </link>
+  <link name="${link_depth}"/>
+  <xacro:sim_3d_sensor name="${name}" visualize="true"/>
+</xacro:macro>
+</robot>

File: ca_description/urdf/sensors/lasers/rplidar.xacro (robot description, xacro)
@@ -1,5 +1,5 @@
 <?xml version="1.0"?>
 <robot xmlns:xacro="http://ros.org/wiki/xacro">
-<xacro:macro name="rplidar" params="name:=rplidar parent:=base_link visualize:=false *origin">
+<xacro:macro name="rplidar_a2" params="name:=rplidar parent:=base_link visualize:=false *origin">
   <xacro:property name="parent_link"              value="${parent}"/>
   <xacro:property name="link_name"                value="${name}_link"/>

Commit message: Fixed a lot of things

File: ca_description/urdf/create_2.xacro (robot description, xacro)
@@ -2,5 +2,4 @@
 <robot name="create_2" xmlns:xacro="http://ros.org/wiki/xacro">
   <xacro:include filename="$(find ca_description)/urdf/create_base.xacro"/>
-  <xacro:include filename="$(find ca_description)/urdf/roomblock.xacro"/>
   <xacro:property name="robot_name" value="$(arg robot_name)"/>
   <xacro:property name="wheel_separation" value="0.235"/>
@@ -15,4 +14,8 @@
     <mesh filename="package://ca_description/meshes/create_2.dae" />
   </xacro:create_base>
+  <!-- ##### STACKS ##### -->
+  <!-- TODO: Implement this in a dictionary (along with include file) -->
+  <xacro:include filename="$(find ca_description)/urdf/stacks/roomblock.xacro"/>
+  <xacro:include filename="$(find ca_description)/urdf/stacks/turtlebot.xacro"/>
   <xacro:property name="stack" value="$(arg stack)"/>
   <!-- Roomblock -->
@@ -22,3 +25,9 @@
     </xacro:roomblock>
   </xacro:if>
+  <!-- Turtlebot stack -->
+  <xacro:if value="${stack == 'turtlebot'}">
+    <xacro:turtlebot_stack>
+      <origin xyz="0 0 0"/>
+    </xacro:turtlebot_stack>
+  </xacro:if>
 </robot>

File: ca_description/urdf/create_base.xacro (robot description, xacro)
@@ -1,12 +1,13 @@
 <?xml version="1.0" ?>
 <robot xmlns:xacro="http://ros.org/wiki/xacro">
+  <xacro:include filename="$(find ca_description)/urdf/common_properties.xacro"/>
+  <xacro:include filename="$(find ca_description)/urdf/create_base_gazebo.xacro"/>
+  <xacro:include filename="$(find ca_description)/urdf/create_caster_wheel.xacro"/>
+  <xacro:include filename="$(find ca_description)/urdf/create_wheel.xacro"/>
+  <xacro:include filename="$(find ca_description)/urdf/sensors/imu_sensor.xacro"/>
+  <xacro:include filename="$(find ca_description)/urdf/sensors/wall_sensor.xacro"/>
+  <xacro:include filename="$(find ca_description)/urdf/sensors/cliff_sensors.xacro"/>
+  <xacro:include filename="$(find ca_description)/urdf/sensors/omni_sensor.xacro"/>
   <xacro:macro name="create_base" params="wheel_separation wheel_radius wheel_width base_diameter *mesh visualize:=false">
-    <xacro:include filename="$(find ca_description)/urdf/create_base_gazebo.xacro"/>
-    <xacro:include filename="$(find ca_description)/urdf/create_caster_wheel.xacro"/>
-    <xacro:include filename="$(find ca_description)/urdf/create_wheel.xacro"/>
-    <xacro:include filename="$(find ca_description)/urdf/sensors/imu_sensor.xacro"/>
-    <xacro:include filename="$(find ca_description)/urdf/sensors/wall_sensor.xacro"/>
-    <xacro:include filename="$(find ca_description)/urdf/sensors/cliff_sensors.xacro"/>
-    <xacro:include filename="$(find ca_description)/urdf/sensors/omni_sensor.xacro"/>
     <xacro:property name="base_link_offset_z" value="0.0308"/>
     <xacro:property name="base_offset_z" value="0.017"/>

File: ca_description/urdf/sensors/lasers/astra.xacro (robot description, xacro)
@@ -2,12 +2,14 @@
 <robot xmlns:xacro="http://ros.org/wiki/xacro">
 <xacro:include filename="$(find ca_description)/urdf/sensors/lasers/sim_3d_sensor.xacro"/>
-<xacro:macro name="orbec_astra" params="name:=astra parent:=base_link visualize:=false *origin">
-  <xacro:property name="parent_link" value="${parent}"/>
-  <xacro:property name="link_name"   value="${name}_link"/>
-  <xacro:property name="link_rgb"    value="${name}_rgb_frame"/>
-  <xacro:property name="link_depth"  value="${name}_depth_frame"/>
-  <!-- Orbbec Astra RGBD Camera -->
+<!-- Orbbec Astra RGBD Camera -->
+<xacro:macro name="orbbec_astra" params="name:=astra parent:=base_link *origin">
+  <xacro:property name="parent_link"    value="${parent}"/>
+  <xacro:property name="link_name"      value="${name}_link"/>
+  <xacro:property name="link_rgb"       value="${name}_rgb_frame"/>
+  <xacro:property name="link_depth"     value="${name}_depth_frame"/>
+  <xacro:property name="link_optical"   value="${name}_depth_optical_frame"/>
+  <xacro:property name="optical_offset" value="0.01"/>
   <joint name="${name}_joint" type="fixed">
-    <origin xyz="-0.03 0 0.18"/>
+    <xacro:insert_block name="origin"/>
     <parent link="${parent_link}"/>
     <child link="${link_name}"/>
@@ -17,10 +19,10 @@
       <origin xyz="-0.01 0 -0.03" rpy="${pi/2} 0 ${pi/2}"/>
       <geometry>
-        <mesh filename="package://ca_description/meshes/astra.dae" scale="0.001 0.001 0.001" />
+        <mesh filename="package://ca_description/meshes/astra.dae"/>
       </geometry>
     </visual>
   </link>
   <joint name="${name}_optical_joint" type="fixed">
-    <origin xyz="0 0 0" rpy="${-pi/2} 0 ${-pi/2}"/>
+    <origin xyz="0 ${optical_offset} 0" rpy="${-pi/2} 0 ${-pi/2}"/>
     <parent link="${link_name}"/>
     <child link="${link_rgb}"/>
@@ -28,10 +30,16 @@
   <link name="${link_rgb}"/>
   <joint name="${name}_depth_joint" type="fixed">
-    <origin xyz="0 0 0" rpy="${-pi/2} 0 ${-pi/2}"/>
+    <origin rpy="${-pi/2} 0 ${-pi/2}"/>
     <parent link="${link_name}"/>
     <child link="${link_depth}"/>
   </joint>
   <link name="${link_depth}"/>
-  <xacro:sim_3d_sensor name="${name}" visualize="true"/>
+   <joint name="${name}_depth_optical_joint" type="fixed">
+    <origin rpy="${-pi/2} 0 ${-pi/2}"/>
+    <parent link="${link_depth}"/>
+    <child link="${link_optical}"/>
+  </joint>
+  <link name="${link_optical}"/>
+  <xacro:sim_3d_sensor name="${name}" color="Gazebo/FlatBlack"/>
 </xacro:macro>
 </robot>

File: ca_description/urdf/sensors/lasers/kinect.xacro (robot description, xacro)
@@ -1,6 +1,4 @@
 <?xml version="1.0"?>
 <robot name="sensor_kinect" xmlns:xacro="http://ros.org/wiki/xacro">
-  <xacro:include filename="$(find turtlebot_description)/urdf/turtlebot_gazebo.urdf.xacro"/>
-  <xacro:include filename="$(find turtlebot_description)/urdf/turtlebot_properties.urdf.xacro"/>
   <xacro:property name="kinect_cam_py" value="-0.0125"/>
   <!-- Parameterised in part by the values in turtlebot_properties.urdf.xacro -->
@@ -27,5 +25,5 @@
        <origin xyz="0 0 0" rpy="0 0 ${M_PI/2}"/>
         <geometry>
-         <mesh filename="package://turtlebot_description/meshes/sensors/kinect.dae"/>
+         <mesh filename="package://ca_description/meshes/sensors/kinect.dae"/>
         </geometry>
       </visual>

File: ca_description/urdf/sensors/lasers/r200.xacro (robot description, xacro)
@@ -1,6 +1,4 @@
 <?xml version="1.0"?>
 <robot name="sensor_r200" xmlns:xacro="http://ros.org/wiki/xacro">
-  <xacro:include filename="$(find turtlebot_description)/urdf/turtlebot_gazebo.urdf.xacro"/>
-  <xacro:include filename="$(find turtlebot_description)/urdf/turtlebot_properties.urdf.xacro"/>
   <!-- Mount and camera parameters -->
   <xacro:property name="pole_px" value="-0.103" />
@@ -35,5 +33,5 @@
        <origin xyz="${-r200_bracket_end_width/2} ${r200_bracket_end_offset_py} ${r200_bracket_end_offset_pz}" rpy="0 0 ${-M_PI/2}"/>
         <geometry>
-         <mesh filename="package://turtlebot_description/meshes/sensors/r200_bracket_end.stl" scale="0.001 0.001 0.001"/>
+         <mesh filename="package://ca_description/meshes/sensors/r200_bracket_end.stl" scale="0.001 0.001 0.001"/>
         </geometry>
         <xacro:insert_block name="material_dark_grey" />
@@ -50,5 +48,5 @@
        <origin xyz="0 0 0" rpy="0 0 ${M_PI/2}"/>
         <geometry>
-         <mesh filename="package://turtlebot_description/meshes/sensors/r200_bracket.stl" scale="0.001 0.001 0.001"/>
+         <mesh filename="package://ca_description/meshes/sensors/r200_bracket.stl" scale="0.001 0.001 0.001"/>
         </geometry>
         <xacro:insert_block name="material_dark_grey" />
@@ -65,5 +63,5 @@
        <origin xyz="${r200_bracket_end_width/2} 0 ${-r200_bracket_end_offset_pz}" rpy="0 0 ${M_PI/2}"/>
         <geometry>
-         <mesh filename="package://turtlebot_description/meshes/sensors/r200_bracket_end.stl" scale="0.001 0.001 0.001"/>
+         <mesh filename="package://ca_description/meshes/sensors/r200_bracket_end.stl" scale="0.001 0.001 0.001"/>
         </geometry>
         <xacro:insert_block name="material_dark_grey" />
@@ -80,5 +78,5 @@
        <origin xyz="0 0 0" rpy="${M_PI/2} 0 ${M_PI/2}"/>
         <geometry>
-         <mesh filename="package://turtlebot_description/meshes/sensors/r200.dae" />
+         <mesh filename="package://ca_description/meshes/sensors/r200.dae" />
         </geometry>
       </visual>

File: ca_description/urdf/sensors/lasers/sim_3d_sensor.xacro (robot description, xacro)
@@ -2,9 +2,9 @@
 <robot xmlns:xacro="http://ros.org/wiki/xacro">
   <!-- Microsoft Kinect / ASUS Xtion PRO Live for simulation -->
-  <xacro:macro name="sim_3d_sensor" params="name visualize:=false">
+  <xacro:macro name="sim_3d_sensor" params="name color">
     <gazebo reference="${name}_link">
+      <material>${color}</material>
       <sensor type="depth" name="${name}">
         <always_on>true</always_on>
-        <visualize>${visualize}</visualize>
         <update_rate>20.0</update_rate>
         <camera>
@@ -20,6 +20,6 @@
           </clip>
         </camera>
-        <plugin name="kinect_camera_controller" filename="libgazebo_ros_openni_kinect.so">
-          <cameraName>camera</cameraName>
+        <plugin name="kinect_${name}_controller" filename="libgazebo_ros_openni_kinect.so">
+          <cameraName>${name}</cameraName>
           <alwaysOn>true</alwaysOn>
           <updateRate>10</updateRate>
@@ -29,5 +29,5 @@
           <cameraInfoTopicName>rgb/camera_info</cameraInfoTopicName>
           <depthImageCameraInfoTopicName>depth/camera_info</depthImageCameraInfoTopicName>
-          <frameName>camera_depth_optical_frame</frameName>
+          <frameName>${name}_depth_optical_frame</frameName>
           <baseline>0.1</baseline>
           <distortion_k1>0.0</distortion_k1>

File: ca_description/urdf/sensors/lasers/xtion_pro.xacro (robot description, xacro)
@@ -1,6 +1,6 @@
 <?xml version="1.0"?>
 <robot name="sensor_xtion_pro" xmlns:xacro="http://ros.org/wiki/xacro">
-  <xacro:include filename="$(find turtlebot_description)/urdf/turtlebot_gazebo.urdf.xacro"/>
-  <xacro:include filename="$(find turtlebot_description)/urdf/turtlebot_properties.urdf.xacro"/>
+  <xacro:include filename="$(find ca_description)/urdf/turtlebot_gazebo.urdf.xacro"/>
+  <xacro:include filename="$(find ca_description)/urdf/turtlebot_properties.urdf.xacro"/>
   <!-- Xacro properties -->
   <xacro:property name="xtion_pro_depth_rel_rgb_py" value="0.0270" />
@@ -32,5 +32,5 @@
         <origin xyz="-0.015 0.0035 0.004" rpy="0 0 0"/>
         <geometry>
-          <mesh filename="package://turtlebot_description/meshes/sensors/xtion_pro_camera.dae"/>
+          <mesh filename="package://ca_description/meshes/sensors/xtion_pro_camera.dae"/>
         </geometry>
       </visual>
@@ -73,5 +73,5 @@
         <origin xyz="0 0 0" rpy="${-M_PI/2} 0 0"/>
         <geometry>
-          <mesh filename="package://turtlebot_description/meshes/sensors/xtion_pro_stack.dae"/>
+          <mesh filename="package://ca_description/meshes/sensors/xtion_pro_stack.dae"/>
         </geometry>
       </visual>

File: ca_description/urdf/stacks/roomblock.xacro (robot description, xacro)
@@ -6,13 +6,11 @@
   <xacro:include filename="$(find ca_description)/urdf/common_properties.xacro"/>
   <xacro:include filename="$(find ca_description)/urdf/sensors/camera_sensor.xacro"/>
-  <xacro:include filename="$(find ca_description)/urdf/sensors/lasers/rplidar.xacro"/>
-  <xacro:include filename="$(find ca_description)/urdf/sensors/lasers/astra.xacro"/>
   <xacro:macro name="roomblock" params="name:=roomblock parent:=base_link visualize:=false *origin">
-    <xacro:property name="parent_link"    value="${parent}"/>
-    <xacro:property name="link_name"      value="${name}_link"/>
-    <xacro:property name="mass"           value="0.1"/>
-    <xacro:property name="size_x"         value="0.1"/>
-    <xacro:property name="size_y"         value="0.1"/>
-    <xacro:property name="size_z"         value="0.07"/>
+    <xacro:property name="parent_link" value="${parent}"/>
+    <xacro:property name="link_name"   value="${name}_link"/>
+    <xacro:property name="mass"        value="0.1"/>
+    <xacro:property name="size_x"      value="0.1"/>
+    <xacro:property name="size_y"      value="0.1"/>
+    <xacro:property name="size_z"      value="0.07"/>
     <joint name="block_joint" type="fixed">
       <xacro:insert_block name="origin"/>
@@ -37,5 +35,21 @@
       <material>Gazebo/Grey</material>
     </gazebo>
+    <xacro:include filename="$(find ca_description)/urdf/sensors/lasers/astra.xacro"/>
+    <!-- <xacro:include filename="$(find ca_description)/urdf/sensors/lasers/kinect.xacro"/> -->
+    <xacro:include filename="$(find ca_description)/urdf/sensors/lasers/realsense.xacro"/>
+    <xacro:include filename="$(find ca_description)/urdf/sensors/lasers/rplidar.xacro"/>
+    <!-- <xacro:include filename="$(find ca_description)/urdf/sensors/lasers/xtion_pro.xacro"/> -->
     <xacro:property name="laser" default="$(arg laser)"/>
+    <!-- TODO: Implement this in a dictionary (along with include file) -->
+    <xacro:if value="${laser == 'astra'}">
+      <xacro:orbbec_astra>
+        <origin xyz="0 0 0.2"/>
+      </xacro:orbbec_astra>
+    </xacro:if>
+    <xacro:if value="${laser == 'kinect'}">
+      <!-- <xacro:kinect>
+        <origin xyz="0 0 0.15"/>
+      </xacro:kinect> -->
+    </xacro:if>
     <xacro:if value="${laser == 'rplidar'}">
       <xacro:rplidar_a2 parent="${link_name}" visualize="${visualize}">
@@ -43,9 +57,13 @@
       </xacro:rplidar_a2>
     </xacro:if>
-    <xacro:if value="${laser == 'astra'}">
-      <xacro:orbec_astra>
-      <!-- TODO: USE ORIGIN TAG -->
-        <origin xyz="0 0 0.1"/>
-      </xacro:orbec_astra>
+    <xacro:if value="${laser == 'r200'}">
+      <xacro:realsense_r200>
+        <origin xyz="0 0 0.15"/>
+      </xacro:realsense_r200>
+    </xacro:if>
+    <xacro:if value="${laser == 'xtion_pro'}">
+      <!-- <xacro:asus_xtion_pro>
+        <origin xyz="0 0 0.15"/>
+      </xacro:asus_xtion_pro> -->
     </xacro:if>
     <!-- TODO (eborghi): ADD CAMERA CAD? REMOVE CAMERA/USE ANOTHER ONE? -->
