Commit message: Improve calling of stacks

File: ca_description/urdf/create_2.xacro (robot description, xacro)
@@ -14,20 +14,9 @@
     <mesh filename="package://ca_description/meshes/create_2.dae" />
   </xacro:create_base>
-  <!-- ##### STACKS ##### -->
-  <!-- TODO: Implement this in a dictionary (along with include file) -->
-  <xacro:include filename="$(find ca_description)/urdf/stacks/roomblock.xacro"/>
-  <xacro:include filename="$(find ca_description)/urdf/stacks/turtlebot.xacro"/>
+  <!-- Stacks -->
   <xacro:property name="stack" value="$(arg stack)"/>
-  <!-- Roomblock -->
-  <xacro:if value="${stack == 'roomblock'}">
-    <xacro:roomblock visualize="$(arg visualize)">
-      <origin xyz="0 0 0.07"/>
-    </xacro:roomblock>
-  </xacro:if>
-  <!-- Turtlebot stack -->
-  <xacro:if value="${stack == 'turtlebot'}">
-    <xacro:turtlebot_stack>
-      <origin xyz="0 0 0"/>
-    </xacro:turtlebot_stack>
-  </xacro:if>
+  <xacro:property name="stack_yaml" value="$(find ca_description)/urdf/stacks/poses.yaml"/>
+  <xacro:property name="stack_dict" value="${load_yaml(stack_yaml)}"/>
+  <xacro:property name="stack_origin" value="${stack_dict[stack]}"/>
+  <xacro:include filename="$(find ca_description)/urdf/stacks/${stack}.xacro"/>
 </robot>

File: ca_description/urdf/stacks/roomblock.xacro (robot description, xacro)
@@ -4,43 +4,43 @@
 -->
 <robot xmlns:xacro="http://ros.org/wiki/xacro">
-  <xacro:include filename="$(find ca_description)/urdf/common_properties.xacro"/>
-  <xacro:include filename="$(find ca_description)/urdf/sensors/camera_sensor.xacro"/>
-  <xacro:macro name="roomblock" params="name:=roomblock parent:=base_link visualize:=false *origin">
-    <xacro:property name="parent_link" value="${parent}"/>
-    <xacro:property name="link_name"   value="${name}_link"/>
-    <xacro:property name="mass"        value="0.1"/>
-    <xacro:property name="size_x"      value="0.1"/>
-    <xacro:property name="size_y"      value="0.1"/>
-    <xacro:property name="size_z"      value="0.07"/>
-    <joint name="block_joint" type="fixed">
-      <xacro:insert_block name="origin"/>
-      <parent link="${parent_link}"/>
-      <child link="${link_name}" />
-    </joint>
-    <link name="${link_name}">
-      <visual>
-        <geometry>
-  	       <mesh filename="package://ca_description/meshes/block.dae"/>
-        </geometry>
-        <material name="Grey" />
-      </visual>
-      <xacro:inertial_cuboid_with_pose mass="${mass}"
-                                       x_length="${size_x}"
-                                       y_length="${size_y}"
-                                       z_length="${size_z}">
-        <origin xyz="0 0 ${size_z/2}"/>
-      </xacro:inertial_cuboid_with_pose>
-    </link>
-    <gazebo reference="${link_name}">
-      <material>Gazebo/Grey</material>
-    </gazebo>
-    <!-- Laser -->
-    <xacro:property name="laser" default="$(arg laser)"/>
-    <xacro:property name="laser_yaml" value="$(find ca_description)/urdf/sensors/lasers/poses.yaml"/>
-    <xacro:property name="laser_dict" value="${load_yaml(laser_yaml)}"/>
-    <xacro:property name="laser_origin" value="${laser_dict['roomblock'][laser]}"/>
-    <xacro:include filename="$(find ca_description)/urdf/sensors/lasers/${laser}.xacro"/>
-    <!-- TODO (eborghi): ADD CAMERA CAD? REMOVE CAMERA/USE ANOTHER ONE? -->
-    <xacro:camera_sensor name="raspicam" parent="${link_name}"/>
-  </xacro:macro>
+<xacro:include filename="$(find ca_description)/urdf/common_properties.xacro"/>
+<xacro:include filename="$(find ca_description)/urdf/sensors/camera_sensor.xacro"/>
+<xacro:property name="name" value="roomblock"/>
+<xacro:property name="parent" value="base_link"/>
+<xacro:property name="parent_link" value="${parent}"/>
+<xacro:property name="link_name"   value="${name}_link"/>
+<xacro:property name="mass"        value="0.1"/>
+<xacro:property name="size_x"      value="0.1"/>
+<xacro:property name="size_y"      value="0.1"/>
+<xacro:property name="size_z"      value="0.07"/>
+<joint name="block_joint" type="fixed">
+  <origin xyz="${stack_origin}"/>
+  <parent link="${parent_link}"/>
+  <child link="${link_name}" />
+</joint>
+<link name="${link_name}">
+  <visual>
+    <geometry>
+        <mesh filename="package://ca_description/meshes/block.dae"/>
+    </geometry>
+    <material name="Grey" />
+  </visual>
+  <xacro:inertial_cuboid_with_pose mass="${mass}"
+                                    x_length="${size_x}"
+                                    y_length="${size_y}"
+                                    z_length="${size_z}">
+    <origin xyz="0 0 ${size_z/2}"/>
+  </xacro:inertial_cuboid_with_pose>
+</link>
+<gazebo reference="${link_name}">
+  <material>Gazebo/Grey</material>
+</gazebo>
+<!-- Laser -->
+<xacro:property name="laser" default="$(arg laser)"/>
+<xacro:property name="laser_yaml" value="$(find ca_description)/urdf/sensors/lasers/poses.yaml"/>
+<xacro:property name="laser_dict" value="${load_yaml(laser_yaml)}"/>
+<xacro:property name="laser_origin" value="${laser_dict['roomblock'][laser]}"/>
+<xacro:include filename="$(find ca_description)/urdf/sensors/lasers/${laser}.xacro"/>
+<!-- TODO (eborghi): ADD CAMERA CAD? REMOVE CAMERA/USE ANOTHER ONE? -->
+<xacro:camera_sensor name="raspicam" parent="${link_name}"/>
 </robot>

File: ca_description/urdf/stacks/turtlebot.xacro (robot description, xacro)
@@ -5,88 +5,103 @@
  -->
 <robot xmlns:xacro="http://ros.org/wiki/xacro">
-  <!-- Pole macro -->
-  <xacro:macro name="stack_pole" params="name parent:=base_link *origin *mesh">
-    <xacro:property name="link_name" value="pole_${name}_link"/>
-    <joint name="pole_${name}_joint" type="fixed">
-      <xacro:insert_block name="origin"/>
-      <parent link="${parent}"/>
-      <child link="${link_name}"/>
-    </joint>
-    <link name="${link_name}">
-      <visual>
-        <geometry>
-          <xacro:insert_block name="mesh"/>
-        </geometry>
-      </visual>
-    </link>
-  </xacro:macro>
-  <!--
-    Stack macro - all the components relative transforms are made with respect
-    to the parent link (usually base_link). They could be made relative to each
-    other, but there is no necessary reason to do so.
-  -->
-  <xacro:macro name="turtlebot_stack" params="name:=turtlebot_stack parent:=base_link *origin">
-    <xacro:stack_pole name="short_0">
-      <origin xyz="0.0381 0.1 0.093"/>
-      <mesh filename="package://ca_description/meshes/turtlebot_stack/short_pole.dae"/>
-    </xacro:stack_pole>
-    <xacro:stack_pole name="short_1">
-      <origin xyz="0.0381 -0.1 0.093"/>
-      <mesh filename="package://ca_description/meshes/turtlebot_stack/short_pole.dae"/>
-    </xacro:stack_pole>
-    <xacro:stack_pole name="short_2">
-      <origin xyz="-0.0381 0.1 0.093"/>
-      <mesh filename="package://ca_description/meshes/turtlebot_stack/short_pole.dae"/>
-    </xacro:stack_pole>
-    <xacro:stack_pole name="short_3">
-      <origin xyz="-0.0381 -0.1 0.093"/>
-      <mesh filename="package://ca_description/meshes/turtlebot_stack/short_pole.dae"/>
-    </xacro:stack_pole>
-    <joint name="plate_bottom_joint" type="fixed">
-      <origin xyz="-0.01364 0 0.125"/>
-      <parent link="${parent}"/>
-      <child link="plate_bottom_link"/>
-    </joint>
-    <link name="plate_bottom_link">
-      <visual>
-        <geometry>
-          <mesh filename="package://ca_description/meshes/turtlebot_stack/bottom_plate.dae" scale="0.5 0.7 1"/>
-        </geometry>
-      </visual>
-    </link>
-    <xacro:stack_pole name="large_0">
-      <origin xyz="0.1 0.098 0.18"/>
-      <mesh filename="package://ca_description/meshes/turtlebot_stack/large_pole.dae"/>
-    </xacro:stack_pole>
-    <xacro:stack_pole name="large_1">
-      <origin xyz="0.1 -0.098 0.18"/>
-      <mesh filename="package://ca_description/meshes/turtlebot_stack/large_pole.dae"/>
-    </xacro:stack_pole>
-    <xacro:stack_pole name="large_2">
-      <origin xyz="-0.1 0.098 0.18"/>
-      <mesh filename="package://ca_description/meshes/turtlebot_stack/large_pole.dae"/>
-    </xacro:stack_pole>
-    <xacro:stack_pole name="large_3">
-      <origin xyz="-0.1 -0.098 0.18"/>
-      <mesh filename="package://ca_description/meshes/turtlebot_stack/large_pole.dae"/>
-    </xacro:stack_pole>
-    <joint name="plate_upper_joint" type="fixed">
-      <origin xyz="-0.01364 0 0.2"/>
-      <parent link="${parent}"/>
-      <child link="plate_upper_link"/>
-    </joint>
-    <link name="plate_upper_link">
-      <visual>
-        <geometry>
-          <mesh filename="package://ca_description/meshes/turtlebot_stack/upper_plate.dae"/>
-        </geometry>
-      </visual>
-    </link>
-    <!-- Laser -->
-    <xacro:property name="laser" default="$(arg laser)"/>
-    <xacro:property name="laser_yaml" value="$(find ca_description)/urdf/sensors/lasers/poses.yaml"/>
-    <xacro:property name="laser_dict" value="${load_yaml(laser_yaml)}"/>
-    <xacro:property name="laser_origin" value="${laser_dict['turtlebot'][laser]}"/>
-    <xacro:include filename="$(find ca_description)/urdf/sensors/lasers/${laser}.xacro"/>
-  </xacro:macro>
+<!-- Pole macro -->
+<xacro:macro name="stack_pole" params="name parent:=base_link *origin *mesh">
+  <xacro:property name="link_name" value="pole_${name}_link"/>
+  <joint name="pole_${name}_joint" type="fixed">
+    <xacro:insert_block name="origin"/>
+    <parent link="${parent}"/>
+    <child link="${link_name}"/>
+  </joint>
+  <link name="${link_name}">
+    <visual>
+      <geometry>
+        <xacro:insert_block name="mesh"/>
+      </geometry>
+    </visual>
+  </link>
+</xacro:macro>
+<!-- turtlebot_stack -->
+<xacro:property name="name" value="turtlebot_stack"/>
+<xacro:property name="parent" value="base_link"/>
+<xacro:property name="base_link" value="${name}_base_link"/>
+<joint name="${name}_base_joint" type="fixed">
+  <origin xyz="${stack_origin}"/>
+  <parent link="${parent}"/>
+  <child link="${base_link}"/>
+</joint>
+<link name="${base_link}"/>
+<xacro:stack_pole name="short_0" parent="${base_link}">
+  <origin xyz="0.03 0.08 0"/>
+  <mesh filename="package://ca_description/meshes/turtlebot_stack/short_pole.dae"/>
+</xacro:stack_pole>
+<xacro:stack_pole name="short_1" parent="${base_link}">
+  <origin xyz="0.03 -0.08 0"/>
+  <mesh filename="package://ca_description/meshes/turtlebot_stack/short_pole.dae"/>
+</xacro:stack_pole>
+<xacro:stack_pole name="short_2" parent="${base_link}">
+  <origin xyz="-0.06 0.08 0"/>
+  <mesh filename="package://ca_description/meshes/turtlebot_stack/short_pole.dae"/>
+</xacro:stack_pole>
+<xacro:stack_pole name="short_3" parent="${base_link}">
+  <origin xyz="-0.06 -0.08 0"/>
+  <mesh filename="package://ca_description/meshes/turtlebot_stack/short_pole.dae"/>
+</xacro:stack_pole>
+<joint name="plate_bottom_joint" type="fixed">
+  <origin xyz="-0.025 0 0.032"/>
+  <parent link="${base_link}"/>
+  <child link="plate_bottom_link"/>
+</joint>
+<link name="plate_bottom_link">
+  <visual>
+    <geometry>
+      <mesh filename="package://ca_description/meshes/turtlebot_stack/bottom_plate.dae" scale="0.5 0.7 1"/>
+    </geometry>
+  </visual>
+</link>
+<xacro:stack_pole name="large_0" parent="${base_link}">
+  <origin xyz="0.03 0.08 0.077"/>
+  <mesh filename="package://ca_description/meshes/turtlebot_stack/large_pole.dae"/>
+</xacro:stack_pole>
+<xacro:stack_pole name="large_1" parent="${base_link}">
+  <origin xyz="0.03 -0.08 0.077"/>
+  <mesh filename="package://ca_description/meshes/turtlebot_stack/large_pole.dae"/>
+</xacro:stack_pole>
+<xacro:stack_pole name="large_2" parent="${base_link}">
+  <origin xyz="-0.06 0.08 0.077"/>
+  <mesh filename="package://ca_description/meshes/turtlebot_stack/large_pole.dae"/>
+</xacro:stack_pole>
+<xacro:stack_pole name="large_3" parent="${base_link}">
+  <origin xyz="-0.06 -0.08 0.077"/>
+  <mesh filename="package://ca_description/meshes/turtlebot_stack/large_pole.dae"/>
+</xacro:stack_pole>
+<joint name="plate_upper_joint" type="fixed">
+  <origin xyz="-0.01364 0 0.117"/>
+  <parent link="${base_link}"/>
+  <child link="plate_upper_link"/>
+</joint>
+<link name="plate_upper_link">
+  <visual>
+    <geometry>
+      <mesh filename="package://ca_description/meshes/turtlebot_stack/upper_plate.dae"/>
+    </geometry>
+  </visual>
+</link>
+<joint name="nvidia_jetson_nano_joint" type="fixed">
+  <origin xyz="0 0 0.117"/>
+  <parent link="${base_link}"/>
+  <child link="nvidia_jetson_nano_link"/>
+</joint>
+<link name="nvidia_jetson_nano_link">
+  <visual>
+    <geometry>
+      <mesh filename="package://ca_description/meshes/nvidia_jetson_nano.dae"/>
+    </geometry>
+  </visual>
+</link>
+<!-- Laser -->
+<xacro:property name="laser" default="$(arg laser)"/>
+<xacro:property name="laser_yaml" value="$(find ca_description)/urdf/sensors/lasers/poses.yaml"/>
+<xacro:property name="laser_dict" value="${load_yaml(laser_yaml)}"/>
+<xacro:property name="laser_origin" value="${laser_dict['turtlebot'][laser]}"/>
+<xacro:include filename="$(find ca_description)/urdf/sensors/lasers/${laser}.xacro"/>
 </robot>

Commit message: Improve visualize argument

File: ca_description/urdf/create_2.xacro (robot description, xacro)
@@ -10,6 +10,5 @@
                      base_diameter="${base_diameter}"
                      wheel_width="${wheel_width}"
-                     wheel_radius="${wheel_radius}"
-                     visualize="$(arg visualize)">
+                     wheel_radius="${wheel_radius}">
     <mesh filename="package://ca_description/meshes/create_2.dae" />
   </xacro:create_base>

File: ca_description/urdf/create_base.xacro (robot description, xacro)
@@ -9,9 +9,10 @@
   <xacro:include filename="$(find ca_description)/urdf/sensors/cliff_sensors.xacro"/>
   <xacro:include filename="$(find ca_description)/urdf/sensors/omni_sensor.xacro"/>
-  <xacro:macro name="create_base" params="wheel_separation wheel_radius wheel_width base_diameter *mesh visualize:=false">
+  <xacro:macro name="create_base" params="wheel_separation wheel_radius wheel_width base_diameter *mesh">
     <xacro:property name="base_link_offset_z" value="0.0308"/>
     <xacro:property name="base_offset_z" value="0.017"/>
     <xacro:property name="base_height" value="0.0611632"/>
     <xacro:property name="base_mass" value="2"/>
+    <xacro:arg name="visualize" default="false"/>
     <!-- The root link base_footprint has an inertia specified in the URDF,
          but KDL does not support a root link with an inertia.
@@ -46,5 +47,5 @@
       </collision>
     </link>
-    <xacro:wall_sensor visualize="${visualize}">
+    <xacro:wall_sensor>
       <origin xyz="0.09 -0.12 0.042" rpy="0 0 -1"/>
     </xacro:wall_sensor>

File: ca_description/urdf/sensors/cliff_sensors.xacro (robot description, xacro)
@@ -1,5 +1,5 @@
 <?xml version="1.0" ?>
 <robot xmlns:xacro="http://ros.org/wiki/xacro">
-<xacro:macro name="cliff_sensor" params="name:=cliff_sensor parent:=base_link *origin visualize:=false">
+<xacro:macro name="cliff_sensor" params="name:=cliff_sensor parent:=base_link *origin">
   <xacro:include filename="$(find ca_description)/urdf/common_properties.xacro"/>
   <xacro:property name="parent_link"        value="${parent}"/>
@@ -19,5 +19,5 @@
       <always_on>true</always_on>
       <update_rate>${rate_hz}</update_rate>
-      <visualize>${visualize}</visualize>
+      <visualize>$(arg visualize)</visualize>
       <ray>
         <scan>

File: ca_description/urdf/sensors/wall_sensor.xacro (robot description, xacro)
@@ -1,5 +1,5 @@
 <?xml version="1.0" ?>
 <robot xmlns:xacro="http://ros.org/wiki/xacro">
-<xacro:macro name="wall_sensor" params="name:=wall_sensor parent:=base_link visualize:=false *origin">
+<xacro:macro name="wall_sensor" params="name:=wall_sensor parent:=base_link *origin">
   <xacro:include filename="$(find ca_description)/urdf/common_properties.xacro"/>
   <xacro:property name="parent_link" value="${parent}"/>
@@ -19,5 +19,5 @@
       <always_on>true</always_on>
       <update_rate>${rate_hz}</update_rate>
-      <visualize>${visualize}</visualize>
+      <visualize>$(arg visualize)</visualize>
       <ray>
         <scan>

Commit message: Fix bumper plugin

File: ca_description/urdf/create_2.xacro (robot description, xacro)
@@ -4,5 +4,5 @@
   <xacro:property name="robot_name" value="$(arg robot_name)"/>
   <xacro:property name="wheel_separation" value="0.235"/>
-  <xacro:property name="base_diameter" value="0.3485"/>
+  <xacro:property name="base_diameter" value="0.32"/>
   <xacro:property name="wheel_width" value="0.024"/>
   <xacro:property name="wheel_radius" value="0.036"/>

File: ca_description/urdf/create_base.xacro (robot description, xacro)
@@ -22,8 +22,5 @@
     </joint>
     <xacro:property name="base_link_origin" value="0 0 ${base_offset_z - caster_radius}"/>
-  <link name="base_link">
-    <xacro:inertial_cylinder_with_pose mass="${base_mass}" radius="${base_diameter/2}" length="${base_height}">
-      <origin xyz="${base_link_origin}"/>
-      </xacro:inertial_cylinder_with_pose>
+    <link name="base_link">
       <visual>
         <origin xyz="${base_link_origin}"/>
@@ -32,8 +29,18 @@
         </geometry>
       </visual>
+    </link>
+    <joint name="bumper_joint" type="continuous">
+      <parent link="base_link"/>
+      <child link="bumper_link"/>
+      <axis xyz="0 0 1"/>
+    </joint>
+    <link name="bumper_link">
+      <xacro:inertial_cylinder_with_pose mass="${base_mass}" radius="${base_diameter/2}" length="${base_height}">
+        <origin xyz="${base_link_origin}"/>
+      </xacro:inertial_cylinder_with_pose>
       <collision>
         <origin xyz="${base_link_origin}"/>
         <geometry>
-          <cylinder length="${base_height}" radius="${base_diameter/2}" />
+          <xacro:insert_block name="mesh" />
         </geometry>
       </collision>

File: ca_description/urdf/create_base_gazebo.xacro (robot description, xacro)
@@ -47,5 +47,5 @@
     </gazebo>
     <!-- Bumpers -->
-    <gazebo reference="base_link">
+    <gazebo reference="bumper_link">
       <gravity>true</gravity>
       <self_collide>false</self_collide>
@@ -55,10 +55,11 @@
         <update_rate>50</update_rate>
         <contact>
-          <collision>base_link_collision</collision>
+          <collision>bumper_link_collision</collision>
         </contact>
         <!-- Plugin -->
         <plugin name="create_bumper_controller" filename="libcreate_bumper_plugin.so">
-          <frameName>base_link</frameName>
-          <bumperTopicName>bumper</bumperTopicName>
+          <frameName>base_footprint</frameName>
+          <robotNamespace>${robot_name}</robotNamespace>
+          <topicName>bumper</topicName>
         </plugin>
       </sensor>
