Commit message: Add RViz colors and change IMU pose

File: ca_description/urdf/create_2.xacro (robot description, xacro)
@@ -2,4 +2,5 @@
 <robot name="create_2" xmlns:xacro="http://ros.org/wiki/xacro">
   <xacro:include filename="$(find ca_description)/urdf/create_base.xacro"/>
+  <xacro:include filename="$(find ca_description)/urdf/utils/materials.xacro"/>
   <xacro:property name="robot_name" value="$(arg robot_name)"/>
   <xacro:property name="wheel_separation" value="0.235"/>

File: ca_description/urdf/create_base.xacro (robot description, xacro)
@@ -1,5 +1,5 @@
 <?xml version="1.0" ?>
 <robot xmlns:xacro="http://ros.org/wiki/xacro">
-  <xacro:include filename="$(find ca_description)/urdf/common_properties.xacro"/>
+  <xacro:include filename="$(find ca_description)/urdf/utils/inertias.xacro"/>
   <xacro:include filename="$(find ca_description)/urdf/create_base_gazebo.xacro"/>
   <xacro:include filename="$(find ca_description)/urdf/create_battery.xacro"/>
@@ -62,7 +62,4 @@
       <origin xyz="0.15 -0.04 -0.01" rpy="0 ${pi/2 - 0.09} 0"/>
     </xacro:cliff_sensor>
-    <xacro:imu_sensor name="imu">
-      <origin xyz="0 -0.04 0.13"/>
-    </xacro:imu_sensor>
     <xacro:omni_sensor>
       <origin xyz="0.145 0 0.0308"/>

File: ca_description/urdf/create_battery.xacro (robot description, xacro)
@@ -2,5 +2,6 @@
 <robot xmlns:xacro="http://ros.org/wiki/xacro">
 <xacro:macro name="battery" params="name:=battery parent:=base_footprint *origin">
-  <xacro:include filename="$(find ca_description)/urdf/common_properties.xacro"/>
+  <xacro:include filename="$(find ca_description)/urdf/utils/inertias.xacro"/>
+  <xacro:include filename="$(find ca_description)/urdf/utils/conversions.xacro"/>
   <xacro:property name="parent_link" value="${parent}"/>
   <xacro:property name="link_name"   value="${name}_link"/>

File: ca_description/urdf/create_caster_wheel.xacro (robot description, xacro)
@@ -2,5 +2,5 @@
 <robot xmlns:xacro="http://ros.org/wiki/xacro">
 <xacro:macro name="caster_wheel" params="name:=caster_wheel parent:=base_link radius *origin">
-  <xacro:include filename="$(find ca_description)/urdf/common_properties.xacro"/>
+  <xacro:include filename="$(find ca_description)/urdf/utils/inertias.xacro"/>
   <xacro:property name="parent_link" value="${parent}"/>
   <xacro:property name="link_name"   value="${name}_link"/>
@@ -18,4 +18,5 @@
         <sphere radius="${radius}" />
       </geometry>
+      <material name="white_smoke"/>
     </visual>
     <collision>

File: ca_description/urdf/create_wheel.xacro (robot description, xacro)
@@ -2,5 +2,5 @@
 <robot xmlns:xacro="http://ros.org/wiki/xacro">
 <xacro:macro name="wheel" params="name:=wheel parent:=base_footprint radius width *origin">
-  <xacro:include filename="$(find ca_description)/urdf/common_properties.xacro"/>
+  <xacro:include filename="$(find ca_description)/urdf/utils/inertias.xacro"/>
   <xacro:property name="parent_link" value="${parent}"/>
   <xacro:property name="link_name"   value="${name}_link"/>
@@ -18,4 +18,5 @@
         <cylinder radius="${radius}" length="${width}" />
       </geometry>
+      <material name="lynch"/>
     </visual>
     <collision>

File: ca_description/urdf/sensors/cliff_sensors.xacro (robot description, xacro)
@@ -2,5 +2,5 @@
 <robot xmlns:xacro="http://ros.org/wiki/xacro">
 <xacro:macro name="cliff_sensor" params="name:=cliff_sensor parent:=base_link *origin">
-  <xacro:include filename="$(find ca_description)/urdf/common_properties.xacro"/>
+  <xacro:include filename="$(find ca_description)/urdf/utils/conversions.xacro"/>
   <xacro:property name="parent_link"        value="${parent}"/>
   <xacro:property name="link_name"          value="${name}_link"/>

File: ca_description/urdf/sensors/imu_sensor.xacro (robot description, xacro)
@@ -1,6 +1,6 @@
 <?xml version="1.0" ?>
 <robot xmlns:xacro="http://ros.org/wiki/xacro">
-<xacro:macro name="imu_sensor" params="name:=imu_sensor parent:=base_link *origin">
-  <xacro:include filename="$(find ca_description)/urdf/common_properties.xacro"/>
+<xacro:macro name="imu_sensor" params="name:=imu_sensor parent:=base_link *origin *mesh">
+  <xacro:include filename="$(find ca_description)/urdf/utils/inertias.xacro"/>
   <xacro:property name="parent_link" value="${parent}"/>
   <xacro:property name="link_name" value="${name}_link"/>
@@ -10,5 +10,12 @@
     <child link="${link_name}" />
   </joint>
-  <link name="${link_name}"/>
+  <link name="${link_name}">
+    <visual>
+      <geometry>
+        <xacro:insert_block name="mesh"/>
+      </geometry>
+      <material name="chambray"/>
+    </visual>
+  </link>
   <gazebo>
     <plugin name="${name}" filename="libgazebo_ros_imu.so">

File: ca_description/urdf/sensors/wall_sensor.xacro (robot description, xacro)
@@ -2,5 +2,5 @@
 <robot xmlns:xacro="http://ros.org/wiki/xacro">
 <xacro:macro name="wall_sensor" params="name:=wall_sensor parent:=base_link *origin">
-  <xacro:include filename="$(find ca_description)/urdf/common_properties.xacro"/>
+  <xacro:include filename="$(find ca_description)/urdf/utils/inertias.xacro"/>
   <xacro:property name="parent_link" value="${parent}"/>
   <xacro:property name="link_name"   value="${name}_link"/>

File: ca_description/urdf/stacks/roomblock.xacro (robot description, xacro)
@@ -4,5 +4,5 @@
 -->
 <robot xmlns:xacro="http://ros.org/wiki/xacro">
-<xacro:include filename="$(find ca_description)/urdf/common_properties.xacro"/>
+<xacro:include filename="$(find ca_description)/urdf/utils/inertias.xacro"/>
 <xacro:include filename="$(find ca_description)/urdf/sensors/camera_sensor.xacro"/>
 <xacro:property name="name" value="roomblock"/>

File: ca_description/urdf/stacks/turtlebot.xacro (robot description, xacro)
@@ -5,6 +5,7 @@
  -->
 <robot xmlns:xacro="http://ros.org/wiki/xacro">
+<xacro:include filename="$(find ca_description)/urdf/utils/conversions.xacro"/>
 <!-- Pole macro -->
-<xacro:macro name="stack_pole" params="name parent:=base_link *origin *mesh">
+<xacro:macro name="stack_pole" params="name parent:=base_link length *origin">
   <xacro:property name="link_name" value="pole_${name}_link"/>
   <joint name="pole_${name}_joint" type="fixed">
@@ -16,8 +17,12 @@
     <visual>
       <geometry>
-        <xacro:insert_block name="mesh"/>
+        <cylinder radius="0.006" length="${length}"/>
       </geometry>
+      <material name="silver"/>
     </visual>
   </link>
+  <gazebo reference="${link_name}">
+    <material>Gazebo/Grey</material>
+  </gazebo>
 </xacro:macro>
 <!-- turtlebot_stack -->
@@ -31,22 +36,21 @@
 </joint>
 <link name="${base_link}"/>
-<xacro:stack_pole name="short_0" parent="${base_link}">
-  <origin xyz="0.03 0.08 0"/>
-  <mesh filename="package://ca_description/meshes/turtlebot_stack/short_pole.dae"/>
+<xacro:property name="short_pole_length" value="0.06"/>
+<xacro:stack_pole name="short_0" parent="${base_link}" length="${short_pole_length}">
+  <origin xyz="0.03 0.08 ${short_pole_length/2.}"/>
 </xacro:stack_pole>
-<xacro:stack_pole name="short_1" parent="${base_link}">
-  <origin xyz="0.03 -0.08 0"/>
-  <mesh filename="package://ca_description/meshes/turtlebot_stack/short_pole.dae"/>
+<xacro:stack_pole name="short_1" parent="${base_link}" length="${short_pole_length}">
+  <origin xyz="0.03 -0.08 ${short_pole_length/2.}"/>
 </xacro:stack_pole>
-<xacro:stack_pole name="short_2" parent="${base_link}">
-  <origin xyz="-0.06 0.08 0"/>
-  <mesh filename="package://ca_description/meshes/turtlebot_stack/short_pole.dae"/>
+<xacro:stack_pole name="short_2" parent="${base_link}" length="${short_pole_length}">
+  <origin xyz="-0.06 0.08 ${short_pole_length/2.}"/>
 </xacro:stack_pole>
-<xacro:stack_pole name="short_3" parent="${base_link}">
-  <origin xyz="-0.06 -0.08 0"/>
-  <mesh filename="package://ca_description/meshes/turtlebot_stack/short_pole.dae"/>
+<xacro:stack_pole name="short_3" parent="${base_link}" length="${short_pole_length}">
+  <origin xyz="-0.06 -0.08 ${short_pole_length/2.}"/>
 </xacro:stack_pole>
+<xacro:property name="plate_height"   value="0.002"/>
+<xacro:property name="plate_bottom_z" value="${short_pole_length + plate_height}"/>
 <joint name="plate_bottom_joint" type="fixed">
-  <origin xyz="-0.025 0 0.032"/>
+  <origin xyz="-0.025 0 ${plate_bottom_z}"/>
   <parent link="${base_link}"/>
   <child link="plate_bottom_link"/>
@@ -59,22 +63,21 @@
   </visual>
 </link>
-<xacro:stack_pole name="large_0" parent="${base_link}">
-  <origin xyz="0.03 0.08 0.077"/>
-  <mesh filename="package://ca_description/meshes/turtlebot_stack/large_pole.dae"/>
+<xacro:property name="large_pole_length" value="0.087"/>
+<xacro:property name="large_pole_z"      value="${plate_bottom_z + plate_height + large_pole_length/2.}"/>
+<xacro:stack_pole name="large_0" parent="${base_link}" length="${large_pole_length}">
+  <origin xyz="0.03 0.08 ${large_pole_z}"/>
 </xacro:stack_pole>
-<xacro:stack_pole name="large_1" parent="${base_link}">
-  <origin xyz="0.03 -0.08 0.077"/>
-  <mesh filename="package://ca_description/meshes/turtlebot_stack/large_pole.dae"/>
+<xacro:stack_pole name="large_1" parent="${base_link}" length="${large_pole_length}">
+  <origin xyz="0.03 -0.08 ${large_pole_z}"/>
 </xacro:stack_pole>
-<xacro:stack_pole name="large_2" parent="${base_link}">
-  <origin xyz="-0.06 0.08 0.077"/>
-  <mesh filename="package://ca_description/meshes/turtlebot_stack/large_pole.dae"/>
+<xacro:stack_pole name="large_2" parent="${base_link}" length="${large_pole_length}">
+  <origin xyz="-0.06 0.08 ${large_pole_z}"/>
 </xacro:stack_pole>
-<xacro:stack_pole name="large_3" parent="${base_link}">
-  <origin xyz="-0.06 -0.08 0.077"/>
-  <mesh filename="package://ca_description/meshes/turtlebot_stack/large_pole.dae"/>
+<xacro:stack_pole name="large_3" parent="${base_link}" length="${large_pole_length}">
+  <origin xyz="-0.06 -0.08 ${large_pole_z}"/>
 </xacro:stack_pole>
+<xacro:property name="plate_upper_z" value="${plate_bottom_z + large_pole_length + plate_height}"/>
 <joint name="plate_upper_joint" type="fixed">
-  <origin xyz="-0.01364 0 0.117"/>
+  <origin xyz="-0.01364 0 ${plate_upper_z}"/>
   <parent link="${base_link}"/>
   <child link="plate_upper_link"/>
@@ -85,9 +88,10 @@
       <mesh filename="package://ca_description/meshes/turtlebot_stack/upper_plate.dae"/>
     </geometry>
+    <material name="silver"/>
   </visual>
 </link>
 <!-- Nvidia Jetson Nano -->
 <joint name="nvidia_jetson_nano_joint" type="fixed">
-  <origin xyz="0 0 0.003" rpy="0 0 ${-pi/2}"/>
+  <origin xyz="-0.015 -0.025 ${plate_height}" rpy="0 0 ${-pi/2}"/>
   <parent link="plate_bottom_link"/>
   <child link="nvidia_jetson_nano_link"/>
@@ -103,4 +107,9 @@
   <material>Gazebo/Grey</material>
 </gazebo>
+<!-- MPU9255 -->
+<xacro:imu_sensor name="mpu9255" parent="plate_upper_link">
+  <origin xyz="0.03 -0.15 ${plate_height + 0.002}" rpy="0 ${3*deg_to_rad} 0"/>
+  <mesh filename="package://ca_description/meshes/sensors/mpu9255.stl" scale="0.001 0.001 0.001"/>
+</xacro:imu_sensor>
 <!-- Laser -->
 <xacro:property name="laser" default="$(arg laser)"/>
