Commit message: Use optical link for camera

File: ca_description/urdf/sensors/camera_sensor.xacro (robot description, xacro)
@@ -5,18 +5,25 @@
   <xacro:property name="parent_link" value="${parent}"/>
   <xacro:property name="camera_link" value="raspicam_link"/>
+  <xacro:property name="optical_link" value="raspicam_link_optical"/>
   <xacro:property name="x" value="0.04"/>
   <xacro:property name="y" value="0.0"/>
   <xacro:property name="z" value="0.1"/>
-  <xacro:property name="R" value="0.0"/>
+  <xacro:property name="R" value="${-pi/2}"/>
   <xacro:property name="P" value="0.0"/>
-  <xacro:property name="Y" value="0.0"/>
+  <xacro:property name="Y" value="${-pi/2}"/>
   <joint name="camera_joint" type="fixed">
-    <origin xyz="${x} ${y} ${z}" rpy="${R} ${P} ${Y}" />
+    <origin xyz="${x} ${y} ${z}" rpy="0 0 0" />
     <parent link="${parent_link}" />
     <child link="${camera_link}" />
   </joint>
   <link name="${camera_link}"/>
+  <joint name="optical_joint" type="fixed">
+    <origin xyz="0 0 0" rpy="${R} ${P} ${Y}" />
+    <parent link="${camera_link}" />
+    <child link="${optical_link}" />
+  </joint>
+  <link name="${optical_link}"/>
   <!-- Gazebo plugin -->
-  <xacro:camera_sensor_gazebo link_name="${camera_link}"/>
+  <xacro:camera_sensor_gazebo link_name="${optical_link}"/>
 </xacro:macro>
 </robot>

File: ca_description/urdf/sensors/camera_sensor_gazebo.xacro (robot description, xacro)
@@ -4,5 +4,5 @@
   <gazebo reference="${link_name}">
     <material>Gazebo/Orange</material>
-    <sensor type="camera" name="camera1">
+    <sensor type="camera" name="raspicam">
       <update_rate>30.0</update_rate>
       <camera name="head">
@@ -33,5 +33,5 @@
         <cameraInfoTopicName>camera_info</cameraInfoTopicName>
         <frameName>${link_name}</frameName>
-        <hackBaseline>0.07</hackBaseline>
+        <hackBaseline>0.0</hackBaseline>
         <distortionK1>0.0</distortionK1>
         <distortionK2>0.0</distortionK2>

Commit message: Fixed camera orientation: added generic_camera XACRO macro

File: ca_description/urdf/sensors/camera_sensor.xacro (robot description, xacro)
@@ -1,29 +1,12 @@
 <?xml version="1.0"?>
 <robot xmlns:xacro="http://ros.org/wiki/xacro">
-<xacro:include filename="$(find ca_description)/urdf/sensors/camera_sensor_gazebo.xacro"/>
+<xacro:include filename="$(find ca_description)/urdf/sensors/camera_generic.xacro"/>
 <xacro:macro name="camera_sensor" params="parent">
-  <xacro:property name="parent_link" value="${parent}"/>
-  <xacro:property name="camera_link" value="raspicam_link"/>
-  <xacro:property name="optical_link" value="raspicam_link_optical"/>
   <xacro:property name="x" value="0.04"/>
   <xacro:property name="y" value="0.0"/>
   <xacro:property name="z" value="0.1"/>
-  <xacro:property name="R" value="${-pi/2}"/>
-  <xacro:property name="P" value="0.0"/>
-  <xacro:property name="Y" value="${-pi/2}"/>
-  <joint name="camera_joint" type="fixed">
-    <origin xyz="${x} ${y} ${z}" rpy="0 0 0" />
-    <parent link="${parent_link}" />
-    <child link="${camera_link}" />
-  </joint>
-  <link name="${camera_link}"/>
-  <joint name="optical_joint" type="fixed">
-    <origin xyz="0 0 0" rpy="${R} ${P} ${Y}" />
-    <parent link="${camera_link}" />
-    <child link="${optical_link}" />
-  </joint>
-  <link name="${optical_link}"/>
-  <!-- Gazebo plugin -->
-  <xacro:camera_sensor_gazebo link_name="${optical_link}"/>
+  <xacro:generic_camera name="raspicam" parent="${parent}">
+    <origin xyz="${x} ${y} ${z}" rpy="0 0 0"/>
+  </xacro:generic_camera>
 </xacro:macro>
 </robot>

Commit message: Fix camera position

File: ca_description/urdf/sensors/camera_sensor.xacro (robot description, xacro)
@@ -5,5 +5,5 @@
   <xacro:property name="x" value="0.04"/>
   <xacro:property name="y" value="0.0"/>
-  <xacro:property name="z" value="0.1"/>
+  <xacro:property name="z" value="0.06"/>
   <xacro:generic_camera name="raspicam" parent="${parent}">
     <origin xyz="${x} ${y} ${z}" rpy="0 0 0"/>
