Commit message: Delete unnecessary fixed joint property

File: ca_description/urdf/sensors/imu_sensor.xacro (robot description, xacro)
@@ -13,5 +13,4 @@
   <xacro:property name="Y" value="0"/>
   <joint name="gyro_joint" type="fixed">
-    <axis xyz="1 0 0" />
     <origin xyz="${x} ${y} ${z}" rpy="${R} ${P} ${Y}"/>
     <parent link="${parent_link}" />

Commit message: Add new frame to IMU

File: ca_description/urdf/sensors/imu_sensor.xacro (robot description, xacro)
@@ -5,4 +5,5 @@
   <xacro:property name="parent_link" value="${parent}"/>
   <xacro:property name="link_name" value="${name}_link"/>
+  <xacro:property name="chip_name" value="${name}_chip_link"/>
   <joint name="${name}_joint" type="fixed">
     <xacro:insert_block name="origin" />
@@ -18,4 +19,13 @@
     </visual>
   </link>
+  <gazebo reference="${link_name}">
+    <material>Gazebo/BlueGlow</material>
+  </gazebo>
+  <joint name="${name}_chip_joint" type="fixed">
+    <origin rpy="${pi} 0 0"/>
+    <parent link="${link_name}" />
+    <child link="${chip_name}" />
+  </joint>
+  <link name="${chip_name}"/>
   <gazebo>
     <plugin name="${name}" filename="libgazebo_ros_imu.so">
@@ -23,6 +33,6 @@
       <updateRate>30</updateRate>
       <robotNamespace>create1</robotNamespace>
-      <bodyName>${link_name}</bodyName>
-      <frameName>create1_tf/${link_name}</frameName>
+      <bodyName>${chip_name}</bodyName>
+      <frameName>create1_tf/${chip_name}</frameName>
       <topicName>${name}/data</topicName>
       <serviceName>${name}/is_calibrated</serviceName>

Commit message: Fix IMU!

File: ca_description/urdf/sensors/imu_sensor.xacro (robot description, xacro)
@@ -5,5 +5,4 @@
   <xacro:property name="parent_link" value="${parent}"/>
   <xacro:property name="link_name" value="${name}_link"/>
-  <xacro:property name="chip_name" value="${name}_chip_link"/>
   <joint name="${name}_joint" type="fixed">
     <xacro:insert_block name="origin" />
@@ -22,10 +21,4 @@
     <material>Gazebo/BlueGlow</material>
   </gazebo>
-  <joint name="${name}_chip_joint" type="fixed">
-    <origin rpy="${pi} 0 0"/>
-    <parent link="${link_name}" />
-    <child link="${chip_name}" />
-  </joint>
-  <link name="${chip_name}"/>
   <gazebo>
     <plugin name="${name}" filename="libgazebo_ros_imu.so">
@@ -33,6 +26,6 @@
       <updateRate>30</updateRate>
       <robotNamespace>create1</robotNamespace>
-      <bodyName>${chip_name}</bodyName>
-      <frameName>create1_tf/${chip_name}</frameName>
+      <bodyName>${link_name}</bodyName>
+      <frameName>create1_tf/${link_name}</frameName>
       <topicName>${name}/data</topicName>
       <serviceName>${name}/is_calibrated</serviceName>
