Commit message: Simplify code using a .yaml to define poses

File: ca_description/urdf/sensors/lasers/astra.xacro (robot description, xacro)
@@ -3,43 +3,43 @@
 <xacro:include filename="$(find ca_description)/urdf/sensors/lasers/sim_3d_sensor.xacro"/>
 <!-- Orbbec Astra RGBD Camera -->
-<xacro:macro name="orbbec_astra" params="name:=astra parent:=base_link *origin">
-  <xacro:property name="parent_link"    value="${parent}"/>
-  <xacro:property name="link_name"      value="${name}_link"/>
-  <xacro:property name="link_rgb"       value="${name}_rgb_frame"/>
-  <xacro:property name="link_depth"     value="${name}_depth_frame"/>
-  <xacro:property name="link_optical"   value="${name}_depth_optical_frame"/>
-  <xacro:property name="optical_offset" value="0.01"/>
-  <joint name="${name}_joint" type="fixed">
-    <xacro:insert_block name="origin"/>
-    <parent link="${parent_link}"/>
-    <child link="${link_name}"/>
-  </joint>
-  <link name="${link_name}">
-    <visual>
-      <origin xyz="-0.01 0 -0.03" rpy="${pi/2} 0 ${pi/2}"/>
-      <geometry>
-        <mesh filename="package://ca_description/meshes/astra.dae"/>
-      </geometry>
-    </visual>
-  </link>
-  <joint name="${name}_optical_joint" type="fixed">
-    <origin xyz="0 ${optical_offset} 0" rpy="${-pi/2} 0 ${-pi/2}"/>
-    <parent link="${link_name}"/>
-    <child link="${link_rgb}"/>
-  </joint>
-  <link name="${link_rgb}"/>
-  <joint name="${name}_depth_joint" type="fixed">
-    <origin rpy="${-pi/2} 0 ${-pi/2}"/>
-    <parent link="${link_name}"/>
-    <child link="${link_depth}"/>
-  </joint>
-  <link name="${link_depth}"/>
-   <joint name="${name}_depth_optical_joint" type="fixed">
-    <origin rpy="${-pi/2} 0 ${-pi/2}"/>
-    <parent link="${link_depth}"/>
-    <child link="${link_optical}"/>
-  </joint>
-  <link name="${link_optical}"/>
-  <xacro:sim_3d_sensor name="${name}" color="Gazebo/FlatBlack"/>
-</xacro:macro>
+<xacro:property name="name" value="astra"/>
+<xacro:property name="parent" value="base_link"/>
+<xacro:property name="parent_link"    value="${parent}"/>
+<xacro:property name="link_name"      value="${name}_link"/>
+<xacro:property name="link_rgb"       value="${name}_rgb_frame"/>
+<xacro:property name="link_depth"     value="${name}_depth_frame"/>
+<xacro:property name="link_optical"   value="${name}_depth_optical_frame"/>
+<xacro:property name="optical_offset" value="0.01"/>
+<joint name="${name}_joint" type="fixed">
+  <origin xyz="${laser_origin}"/>
+  <parent link="${parent_link}"/>
+  <child link="${link_name}"/>
+</joint>
+<link name="${link_name}">
+  <visual>
+    <origin xyz="-0.01 0 -0.03" rpy="${pi/2} 0 ${pi/2}"/>
+    <geometry>
+      <mesh filename="package://ca_description/meshes/astra.dae"/>
+    </geometry>
+  </visual>
+</link>
+<joint name="${name}_optical_joint" type="fixed">
+  <origin xyz="0 ${optical_offset} 0" rpy="${-pi/2} 0 ${-pi/2}"/>
+  <parent link="${link_name}"/>
+  <child link="${link_rgb}"/>
+</joint>
+<link name="${link_rgb}"/>
+<joint name="${name}_depth_joint" type="fixed">
+  <origin rpy="${-pi/2} 0 ${-pi/2}"/>
+  <parent link="${link_name}"/>
+  <child link="${link_depth}"/>
+</joint>
+<link name="${link_depth}"/>
+  <joint name="${name}_depth_optical_joint" type="fixed">
+  <origin rpy="${-pi/2} 0 ${-pi/2}"/>
+  <parent link="${link_depth}"/>
+  <child link="${link_optical}"/>
+</joint>
+<link name="${link_optical}"/>
+<xacro:sim_3d_sensor name="${name}" color="Gazebo/FlatBlack"/>
 </robot>

File: ca_description/urdf/sensors/lasers/kinect.xacro (robot description, xacro)
@@ -2,50 +2,50 @@
 <robot xmlns:xacro="http://ros.org/wiki/xacro">
 <xacro:include filename="$(find ca_description)/urdf/sensors/lasers/sim_3d_sensor.xacro"/>
-<xacro:macro name="kinect" params="name:=kinect parent:=base_link *origin">
-  <xacro:property name="parent_link"        value="${parent}"/>
-  <xacro:property name="link_name"          value="${name}_link"/>
-  <xacro:property name="link_rgb"           value="${name}_rgb_frame"/>
-  <xacro:property name="link_rgb_optical"   value="${name}_rgb_optical_frame"/>
-  <xacro:property name="link_depth"         value="${name}_depth_frame"/>
-  <xacro:property name="link_depth_optical" value="${name}_depth_optical_frame"/>
-  <xacro:property name="kinect_cam_py" value="-0.0125"/>
-  <joint name="camera_rgb_joint" type="fixed">
-    <xacro:insert_block name="origin"/>
-    <parent link="${parent}"/>
-    <child link="${link_rgb}" />
-  </joint>
-  <link name="${link_rgb}"/>
-  <joint name="${name}_rgb_optical_joint" type="fixed">
-    <origin rpy="${-pi/2} 0 ${-pi/2}" />
-    <parent link="${link_rgb}" />
-    <child link="${link_rgb_optical}" />
-  </joint>
-  <link name="${link_rgb_optical}"/>
-  <joint name="camera_joint" type="fixed">
-    <origin xyz="-0.031 ${-kinect_cam_py} -0.016"/>
-    <parent link="${link_rgb}"/>
-    <child link="${link_name}"/>
-  </joint>
-  <link name="${link_name}">
-    <visual>
-      <origin rpy="0 0 ${pi/2}"/>
-      <geometry>
-        <mesh filename="package://ca_description/meshes/kinect.dae"/>
-      </geometry>
-    </visual>
-  </link>
-	<joint name="${name}_depth_joint" type="fixed">
-	  <origin xyz="0 ${2 * -kinect_cam_py} 0"/>
-	  <parent link="${link_rgb}" />
-	  <child link="${link_depth}" />
-	</joint>
-	<link name="${link_depth}"/>
-	<joint name="${name}_depth_optical_joint" type="fixed">
-	  <origin rpy="${-pi/2} 0 ${-pi/2}" />
-	  <parent link="${link_depth}" />
-	  <child link="${link_depth_optical}"/>
-	</joint>
-	<link name="${link_depth_optical}"/>
-	<xacro:sim_3d_sensor name="${name}" color="Gazebo/FlatBlack"/>
-</xacro:macro>
+<xacro:property name="name" value="kinect"/>
+<xacro:property name="parent" value="base_link"/>
+<xacro:property name="parent_link"        value="${parent}"/>
+<xacro:property name="link_name"          value="${name}_link"/>
+<xacro:property name="link_rgb"           value="${name}_rgb_frame"/>
+<xacro:property name="link_rgb_optical"   value="${name}_rgb_optical_frame"/>
+<xacro:property name="link_depth"         value="${name}_depth_frame"/>
+<xacro:property name="link_depth_optical" value="${name}_depth_optical_frame"/>
+<xacro:property name="kinect_cam_py" value="-0.0125"/>
+<joint name="camera_rgb_joint" type="fixed">
+  <origin xyz="${laser_origin}"/>
+  <parent link="${parent}"/>
+  <child link="${link_rgb}" />
+</joint>
+<link name="${link_rgb}"/>
+<joint name="${name}_rgb_optical_joint" type="fixed">
+  <origin rpy="${-pi/2} 0 ${-pi/2}" />
+  <parent link="${link_rgb}" />
+  <child link="${link_rgb_optical}" />
+</joint>
+<link name="${link_rgb_optical}"/>
+<joint name="camera_joint" type="fixed">
+  <origin xyz="-0.031 ${-kinect_cam_py} -0.016"/>
+  <parent link="${link_rgb}"/>
+  <child link="${link_name}"/>
+</joint>
+<link name="${link_name}">
+  <visual>
+    <origin rpy="0 0 ${pi/2}"/>
+    <geometry>
+      <mesh filename="package://ca_description/meshes/kinect.dae"/>
+    </geometry>
+  </visual>
+</link>
+<joint name="${name}_depth_joint" type="fixed">
+  <origin xyz="0 ${2 * -kinect_cam_py} 0"/>
+  <parent link="${link_rgb}" />
+  <child link="${link_depth}" />
+</joint>
+<link name="${link_depth}"/>
+<joint name="${name}_depth_optical_joint" type="fixed">
+  <origin rpy="${-pi/2} 0 ${-pi/2}" />
+  <parent link="${link_depth}" />
+  <child link="${link_depth_optical}"/>
+</joint>
+<link name="${link_depth_optical}"/>
+<xacro:sim_3d_sensor name="${name}" color="Gazebo/FlatBlack"/>
 </robot>

File: ca_description/urdf/sensors/lasers/rplidar.xacro (robot description, xacro)
@@ -1,65 +1,65 @@
 <?xml version="1.0"?>
 <robot xmlns:xacro="http://ros.org/wiki/xacro">
-<xacro:macro name="rplidar_a2" params="name:=rplidar parent:=base_link visualize:=false *origin">
-  <xacro:property name="parent_link"              value="${parent}"/>
-  <xacro:property name="link_name"                value="${name}_link"/>
-  <xacro:property name="laser_link"               value="laser_link"/>
-  <xacro:property name="rplidar_a2_rate_hz"       value="10"/>
-  <xacro:property name="rplidar_a2_min_range_m"   value="0.15"/>
-  <xacro:property name="rplidar_a2_max_range_m"   value="12.0"/>
-  <xacro:property name="rplidar_a2_samples"       value="720"/>
-  <xacro:property name="rplidar_a2_resolution_mm" value="0.5"/>
-  <xacro:property name="rplidar_a2_min_angle_rad" value="${-pi}"/>
-  <xacro:property name="rplidar_a2_max_angle_rad" value="${pi}"/>
-  <xacro:property name="topic_name"               value="laser/scan"/>
-  <joint name="${name}_joint" type="fixed">
-    <xacro:insert_block name="origin"/>
-    <parent link="${parent_link}"/>
-    <child link="${link_name}"/>
-  </joint>
-  <link name="${link_name}">
-    <visual>
-      <geometry>
-        <mesh filename="package://ca_description/meshes/rplidar.dae"/>
-      </geometry>
-    </visual>
-  </link>
-  <joint name="laser_joint" type="fixed">
-    <origin xyz="0 0 0.0308"/>
-    <parent link="${link_name}"/>
-    <child link="${laser_link}"/>
-  </joint>
-  <link name="${laser_link}"/>
-  <gazebo reference="${laser_link}">
-    <material>Gazebo/FlatBlack</material>
-    <sensor type="ray" name="${name}_sensor">
-      <visualize>${visualize}</visualize>
-      <update_rate>${rplidar_a2_rate_hz}</update_rate>
-      <ray>
-        <scan>
-          <horizontal>
-            <samples>${rplidar_a2_samples}</samples>
-            <resolution>1</resolution>
-            <min_angle>${rplidar_a2_min_angle_rad}</min_angle>
-            <max_angle>${rplidar_a2_max_angle_rad}</max_angle>
-          </horizontal>
-        </scan>
-        <range>
-          <min>${rplidar_a2_min_range_m}</min>
-          <max>${rplidar_a2_max_range_m}</max>
-          <resolution>${rplidar_a2_resolution_mm / 1000.0}</resolution>
-        </range>
-        <noise>
-          <type>gaussian</type>
-          <mean>0.0</mean>
-          <stddev>0.01</stddev>
-        </noise>
-      </ray>
-      <plugin name="gazebo_ros_${name}" filename="libgazebo_ros_laser.so">
-        <topicName>${topic_name}</topicName>
-        <frameName>${laser_link}</frameName>
-      </plugin>
-    </sensor>
-  </gazebo>
-</xacro:macro>
+<xacro:property name="name" value="rplidar"/>
+<xacro:property name="parent" value="base_link"/>
+<xacro:property name="parent_link"              value="${parent}"/>
+<xacro:property name="link_name"                value="${name}_link"/>
+<xacro:property name="laser_link"               value="laser_link"/>
+<xacro:property name="rplidar_a2_rate_hz"       value="10"/>
+<xacro:property name="rplidar_a2_min_range_m"   value="0.15"/>
+<xacro:property name="rplidar_a2_max_range_m"   value="12.0"/>
+<xacro:property name="rplidar_a2_samples"       value="720"/>
+<xacro:property name="rplidar_a2_resolution_mm" value="0.5"/>
+<xacro:property name="rplidar_a2_min_angle_rad" value="${-pi}"/>
+<xacro:property name="rplidar_a2_max_angle_rad" value="${pi}"/>
+<xacro:property name="topic_name"               value="laser/scan"/>
+<joint name="${name}_joint" type="fixed">
+  <origin xyz="${laser_origin}"/>
+  <parent link="${parent_link}"/>
+  <child link="${link_name}"/>
+</joint>
+<link name="${link_name}">
+  <visual>
+    <geometry>
+      <mesh filename="package://ca_description/meshes/rplidar.dae"/>
+    </geometry>
+  </visual>
+</link>
+<joint name="laser_joint" type="fixed">
+  <origin xyz="0 0 0.0308"/>
+  <parent link="${link_name}"/>
+  <child link="${laser_link}"/>
+</joint>
+<link name="${laser_link}"/>
+<gazebo reference="${laser_link}">
+  <material>Gazebo/FlatBlack</material>
+  <sensor type="ray" name="${name}_sensor">
+    <visualize>${visualize}</visualize>
+    <update_rate>${rplidar_a2_rate_hz}</update_rate>
+    <ray>
+      <scan>
+        <horizontal>
+          <samples>${rplidar_a2_samples}</samples>
+          <resolution>1</resolution>
+          <min_angle>${rplidar_a2_min_angle_rad}</min_angle>
+          <max_angle>${rplidar_a2_max_angle_rad}</max_angle>
+        </horizontal>
+      </scan>
+      <range>
+        <min>${rplidar_a2_min_range_m}</min>
+        <max>${rplidar_a2_max_range_m}</max>
+        <resolution>${rplidar_a2_resolution_mm / 1000.0}</resolution>
+      </range>
+      <noise>
+        <type>gaussian</type>
+        <mean>0.0</mean>
+        <stddev>0.01</stddev>
+      </noise>
+    </ray>
+    <plugin name="gazebo_ros_${name}" filename="libgazebo_ros_laser.so">
+      <topicName>${topic_name}</topicName>
+      <frameName>${laser_link}</frameName>
+    </plugin>
+  </sensor>
+</gazebo>
 </robot>

File: ca_description/urdf/stacks/roomblock.xacro (robot description, xacro)
@@ -35,36 +35,10 @@
       <material>Gazebo/Grey</material>
     </gazebo>
-    <xacro:include filename="$(find ca_description)/urdf/sensors/lasers/astra.xacro"/>
-    <xacro:include filename="$(find ca_description)/urdf/sensors/lasers/kinect.xacro"/>
-    <xacro:include filename="$(find ca_description)/urdf/sensors/lasers/realsense.xacro"/>
-    <xacro:include filename="$(find ca_description)/urdf/sensors/lasers/rplidar.xacro"/>
-    <xacro:include filename="$(find ca_description)/urdf/sensors/lasers/xtion_pro.xacro"/>
+    <!-- Laser -->
     <xacro:property name="laser" default="$(arg laser)"/>
-    <!-- TODO: Implement this in a dictionary (along with include file) -->
-    <xacro:if value="${laser == 'astra'}">
-      <xacro:orbbec_astra>
-        <origin xyz="0 0 0.2"/>
-      </xacro:orbbec_astra>
-    </xacro:if>
-    <xacro:if value="${laser == 'kinect'}">
-      <xacro:kinect>
-        <origin xyz="0.025 -0.01 0.22"/>
-      </xacro:kinect>
-    </xacro:if>
-    <xacro:if value="${laser == 'rplidar'}">
-      <xacro:rplidar_a2 parent="${link_name}" visualize="${visualize}">
-        <origin xyz="0 0 0.1"/>
-      </xacro:rplidar_a2>
-    </xacro:if>
-    <xacro:if value="${laser == 'r200'}">
-      <xacro:realsense_r200>
-        <origin xyz="0 0 0.182"/>
-      </xacro:realsense_r200>
-    </xacro:if>
-    <xacro:if value="${laser == 'xtion_pro'}">
-      <xacro:asus_xtion_pro>
-        <origin xyz="0.015 0.018 0.191"/>
-      </xacro:asus_xtion_pro>
-    </xacro:if>
+    <xacro:property name="laser_yaml" value="$(find ca_description)/urdf/sensors/lasers/poses.yaml"/>
+    <xacro:property name="laser_dict" value="${load_yaml(laser_yaml)}"/>
+    <xacro:property name="laser_origin" value="${laser_dict['roomblock'][laser]}"/>
+    <xacro:include filename="$(find ca_description)/urdf/sensors/lasers/${laser}.xacro"/>
     <!-- TODO (eborghi): ADD CAMERA CAD? REMOVE CAMERA/USE ANOTHER ONE? -->
     <xacro:camera_sensor name="raspicam" parent="${link_name}"/>

File: ca_description/urdf/stacks/turtlebot.xacro (robot description, xacro)
@@ -5,5 +5,4 @@
  -->
 <robot xmlns:xacro="http://ros.org/wiki/xacro">
-  <!-- <xacro:include filename="$(find ca_description)/urdf/common_properties.urdf.xacro"/> -->
   <!-- Pole macros -->
   <xacro:macro name="stack_bottom_pole" params="parent:=base_link number *origin">
@@ -158,4 +157,10 @@
       </visual>
     </link>
+    <!-- Laser -->
+    <xacro:property name="laser" default="$(arg laser)"/>
+    <xacro:property name="laser_yaml" value="$(find ca_description)/urdf/sensors/lasers/poses.yaml"/>
+    <xacro:property name="laser_dict" value="${load_yaml(laser_yaml)}"/>
+    <xacro:property name="laser_origin" value="${laser_dict['turtlebot'][laser]}"/>
+    <xacro:include filename="$(find ca_description)/urdf/sensors/lasers/${laser}.xacro"/>
   </xacro:macro>
 </robot>

Commit message: Use meshes from new directory

File: ca_description/urdf/sensors/lasers/astra.xacro (robot description, xacro)
@@ -20,5 +20,5 @@
     <origin xyz="-0.01 0 -0.03" rpy="${pi/2} 0 ${pi/2}"/>
     <geometry>
-      <mesh filename="package://ca_description/meshes/astra.dae"/>
+      <mesh filename="package://ca_description/meshes/sensors/astra.dae"/>
     </geometry>
   </visual>

File: ca_description/urdf/sensors/lasers/kinect.xacro (robot description, xacro)
@@ -32,5 +32,5 @@
     <origin rpy="0 0 ${pi/2}"/>
     <geometry>
-      <mesh filename="package://ca_description/meshes/kinect.dae"/>
+      <mesh filename="package://ca_description/meshes/sensors/kinect.dae"/>
     </geometry>
   </visual>

File: ca_description/urdf/sensors/lasers/r200.xacro (robot description, xacro)
@@ -20,5 +20,5 @@
   <visual>
     <geometry>
-      <mesh filename="package://ca_description/meshes/realsense_r200.dae"/>
+      <mesh filename="package://ca_description/meshes/sensors/realsense_r200.dae"/>
     </geometry>
   </visual>

File: ca_description/urdf/sensors/lasers/rplidar.xacro (robot description, xacro)
@@ -22,5 +22,5 @@
   <visual>
     <geometry>
-      <mesh filename="package://ca_description/meshes/rplidar.dae"/>
+      <mesh filename="package://ca_description/meshes/sensors/rplidar.dae"/>
     </geometry>
   </visual>
@@ -32,6 +32,8 @@
 </joint>
 <link name="${laser_link}"/>
+<gazebo reference="${link_name}">
+  <material>Gazebo/FlatBlack</material>
+</gazebo>
 <gazebo reference="${laser_link}">
-  <material>Gazebo/FlatBlack</material>
   <sensor type="ray" name="${name}_sensor">
     <visualize>$(arg visualize)</visualize>

File: ca_description/urdf/sensors/lasers/xtion_pro.xacro (robot description, xacro)
@@ -2,52 +2,53 @@
 <robot xmlns:xacro="http://ros.org/wiki/xacro">
 <xacro:include filename="$(find ca_description)/urdf/sensors/lasers/sim_3d_sensor.xacro"/>
-<xacro:macro name="asus_xtion_pro" params="name:=xtion_pro parent:=base_link *origin">
-  <xacro:property name="parent_link"        value="${parent}"/>
-  <xacro:property name="link_name"          value="${name}_link"/>
-  <xacro:property name="link_rgb"           value="${name}_rgb_frame"/>
-  <xacro:property name="link_rgb_optical"   value="${name}_rgb_optical_frame"/>
-  <xacro:property name="link_depth"         value="${name}_depth_frame"/>
-  <xacro:property name="link_depth_optical" value="${name}_depth_optical_frame"/>
-  <!-- Xacro properties -->
-  <xacro:property name="xtion_pro_depth_rel_rgb_py" value="0.0270" />
-  <xacro:property name="xtion_pro_cam_rel_rgb_py"   value="-0.0220" />
-  <joint name="${name}_rgb_joint" type="fixed">
-    <xacro:insert_block name="origin"/>
-    <parent link="${parent}"/>
-    <child link="${link_rgb}" />
-  </joint>
-  <link name="${link_rgb}"/>
-  <joint name="${name}_rgb_optical_joint" type="fixed">
-    <origin rpy="${-pi/2} 0 ${-pi/2}" />
-    <parent link="${link_rgb}" />
-    <child link="${link_rgb_optical}" />
-  </joint>
-  <link name="${link_rgb_optical}"/>
-  <joint name="${name}_joint" type="fixed">
-    <origin xyz="0 ${xtion_pro_cam_rel_rgb_py} 0"/>
-    <parent link="${link_rgb}"/>
-    <child link="${link_name}"/>
-  </joint>
-  <link name="${link_name}">
-    <visual>
-      <origin xyz="-0.015 0.0035 0.004"/>
-      <geometry>
-        <mesh filename="package://ca_description/meshes/asus_xtion_pro_live.dae"/>
-      </geometry>
-    </visual>
-  </link>
-  <joint name="${name}_depth_joint" type="fixed">
-    <origin xyz="0 ${xtion_pro_depth_rel_rgb_py} 0"/>
-    <parent link="${link_rgb}" />
-    <child link="${link_depth}"/>
-  </joint>
-  <link name="${link_depth}"/>
-  <joint name="${name}_depth_optical_joint" type="fixed">
-    <origin rpy="${-pi/2} 0 ${-pi/2}" />
-    <parent link="${link_depth}" />
-    <child link="${link_depth_optical}" />
-  </joint>
-  <link name="${link_depth_optical}"/>
-  <xacro:sim_3d_sensor name="${name}" color="Gazebo/FlatBlack"/>
-</xacro:macro>
+<!-- Orbbec Astra RGBD Camera -->
+<xacro:property name="name" value="xtion_pro"/>
+<xacro:property name="parent" value="base_link"/>
+<xacro:property name="parent_link"        value="${parent}"/>
+<xacro:property name="link_name"          value="${name}_link"/>
+<xacro:property name="link_rgb"           value="${name}_rgb_frame"/>
+<xacro:property name="link_rgb_optical"   value="${name}_rgb_optical_frame"/>
+<xacro:property name="link_depth"         value="${name}_depth_frame"/>
+<xacro:property name="link_depth_optical" value="${name}_depth_optical_frame"/>
+<!-- Xacro properties -->
+<xacro:property name="xtion_pro_depth_rel_rgb_py" value="0.0270" />
+<xacro:property name="xtion_pro_cam_rel_rgb_py"   value="-0.0220" />
+<joint name="${name}_rgb_joint" type="fixed">
+  <origin xyz="${laser_origin}"/>
+  <parent link="${parent}"/>
+  <child link="${link_rgb}" />
+</joint>
+<link name="${link_rgb}"/>
+<joint name="${name}_rgb_optical_joint" type="fixed">
+  <origin rpy="${-pi/2} 0 ${-pi/2}" />
+  <parent link="${link_rgb}" />
+  <child link="${link_rgb_optical}" />
+</joint>
+<link name="${link_rgb_optical}"/>
+<joint name="${name}_joint" type="fixed">
+  <origin xyz="0 ${xtion_pro_cam_rel_rgb_py} 0"/>
+  <parent link="${link_rgb}"/>
+  <child link="${link_name}"/>
+</joint>
+<link name="${link_name}">
+  <visual>
+    <origin xyz="-0.015 0.0035 0.004"/>
+    <geometry>
+      <mesh filename="package://ca_description/meshes/sensors/asus_xtion_pro_live.dae"/>
+    </geometry>
+  </visual>
+</link>
+<joint name="${name}_depth_joint" type="fixed">
+  <origin xyz="0 ${xtion_pro_depth_rel_rgb_py} 0"/>
+  <parent link="${link_rgb}" />
+  <child link="${link_depth}"/>
+</joint>
+<link name="${link_depth}"/>
+<joint name="${name}_depth_optical_joint" type="fixed">
+  <origin rpy="${-pi/2} 0 ${-pi/2}" />
+  <parent link="${link_depth}" />
+  <child link="${link_depth_optical}" />
+</joint>
+<link name="${link_depth_optical}"/>
+<xacro:sim_3d_sensor name="${name}" color="Gazebo/FlatBlack"/>
 </robot>

Commit message: Fix astra rotation

File: ca_description/urdf/sensors/lasers/astra.xacro (robot description, xacro)
@@ -12,5 +12,5 @@
 <xacro:property name="optical_offset" value="0.01"/>
 <joint name="${name}_joint" type="fixed">
-  <origin xyz="${laser_origin}"/>
+  <origin xyz="${laser_origin}" rpy="${pi/2} 0 0"/>
   <parent link="${parent_link}"/>
   <child link="${link_name}"/>
@@ -18,5 +18,5 @@
 <link name="${link_name}">
   <visual>
-    <origin xyz="-0.01 0 -0.03" rpy="${pi/2} 0 ${pi/2}"/>
+    <origin xyz="-0.01 0 -0.03" rpy="0 0 ${pi/2}"/>
     <geometry>
       <mesh filename="package://ca_description/meshes/sensors/astra.dae"/>
