Commit message: Fix Tf for 3D cameras

File: ca_description/urdf/sensors/lasers/astra.xacro (robot description, xacro)
@@ -5,10 +5,11 @@
 <xacro:property name="name" value="astra"/>
 <xacro:property name="parent" value="base_link"/>
-<xacro:property name="parent_link"    value="${parent}"/>
-<xacro:property name="link_name"      value="${name}_link"/>
-<xacro:property name="link_rgb"       value="${name}_rgb_frame"/>
-<xacro:property name="link_depth"     value="${name}_depth_frame"/>
-<xacro:property name="link_optical"   value="${name}_depth_optical_frame"/>
-<xacro:property name="optical_offset" value="0.01"/>
+<xacro:property name="parent_link"        value="${parent}"/>
+<xacro:property name="link_name"          value="${name}_link"/>
+<xacro:property name="link_rgb"           value="${name}_rgb_frame"/>
+<xacro:property name="link_rgb_optical"   value="${name}_rgb_optical_frame"/>
+<xacro:property name="link_depth"         value="${name}_depth_frame"/>
+<xacro:property name="link_depth_optical" value="${name}_depth_optical_frame"/>
+<xacro:property name="optical_rotation" value="${-pi/2} 0 ${-pi/2}"/>
 <joint name="${name}_joint" type="fixed">
   <origin xyz="${laser_origin}"/>
@@ -24,12 +25,18 @@
   </visual>
 </link>
-<joint name="${name}_optical_joint" type="fixed">
-  <origin xyz="0 ${optical_offset} 0" rpy="${-pi/2} 0 ${-pi/2}"/>
+<joint name="${name}_rgb_joint" type="fixed">
+  <origin xyz="0 -0.045 0"/>
   <parent link="${link_name}"/>
   <child link="${link_rgb}"/>
 </joint>
 <link name="${link_rgb}"/>
+<joint name="${name}_rgb_optical_joint" type="fixed">
+  <origin rpy="${optical_rotation}"/>
+  <parent link="${link_rgb}"/>
+  <child link="${link_rgb_optical}"/>
+</joint>
+<link name="${link_rgb_optical}"/>
 <joint name="${name}_depth_joint" type="fixed">
-  <origin rpy="${-pi/2} 0 ${-pi/2}"/>
+  <origin xyz="0 -0.02 0"/>
   <parent link="${link_name}"/>
   <child link="${link_depth}"/>
@@ -37,9 +44,9 @@
 <link name="${link_depth}"/>
   <joint name="${name}_depth_optical_joint" type="fixed">
-  <origin rpy="${-pi/2} 0 ${-pi/2}"/>
+  <origin rpy="${optical_rotation}"/>
   <parent link="${link_depth}"/>
-  <child link="${link_optical}"/>
+  <child link="${link_depth_optical}"/>
 </joint>
-<link name="${link_optical}"/>
+<link name="${link_depth_optical}"/>
 <xacro:sim_3d_sensor name="${name}" color="Gazebo/FlatBlack"/>
 </robot>

File: ca_description/urdf/sensors/lasers/kinect.xacro (robot description, xacro)
@@ -10,5 +10,6 @@
 <xacro:property name="link_depth"         value="${name}_depth_frame"/>
 <xacro:property name="link_depth_optical" value="${name}_depth_optical_frame"/>
-<xacro:property name="kinect_cam_py" value="-0.0125"/>
+<xacro:property name="kinect_cam_py"    value="-0.0125"/>
+<xacro:property name="optical_rotation" value="${-pi/2} 0 ${-pi/2}"/>
 <joint name="camera_rgb_joint" type="fixed">
   <origin xyz="${laser_origin}"/>
@@ -18,5 +19,5 @@
 <link name="${link_rgb}"/>
 <joint name="${name}_rgb_optical_joint" type="fixed">
-  <origin rpy="${-pi/2} 0 ${-pi/2}" />
+  <origin rpy="${optical_rotation}" />
   <parent link="${link_rgb}" />
   <child link="${link_rgb_optical}" />
@@ -43,5 +44,5 @@
 <link name="${link_depth}"/>
 <joint name="${name}_depth_optical_joint" type="fixed">
-  <origin rpy="${-pi/2} 0 ${-pi/2}" />
+  <origin rpy="${optical_rotation}" />
   <parent link="${link_depth}" />
   <child link="${link_depth_optical}"/>

File: ca_description/urdf/sensors/lasers/r200.xacro (robot description, xacro)
@@ -10,6 +10,7 @@
 <xacro:property name="link_depth"         value="${name}_depth_frame"/>
 <xacro:property name="link_depth_optical" value="${name}_depth_optical_frame"/>
-<xacro:property name="rgb_offset"     value="-0.039895"/>
-<xacro:property name="depth_offset"   value="-0.045395"/>
+<xacro:property name="rgb_offset"       value="-0.039895"/>
+<xacro:property name="depth_offset"     value="-0.045395"/>
+<xacro:property name="optical_rotation" value="${-pi/2} 0 ${-pi/2}"/>
 <joint name="${name}_joint" type="fixed">
   <origin xyz="${laser_origin}"/>
@@ -31,5 +32,5 @@
 <link name="${link_rgb}"/>
 <joint name="${name}_rgb_optical_joint" type="fixed">
-    <origin rpy="${-pi/2} 0 ${-pi/2}"/>
+    <origin rpy="${optical_rotation}"/>
     <parent link="${link_rgb}"/>
     <child link="${link_rgb_optical}"/>
@@ -43,5 +44,5 @@
 <link name="${link_depth}"/>
 <joint name="${name}_depth_optical_joint" type="fixed">
-    <origin rpy="${-pi/2} 0 ${-pi/2}"/>
+    <origin rpy="${optical_rotation}"/>
     <parent link="${link_depth}"/>
     <child link="${link_depth_optical}"/>

File: ca_description/urdf/sensors/lasers/xtion_pro.xacro (robot description, xacro)
@@ -14,4 +14,5 @@
 <xacro:property name="xtion_pro_depth_rel_rgb_py" value="0.0270" />
 <xacro:property name="xtion_pro_cam_rel_rgb_py"   value="-0.0220" />
+<xacro:property name="optical_rotation"           value="${-pi/2} 0 ${-pi/2}"/>
 <joint name="${name}_rgb_joint" type="fixed">
   <origin xyz="${laser_origin}"/>
@@ -21,5 +22,5 @@
 <link name="${link_rgb}"/>
 <joint name="${name}_rgb_optical_joint" type="fixed">
-  <origin rpy="${-pi/2} 0 ${-pi/2}" />
+  <origin rpy="${optical_rotation}" />
   <parent link="${link_rgb}" />
   <child link="${link_rgb_optical}" />
@@ -46,5 +47,5 @@
 <link name="${link_depth}"/>
 <joint name="${name}_depth_optical_joint" type="fixed">
-  <origin rpy="${-pi/2} 0 ${-pi/2}" />
+  <origin rpy="${optical_rotation}" />
   <parent link="${link_depth}" />
   <child link="${link_depth_optical}" />

Commit message: Apply calibration to 3D sensors

File: ca_description/urdf/sensors/lasers/astra.xacro (robot description, xacro)
@@ -1,4 +1,5 @@
 <?xml version="1.0"?>
 <robot xmlns:xacro="http://ros.org/wiki/xacro">
+<xacro:include filename="$(find ca_description)/urdf/sensors/lasers/calibration.xacro"/>
 <xacro:include filename="$(find ca_description)/urdf/sensors/lasers/sim_3d_sensor.xacro"/>
 <!-- Orbbec Astra RGBD Camera -->
@@ -12,5 +13,4 @@
 <xacro:property name="link_depth"         value="${name}_depth_frame"/>
 <xacro:property name="link_depth_optical" value="${name}_depth_optical_frame"/>
-<xacro:property name="optical_rotation" value="${-pi/2} 0 ${-pi/2}"/>
 <joint name="${name}_joint" type="fixed">
   <origin xyz="${laser_origin}"/>
@@ -33,5 +33,5 @@
 <link name="${link_rgb}"/>
 <joint name="${name}_rgb_optical_joint" type="fixed">
-  <origin rpy="${optical_rotation}"/>
+  <xacro:origin_calibrated camera="${name}" type="rgb"/>
   <parent link="${link_rgb}"/>
   <child link="${link_rgb_optical}"/>
@@ -45,5 +45,5 @@
 <link name="${link_depth}"/>
   <joint name="${name}_depth_optical_joint" type="fixed">
-  <origin rpy="${optical_rotation}"/>
+  <xacro:origin_calibrated camera="${name}" type="depth"/>
   <parent link="${link_depth}"/>
   <child link="${link_depth_optical}"/>

File: ca_description/urdf/sensors/lasers/kinect.xacro (robot description, xacro)
@@ -1,4 +1,5 @@
 <?xml version="1.0"?>
 <robot xmlns:xacro="http://ros.org/wiki/xacro">
+<xacro:include filename="$(find ca_description)/urdf/sensors/lasers/calibration.xacro"/>
 <xacro:include filename="$(find ca_description)/urdf/sensors/lasers/sim_3d_sensor.xacro"/>
 <xacro:property name="name" value="kinect"/>
@@ -11,5 +12,4 @@
 <xacro:property name="link_depth_optical" value="${name}_depth_optical_frame"/>
 <xacro:property name="kinect_cam_py"    value="-0.0125"/>
-<xacro:property name="optical_rotation" value="${-pi/2} 0 ${-pi/2}"/>
 <joint name="camera_rgb_joint" type="fixed">
   <origin xyz="${laser_origin}"/>
@@ -19,5 +19,5 @@
 <link name="${link_rgb}"/>
 <joint name="${name}_rgb_optical_joint" type="fixed">
-  <origin rpy="${optical_rotation}" />
+  <xacro:origin_calibrated camera="${name}" type="rgb"/>
   <parent link="${link_rgb}" />
   <child link="${link_rgb_optical}" />
@@ -44,5 +44,5 @@
 <link name="${link_depth}"/>
 <joint name="${name}_depth_optical_joint" type="fixed">
-  <origin rpy="${optical_rotation}" />
+  <xacro:origin_calibrated camera="${name}" type="depth"/>
   <parent link="${link_depth}" />
   <child link="${link_depth_optical}"/>

File: ca_description/urdf/sensors/lasers/r200.xacro (robot description, xacro)
@@ -1,4 +1,5 @@
 <?xml version="1.0"?>
 <robot xmlns:xacro="http://www.ros.org/wiki/xacro">
+<xacro:include filename="$(find ca_description)/urdf/sensors/lasers/calibration.xacro"/>
 <xacro:include filename="$(find ca_description)/urdf/sensors/lasers/sim_3d_sensor.xacro"/>
 <xacro:property name="name" value="r200"/>
@@ -10,7 +11,6 @@
 <xacro:property name="link_depth"         value="${name}_depth_frame"/>
 <xacro:property name="link_depth_optical" value="${name}_depth_optical_frame"/>
-<xacro:property name="rgb_offset"       value="-0.039895"/>
-<xacro:property name="depth_offset"     value="-0.045395"/>
-<xacro:property name="optical_rotation" value="${-pi/2} 0 ${-pi/2}"/>
+<xacro:property name="rgb_offset"   value="-0.039895"/>
+<xacro:property name="depth_offset" value="-0.045395"/>
 <joint name="${name}_joint" type="fixed">
   <origin xyz="${laser_origin}"/>
@@ -26,25 +26,25 @@
 </link>
 <joint name="${name}_rgb_joint" type="fixed">
-    <origin xyz="0 ${rgb_offset} 0"/>
-    <parent link="${link_name}"/>
-    <child link="${link_rgb}" />
+  <origin xyz="0 ${rgb_offset} 0"/>
+  <parent link="${link_name}"/>
+  <child link="${link_rgb}" />
 </joint>
 <link name="${link_rgb}"/>
 <joint name="${name}_rgb_optical_joint" type="fixed">
-    <origin rpy="${optical_rotation}"/>
-    <parent link="${link_rgb}"/>
-    <child link="${link_rgb_optical}"/>
+  <xacro:origin_calibrated camera="${name}" type="rgb"/>
+  <parent link="${link_rgb}"/>
+  <child link="${link_rgb_optical}"/>
 </joint>
 <link name="${link_rgb_optical}"/>
 <joint name="${name}_depth_joint" type="fixed">
-    <origin xyz="0 ${depth_offset} 0"/>
-    <parent link="${link_name}"/>
-    <child link="${link_depth}"/>
+  <origin xyz="0 ${depth_offset} 0"/>
+  <parent link="${link_name}"/>
+  <child link="${link_depth}"/>
 </joint>
 <link name="${link_depth}"/>
 <joint name="${name}_depth_optical_joint" type="fixed">
-    <origin rpy="${optical_rotation}"/>
-    <parent link="${link_depth}"/>
-    <child link="${link_depth_optical}"/>
+  <xacro:origin_calibrated camera="${name}" type="depth"/>
+  <parent link="${link_depth}"/>
+  <child link="${link_depth_optical}"/>
 </joint>
 <link name="${link_depth_optical}"/>

File: ca_description/urdf/sensors/lasers/xtion_pro.xacro (robot description, xacro)
@@ -1,4 +1,5 @@
 <?xml version="1.0"?>
 <robot xmlns:xacro="http://ros.org/wiki/xacro">
+<xacro:include filename="$(find ca_description)/urdf/sensors/lasers/calibration.xacro"/>
 <xacro:include filename="$(find ca_description)/urdf/sensors/lasers/sim_3d_sensor.xacro"/>
 <!-- Orbbec Astra RGBD Camera -->
@@ -15,8 +16,7 @@
 <!-- This relates the IR sensor to the Xtion base link -->
 <!-- 4.8 cm because sensors are offset to right, from center -->
-<xacro:property name="ir_offset"        value="0.048"/>
+<xacro:property name="ir_offset"  value="0.048"/>
 <!-- The measured distance from RGB lens back to IR lens, approx 2.5cm -->
-<xacro:property name="rgb_offset"       value="-0.025"/>
-<xacro:property name="optical_rotation" value="${-pi/2} 0 ${-pi/2}"/>
+<xacro:property name="rgb_offset" value="-0.025"/>
 <joint name="${name}_joint" type="fixed">
   <origin xyz="${laser_origin}"/>
@@ -41,5 +41,5 @@
 <!-- Xtion RGB sensor frame -->
 <joint name="${name}_rgb_optical_joint" type="fixed">
-  <origin rpy="${optical_rotation}" />
+  <xacro:origin_calibrated camera="${name}" type="rgb"/>
   <parent link="${link_rgb}" />
   <child link="${link_rgb_optical}" />
@@ -55,5 +55,5 @@
 <!-- Xtion IR sensor frame -->
 <joint name="${name}_depth_optical_joint" type="fixed">
-  <origin rpy="${optical_rotation}" />
+  <xacro:origin_calibrated camera="${name}" type="depth"/>
   <parent link="${link_depth}" />
   <child link="${link_depth_optical}" />
