Commit message: Fix Lidar error

File: ca_description/urdf/sensors/lasers/rplidar.xacro (robot description, xacro)
@@ -1,17 +1,17 @@
 <?xml version="1.0"?>
 <robot xmlns:xacro="http://ros.org/wiki/xacro">
-<xacro:property name="name" value="rplidar"/>
-<xacro:property name="parent" value="base_link"/>
-<xacro:property name="parent_link"              value="${parent}"/>
-<xacro:property name="link_name"                value="${name}_link"/>
-<xacro:property name="laser_link"               value="laser_link"/>
-<xacro:property name="rplidar_a2_rate_hz"       value="10"/>
-<xacro:property name="rplidar_a2_min_range_m"   value="0.15"/>
-<xacro:property name="rplidar_a2_max_range_m"   value="12.0"/>
-<xacro:property name="rplidar_a2_samples"       value="720"/>
-<xacro:property name="rplidar_a2_resolution_mm" value="0.5"/>
-<xacro:property name="rplidar_a2_min_angle_rad" value="${-pi}"/>
-<xacro:property name="rplidar_a2_max_angle_rad" value="${pi}"/>
-<xacro:property name="topic_name"               value="laser/scan"/>
+<xacro:property name="name"          value="rplidar"/>
+<xacro:property name="parent"        value="base_link"/>
+<xacro:property name="parent_link"   value="${parent}"/>
+<xacro:property name="link_name"     value="${name}_link"/>
+<xacro:property name="laser_link"    value="laser_link"/>
+<xacro:property name="rate_hz"       value="10"/>
+<xacro:property name="min_range_m"   value="0.15"/>
+<xacro:property name="max_range_m"   value="12.0"/>
+<xacro:property name="samples"       value="720"/>
+<xacro:property name="resolution_mm" value="0.5"/>
+<xacro:property name="min_angle_rad" value="${-pi}"/>
+<xacro:property name="max_angle_rad" value="${pi}"/>
+<xacro:property name="topic_name"    value="laser/scan"/>
 <joint name="${name}_joint" type="fixed">
   <origin xyz="${laser_origin}"/>
@@ -35,19 +35,19 @@
   <material>Gazebo/FlatBlack</material>
   <sensor type="ray" name="${name}_sensor">
-    <visualize>${visualize}</visualize>
-    <update_rate>${rplidar_a2_rate_hz}</update_rate>
+    <visualize>$(arg visualize)</visualize>
+    <update_rate>${rate_hz}</update_rate>
     <ray>
       <scan>
         <horizontal>
-          <samples>${rplidar_a2_samples}</samples>
+          <samples>${samples}</samples>
           <resolution>1</resolution>
-          <min_angle>${rplidar_a2_min_angle_rad}</min_angle>
-          <max_angle>${rplidar_a2_max_angle_rad}</max_angle>
+          <min_angle>${min_angle_rad}</min_angle>
+          <max_angle>${max_angle_rad}</max_angle>
         </horizontal>
       </scan>
       <range>
-        <min>${rplidar_a2_min_range_m}</min>
-        <max>${rplidar_a2_max_range_m}</max>
-        <resolution>${rplidar_a2_resolution_mm / 1000.0}</resolution>
+        <min>${min_range_m}</min>
+        <max>${max_range_m}</max>
+        <resolution>${resolution_mm / 1000.0}</resolution>
       </range>
       <noise>

Commit message: fixup! Improve LiDAR config

File: ca_description/urdf/sensors/lasers/rplidar.xacro (robot description, xacro)
@@ -15,5 +15,5 @@
 <xacro:property name="topic_name"    value="${name}/scan"/>
 <joint name="${name}_joint" type="fixed">
-  <origin xyz="${laser_origin}"/>
+  <origin xyz="${laser_origin}" rpy="0 0 ${pi}"/>
   <parent link="${parent_link}"/>
   <child link="${link_name}"/>
