Commit message: Improve turtlebot.xacro

File: ca_description/urdf/stacks/turtlebot.xacro (robot description, xacro)
@@ -2,4 +2,5 @@
 <!--
   Hexagon stacks
+  https://github.com/turtlebot/turtlebot/blob/melodic/turtlebot_description/urdf/stacks/hexagons.urdf.xacro
  -->
 <robot xmlns:xacro="http://ros.org/wiki/xacro">
@@ -19,10 +20,4 @@
         </geometry>
       </visual>
-      <!-- <inertial>
-        <mass value="0.008"/>
-        <inertia ixx="0.000001686" ixy="0.0" ixz="0.0"
-                 iyy="0.000001686" iyz="0.0"
-                 izz="0.000000144"/>
-      </inertial> -->
     </link>
   </xacro:macro>
@@ -41,10 +36,34 @@
         </geometry>
       </visual>
-      <!-- <inertial>
-        <mass value="0.012"/>
-        <inertia ixx="0.000003805" ixy="0.0" ixz="0.0"
-                 iyy="0.000003805" iyz="0.0"
-                 izz="0.000000216"/>
-      </inertial> -->
+    </link>
+  </xacro:macro>
+  <xacro:macro name="stack_top_pole" params="parent:=base_link number *origin">
+    <xacro:property name="link_name" value="pole_top_${number}_link"/>
+    <joint name="pole_top_${number}_joint" type="fixed">
+      <xacro:insert_block name="origin"/>
+      <parent link="${parent}"/>
+      <child link="${link_name}"/>
+    </joint>
+    <link name="${link_name}">
+      <visual>
+        <geometry>
+          <mesh filename="package://ca_description/meshes/turtlebot_stack/pole_top.dae"/>
+        </geometry>
+      </visual>
+    </link>
+  </xacro:macro>
+  <xacro:macro name="stack_3d_sensor_pole" params="parent:=base_link number *origin">
+    <xacro:property name="link_name" value="pole_kinect_${number}_link"/>
+    <joint name="pole_kinect_${number}_joint" type="fixed">
+      <xacro:insert_block name="origin"/>
+      <parent link="${parent}"/>
+      <child link="${link_name}"/>
+    </joint>
+    <link name="${link_name}">
+      <visual>
+        <geometry>
+          <mesh filename="package://ca_description/meshes/turtlebot_stack/pole_kinect.dae"/>
+        </geometry>
+      </visual>
     </link>
   </xacro:macro>
@@ -84,10 +103,4 @@
         </geometry>
       </visual>
-      <!-- <inertial>
-        <mass value="0.520" />
-        <inertia ixx="0.003328" ixy="0.0" ixz="0.0"
-                 iyy="0.003328" iyz="0.0"
-                 izz="0.006656" />
-      </inertial> -->
     </link>
     <xacro:stack_middle_pole number="0">
@@ -114,10 +127,34 @@
         </geometry>
       </visual>
-      <!-- <inertial>
-        <mass value="0.520" />
-        <inertia ixx="0.003328" ixy="0.0" ixz="0.0"
-                 iyy="0.003328" iyz="0.0"
-                 izz="0.006656" />
-      </inertial> -->
+    </link>
+    <xacro:stack_top_pole number="0">
+      <origin xyz="0.0381 0.1505 0.2920"/>
+    </xacro:stack_top_pole>
+    <xacro:stack_top_pole number="1">
+      <origin xyz="0.0381 -0.1505 0.2920"/>
+    </xacro:stack_top_pole>
+    <xacro:stack_top_pole number="2">
+      <origin xyz="-0.0381 0.1505 0.2920"/>
+    </xacro:stack_top_pole>
+    <xacro:stack_top_pole number="3">
+      <origin xyz="-0.0381 -0.1505 0.2920"/>
+    </xacro:stack_top_pole>
+    <xacro:stack_3d_sensor_pole number="0">
+      <origin xyz="-0.1024 0.098 0.2372"/>
+    </xacro:stack_3d_sensor_pole>
+    <xacro:stack_3d_sensor_pole number="1">
+      <origin xyz="-0.1024 -0.098 0.2372"/>
+    </xacro:stack_3d_sensor_pole>
+    <joint name="plate_top_joint" type="fixed">
+      <origin xyz="-0.01364 0 0.3966"/>
+      <parent link="${parent}"/>
+      <child link="plate_top_link"/>
+    </joint>
+    <link name="plate_top_link">
+      <visual>
+        <geometry>
+          <mesh filename="package://ca_description/meshes/turtlebot_stack/plate_top.dae"/>
+        </geometry>
+      </visual>
     </link>
   </xacro:macro>

Commit message: Improve Turtlebot stack

File: ca_description/urdf/stacks/turtlebot.xacro (robot description, xacro)
@@ -5,8 +5,8 @@
  -->
 <robot xmlns:xacro="http://ros.org/wiki/xacro">
-  <!-- Pole macros -->
-  <xacro:macro name="stack_bottom_pole" params="parent:=base_link number *origin">
-    <xacro:property name="link_name" value="pole_bottom_${number}_link"/>
-    <joint name="pole_bottom_${number}_joint" type="fixed">
+  <!-- Pole macro -->
+  <xacro:macro name="stack_pole" params="name parent:=base_link *origin *mesh">
+    <xacro:property name="link_name" value="pole_${name}_link"/>
+    <joint name="pole_${name}_joint" type="fixed">
       <xacro:insert_block name="origin"/>
       <parent link="${parent}"/>
@@ -16,51 +16,5 @@
       <visual>
         <geometry>
-          <mesh filename="package://ca_description/meshes/turtlebot_stack/pole_bottom.dae"/>
-        </geometry>
-      </visual>
-    </link>
-  </xacro:macro>
-  <xacro:macro name="stack_middle_pole" params="parent:=base_link number *origin">
-    <xacro:property name="link_name" value="pole_middle_${number}_link"/>
-    <joint name="pole_middle_${number}_joint" type="fixed">
-      <xacro:insert_block name="origin"/>
-      <parent link="${parent}"/>
-      <child link="${link_name}"/>
-    </joint>
-    <link name="${link_name}">
-      <visual>
-        <origin rpy="0 ${pi} 0"/>
-        <geometry>
-          <mesh filename="package://ca_description/meshes/turtlebot_stack/pole_middle.dae"/>
-        </geometry>
-      </visual>
-    </link>
-  </xacro:macro>
-  <xacro:macro name="stack_top_pole" params="parent:=base_link number *origin">
-    <xacro:property name="link_name" value="pole_top_${number}_link"/>
-    <joint name="pole_top_${number}_joint" type="fixed">
-      <xacro:insert_block name="origin"/>
-      <parent link="${parent}"/>
-      <child link="${link_name}"/>
-    </joint>
-    <link name="${link_name}">
-      <visual>
-        <geometry>
-          <mesh filename="package://ca_description/meshes/turtlebot_stack/pole_top.dae"/>
-        </geometry>
-      </visual>
-    </link>
-  </xacro:macro>
-  <xacro:macro name="stack_3d_sensor_pole" params="parent:=base_link number *origin">
-    <xacro:property name="link_name" value="pole_kinect_${number}_link"/>
-    <joint name="pole_kinect_${number}_joint" type="fixed">
-      <xacro:insert_block name="origin"/>
-      <parent link="${parent}"/>
-      <child link="${link_name}"/>
-    </joint>
-    <link name="${link_name}">
-      <visual>
-        <geometry>
-          <mesh filename="package://ca_description/meshes/turtlebot_stack/pole_kinect.dae"/>
+          <xacro:insert_block name="mesh"/>
         </geometry>
       </visual>
@@ -73,24 +27,22 @@
   -->
   <xacro:macro name="turtlebot_stack" params="name:=turtlebot_stack parent:=base_link *origin">
-    <xacro:stack_bottom_pole number="0">
-      <origin xyz="0.12 0.082 0.1028"/>
-    </xacro:stack_bottom_pole>
-    <xacro:stack_bottom_pole number="1">
-      <origin xyz="0.055 0.12 0.1028"/>
-    </xacro:stack_bottom_pole>
-    <xacro:stack_bottom_pole number="2">
-      <origin xyz="-0.055 0.12 0.1028"/>
-    </xacro:stack_bottom_pole>
-    <xacro:stack_bottom_pole number="3">
-      <origin xyz="0.12 -0.082 0.1028"/>
-    </xacro:stack_bottom_pole>
-    <xacro:stack_bottom_pole number="4">
-      <origin xyz="0.055 -0.12 0.1028"/>
-    </xacro:stack_bottom_pole>
-    <xacro:stack_bottom_pole number="5">
-      <origin xyz="-0.055 -0.12 0.1028"/>
-    </xacro:stack_bottom_pole>
+    <xacro:stack_pole name="short_0">
+      <origin xyz="0.0381 0.1 0.093"/>
+      <mesh filename="package://ca_description/meshes/turtlebot_stack/short_pole.dae"/>
+    </xacro:stack_pole>
+    <xacro:stack_pole name="short_1">
+      <origin xyz="0.0381 -0.1 0.093"/>
+      <mesh filename="package://ca_description/meshes/turtlebot_stack/short_pole.dae"/>
+    </xacro:stack_pole>
+    <xacro:stack_pole name="short_2">
+      <origin xyz="-0.0381 0.1 0.093"/>
+      <mesh filename="package://ca_description/meshes/turtlebot_stack/short_pole.dae"/>
+    </xacro:stack_pole>
+    <xacro:stack_pole name="short_3">
+      <origin xyz="-0.0381 -0.1 0.093"/>
+      <mesh filename="package://ca_description/meshes/turtlebot_stack/short_pole.dae"/>
+    </xacro:stack_pole>
     <joint name="plate_bottom_joint" type="fixed">
-      <origin xyz="0.02364 0.0 0.1306"/>
+      <origin xyz="-0.01364 0 0.125"/>
       <parent link="${parent}"/>
       <child link="plate_bottom_link"/>
@@ -99,59 +51,33 @@
       <visual>
         <geometry>
-          <mesh filename="package://ca_description/meshes/turtlebot_stack/plate_bottom.dae"/>
+          <mesh filename="package://ca_description/meshes/turtlebot_stack/bottom_plate.dae" scale="0.5 0.7 1"/>
         </geometry>
       </visual>
     </link>
-    <xacro:stack_middle_pole number="0">
-      <origin xyz="0.0381 0.1505 0.1640"/>
-    </xacro:stack_middle_pole>
-    <xacro:stack_middle_pole number="1">
-      <origin xyz="-0.0381 -0.1505 0.1640"/>
-    </xacro:stack_middle_pole>
-    <xacro:stack_middle_pole number="2">
-      <origin xyz="-0.0381 0.1505 0.1640"/>
-    </xacro:stack_middle_pole>
-    <xacro:stack_middle_pole number="3">
-      <origin xyz="-0.0381 -0.1505 0.1640"/>
-    </xacro:stack_middle_pole>
-    <joint name="plate_middle_joint" type="fixed">
-      <origin xyz="-0.01364 0 0.1874"/>
+    <xacro:stack_pole name="large_0">
+      <origin xyz="0.1 0.098 0.18"/>
+      <mesh filename="package://ca_description/meshes/turtlebot_stack/large_pole.dae"/>
+    </xacro:stack_pole>
+    <xacro:stack_pole name="large_1">
+      <origin xyz="0.1 -0.098 0.18"/>
+      <mesh filename="package://ca_description/meshes/turtlebot_stack/large_pole.dae"/>
+    </xacro:stack_pole>
+    <xacro:stack_pole name="large_2">
+      <origin xyz="-0.1 0.098 0.18"/>
+      <mesh filename="package://ca_description/meshes/turtlebot_stack/large_pole.dae"/>
+    </xacro:stack_pole>
+    <xacro:stack_pole name="large_3">
+      <origin xyz="-0.1 -0.098 0.18"/>
+      <mesh filename="package://ca_description/meshes/turtlebot_stack/large_pole.dae"/>
+    </xacro:stack_pole>
+    <joint name="plate_upper_joint" type="fixed">
+      <origin xyz="-0.01364 0 0.2"/>
       <parent link="${parent}"/>
-      <child link="plate_middle_link"/>
+      <child link="plate_upper_link"/>
     </joint>
-    <link name="plate_middle_link">
+    <link name="plate_upper_link">
       <visual>
         <geometry>
-          <mesh filename="package://ca_description/meshes/turtlebot_stack/plate_middle.dae"/>
-        </geometry>
-      </visual>
-    </link>
-    <xacro:stack_top_pole number="0">
-      <origin xyz="0.0381 0.1505 0.2920"/>
-    </xacro:stack_top_pole>
-    <xacro:stack_top_pole number="1">
-      <origin xyz="0.0381 -0.1505 0.2920"/>
-    </xacro:stack_top_pole>
-    <xacro:stack_top_pole number="2">
-      <origin xyz="-0.0381 0.1505 0.2920"/>
-    </xacro:stack_top_pole>
-    <xacro:stack_top_pole number="3">
-      <origin xyz="-0.0381 -0.1505 0.2920"/>
-    </xacro:stack_top_pole>
-    <xacro:stack_3d_sensor_pole number="0">
-      <origin xyz="-0.1024 0.098 0.2372"/>
-    </xacro:stack_3d_sensor_pole>
-    <xacro:stack_3d_sensor_pole number="1">
-      <origin xyz="-0.1024 -0.098 0.2372"/>
-    </xacro:stack_3d_sensor_pole>
-    <joint name="plate_top_joint" type="fixed">
-      <origin xyz="-0.01364 0 0.3966"/>
-      <parent link="${parent}"/>
-      <child link="plate_top_link"/>
-    </joint>
-    <link name="plate_top_link">
-      <visual>
-        <geometry>
-          <mesh filename="package://ca_description/meshes/turtlebot_stack/plate_top.dae"/>
+          <mesh filename="package://ca_description/meshes/turtlebot_stack/upper_plate.dae"/>
         </geometry>
       </visual>

Commit message: Add Nvidia Jetson Nano

File: ca_description/urdf/stacks/turtlebot.xacro (robot description, xacro)
@@ -87,7 +87,8 @@
   </visual>
 </link>
+<!-- Nvidia Jetson Nano -->
 <joint name="nvidia_jetson_nano_joint" type="fixed">
-  <origin xyz="0 0 0.117"/>
-  <parent link="${base_link}"/>
+  <origin xyz="0 0 0.003" rpy="0 0 ${-pi/2}"/>
+  <parent link="plate_bottom_link"/>
   <child link="nvidia_jetson_nano_link"/>
 </joint>
@@ -95,8 +96,11 @@
   <visual>
     <geometry>
-      <mesh filename="package://ca_description/meshes/nvidia_jetson_nano.dae"/>
+      <mesh filename="package://ca_description/meshes/turtlebot_stack/nvidia_jetson_nano.dae"/>
     </geometry>
   </visual>
 </link>
+<gazebo reference="nvidia_jetson_nano_link">
+  <material>Gazebo/Grey</material>
+</gazebo>
 <!-- Laser -->
 <xacro:property name="laser" default="$(arg laser)"/>
